File: atari-16-32-bits/motherboards/c300780-001/sheet_1.sch (KiCad schematic (older format))
At the start: 0 parts

Commit message: done u100,u101
Changed lines of the file:
@@
 F0 "U100 - MC68000" 50
 F1 "subsheet_100.sch" 50
-F2 "DATA" T R 3500 1100 50
 $EndSheet
 $Sheet

Commit message: sheet 1 done
Changed lines of the file:
@@
 S 1000 8500 2500 1000
 U 6078774E
-F0 "J100 -- Power connector, bypass capacitors and pull-ups" 50
+F0 "J100 -- Power connector" 50
 F1 "subsheet_105.sch" 50
 $EndSheet
@@
 S 4500 7000 2500 2500
 U 60787796
-F0 "32 MHz source" 50
+F0 "32 MHz clock and video clocks" 50
 F1 "subsheet_106.sch" 50
 $EndSheet
