File: atari-16-32-bits/motherboards/c300780-001/subsheet_302.sch (KiCad schematic (older format))
At the start: 0 parts

Commit message: done subsheet 302 : floppy drives controller and ports
Parts:
- added C304, C305: 0.1uF, symbol Device:C
- added J302: Internal FDD Power, symbol Connector_Generic:Conn_01x04
- added J303: Internal FDD Port, symbol Connector_Generic:Conn_02x17_Odd_Even
- added J304: DIN 14 — External FDD Port, symbol Connector_Generic:Conn_01x14
- added L300, L301, L302, L303, L304, L305, L306, L307, L308, L309, L310, L311: EMI_Filter_LCL, symbol Device:EMI_Filter_LCL
- added R300, R301, R302, R304, R305, R306: 1K, symbol Device:R_Small_US
- added R307: 220, symbol Device:R_Small_US
- added R308, R309, R310, R311: 47, symbol Device:R_Small_US
- added U301: WD1772_FLOPPY_DISK_CONTROLLER_AND_FORMATTER_PHY, Package_DIP:DIP-28_W15.24mm_LongPads, symbol wd1772:WD1772_FLOPPY_DISK_CONTROLLER_AND_FORMATTER_PHY
- added U305: 7406_PHY, Package_DIP:DIP-14_W7.62mm_LongPads, symbol 74x06:7406_PHY
- added W300, W301: SW_SPDT, symbol Switch:SW_SPDT
Connections:
- new net: R302.1, W300.3 (C)
- new net: L308.1, W301.2 (B)
- new net: L307.1, W300.2 (B)
- new net +12V: J302.4 (Pin_4)
- new net ACSI_19_HDRQ: R300.1, U305.13 (6A)
- new net CA1: U301.3 (A0)
- new net CA2: U301.4 (A1)
- new net CD0: U301.5 (DAL0)
- new net CD1: U301.6 (DAL1)
- new net CD2: U301.7 (DAL2)
- new net CD3: U301.8 (DAL3)
- new net CD4: U301.9 (DAL4)
- new net CD5: U301.10 (DAL5)
- new net CD6: U301.11 (DAL6)
- new net CD7: U301.12 (DAL7)
- new net D0SEL: J303.10 (Pin_10), W301.1 (A)
- new net D1SEL: J303.12 (Pin_12), W300.1 (A), W301.3 (C)
- new net DMA_FDCS: U301.1 (~CS~)
- new net DMA_FDRQ: U301.27 (DRQ)
- new net DMA_HDRQ: R301.1, U305.12 (6Y)
- new net DMA_RW: U301.2 (R/~W~)
- new net DRV_DOIN: J303.18 (Pin_18), L305.1, R311.1
- new net DRV_MON: J303.16 (Pin_16), L306.1, U305.10 (5Y)
- new net DRV_STEP: J303.20 (Pin_20), L304.1, R310.1
- new net DRV_WDATA: J303.22 (Pin_22), L303.1, R309.1
- new net DRV_WGATE: J303.24 (Pin_24), L302.1, R308.1
- new net FDINT: U301.28 (INTRQ)
- new net GND: C304.2, C305.2, J302.2 (Pin_2), J302.3 (Pin_3), J303.1 (Pin_1), J303.11 (Pin_11), J303.13 (Pin_13), J303.15 (Pin_15), J303.17 (Pin_17), J303.19 (Pin_19), J303.21 (Pin_21), J303.23 (Pin_23), J303.25 (Pin_25), J303.27 (Pin_27), J303.29 (Pin_29), J303.3 (Pin_3), J303.31 (Pin_31), J303.33 (Pin_33), J303.5 (Pin_5), J303.7 (Pin_7), J303.9 (Pin_9), J304.3 (Pin_3), J304.7 (Pin_7), L300.2, L301.2, L302.2, L303.2, L304.2, L305.2, L306.2, L307.2, L308.2, L309.2, L310.2, L311.2, U301.14 (GND), U301.26 (~DDEN~), U305.7 (GND)
- new net S0SEL: J303.32 (Pin_32), L310.1
- new net SCLK: U301.18 (CLK)
- new net VCC: C304.1, C305.1, J302.1 (Pin_1), R300.2, R301.2, R302.2, R304.1, R305.1, R306.1, R307.1, U301.15 (Vcc), U305.14 (Vcc)
- new net XRESET: U301.13 (~MR~)
- new net dirc: U301.17 (DIRC), U305.9 (4A)
- new net ext_fdc_1: J304.1 (Pin_1), L311.3
- new net ext_fdc_10: J304.10 (Pin_10), L304.3
- new net ext_fdc_11: J304.11 (Pin_11), L303.3
- new net ext_fdc_12: J304.12 (Pin_12), L302.3
- new net ext_fdc_13: J304.13 (Pin_13), L301.3
- new net ext_fdc_14: J304.14 (Pin_14), L300.3
- new net ext_fdc_2: J304.2 (Pin_2), L310.3
- new net ext_fdc_4: J304.4 (Pin_4), L309.3
- new net ext_fdc_5: J304.5 (Pin_5), L308.3
- new net ext_fdc_6: J304.6 (Pin_6), L307.3
- new net ext_fdc_8: J304.8 (Pin_8), L306.3
- new net ext_fdc_9: J304.9 (Pin_9), L305.3
- new net ip: J303.8 (Pin_8), L309.1, R306.2, U301.24 (~IP~)
- new net mo: U301.20 (MO), U305.11 (5A)
- new net not_dirc: R311.2, U305.8 (4Y)
- new net not_step: R310.2, U305.6 (3Y)
- new net not_wd: R309.2, U305.4 (2Y)
- new net not_wg: R308.2, U305.2 (1Y)
- new net rd: J303.30 (Pin_30), L311.1, R307.2, U301.19 (~RD~)
- new net step: U301.16 (STEP), U305.5 (3A)
- new net tr00: J303.26 (Pin_26), L301.1, R305.2, U301.23 (~TR00~)
- new net wd: U301.22 (WD), U305.3 (2A)
- new net wg: U301.21 (WG), U305.1 (1A)
- new net wprt: J303.28 (Pin_28), L300.1, R304.2, U301.25 (~WPRT~)
- no-connect marks 0 -> 5
Other:
- note added: "Factory setting : D1SEL"
- note added: "Factory setting : VCC"
