File: atari-16-32-bits/motherboards/c300780-001/subsheet_302.sch (KiCad schematic (older format))
At the start: 32 parts, among them J302 Internal FDD Power, J303 Internal FDD Port, J304 DIN 14 — External FDD Port, U301 WD1772_FLOPPY_DISK_CONTROLLER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, U305 7406_PHY

Commit message: [PCB] Assign builtins footprint when possible - resistors, ports
Parts:
- J302: footprint (none) -> Connector_Molex:Molex_KK-254_AE-6410-04A_1x04_P2.54mm_Vertical
- J303: footprint (none) -> Connector_IDC:IDC-Header_2x17_P2.54mm_Vertical
- R300, R301, R302, R304, R305, R306, R307, R308, R309, R310, R311: footprint (none) -> Resistor_THT:R_Axial_DIN0204_L3.6mm_D1.6mm_P7.62mm_Horizontal
Changed lines of the file:
@@
 F 0 "R304" V 4900 2000 50  0000 C CNN
 F 1 "1K" V 5100 2000 50  0000 C CNN
-F 2 "" H 5000 2000 50  0001 C CNN
+F 2 "Resistor_THT:R_Axial_DIN0204_L3.6mm_D1.6mm_P7.62mm_Horizontal" H 5000 2000 50  0001 C CNN
 F 3 "~" H 5000 2000 50  0001 C CNN
 	1    5000 2000
@@
 F 0 "R307" V 6150 2500 50  0000 C CNN
 F 1 "220" V 6350 2500 50  0000 C CNN
-F 2 "" H 6250 2500 50  0001 C CNN
+F 2 "Resistor_THT:R_Axial_DIN0204_L3.6mm_D1.6mm_P7.62mm_Horizontal" H 6250 2500 50  0001 C CNN
 F 3 "~" H 6250 2500 50  0001 C CNN
 	1    6250 2500
@@
 F 0 "R305" V 6150 2000 50  0000 C CNN
 F 1 "1K" V 6350 2000 50  0000 C CNN
-F 2 "" H 6250 2000 50  0001 C CNN
+F 2 "Resistor_THT:R_Axial_DIN0204_L3.6mm_D1.6mm_P7.62mm_Horizontal" H 6250 2000 50  0001 C CNN
 F 3 "~" H 6250 2000 50  0001 C CNN
 	1    6250 2000
@@
 F 0 "R306" V 4900 2500 50  0000 C CNN
 F 1 "1K" V 5100 2500 50  0000 C CNN
-F 2 "" H 5000 2500 50  0001 C CNN
+F 2 "Resistor_THT:R_Axial_DIN0204_L3.6mm_D1.6mm_P7.62mm_Horizontal" H 5000 2500 50  0001 C CNN
 F 3 "~" H 5000 2500 50  0001 C CNN
 	1    5000 2500
@@
 F 0 "R301" V 6100 3700 50  0000 C CNN
 F 1 "1K" V 6300 3700 50  0000 C CNN
-F 2 "" H 6200 3700 50  0001 C CNN
+F 2 "Resistor_THT:R_Axial_DIN0204_L3.6mm_D1.6mm_P7.62mm_Horizontal" H 6200 3700 50  0001 C CNN
 F 3 "~" H 6200 3700 50  0001 C CNN
 	1    6200 3700
@@
 F 0 "R300" V 4800 3700 50  0000 C CNN
 F 1 "1K" V 5000 3700 50  0000 C CNN
-F 2 "" H 4900 3700 50  0001 C CNN
+F 2 "Resistor_THT:R_Axial_DIN0204_L3.6mm_D1.6mm_P7.62mm_Horizontal" H 4900 3700 50  0001 C CNN
 F 3 "~" H 4900 3700 50  0001 C CNN
 	1    4900 3700
@@
 F 0 "R308" V 5000 4200 50  0000 C CNN
 F 1 "47" V 5200 4200 50  0000 C CNN
-F 2 "" H 5100 4200 50  0001 C CNN
+F 2 "Resistor_THT:R_Axial_DIN0204_L3.6mm_D1.6mm_P7.62mm_Horizontal" H 5100 4200 50  0001 C CNN
 F 3 "~" H 5100 4200 50  0001 C CNN
 	1    5100 4200
@@
 F 0 "R310" V 5000 4700 50  0000 C CNN
 F 1 "47" V 5200 4700 50  0000 C CNN
-F 2 "" H 5100 4700 50  0001 C CNN
+F 2 "Resistor_THT:R_Axial_DIN0204_L3.6mm_D1.6mm_P7.62mm_Horizontal" H 5100 4700 50  0001 C CNN
 F 3 "~" H 5100 4700 50  0001 C CNN
 	1    5100 4700
@@
 F 0 "R309" V 6300 4200 50  0000 C CNN
 F 1 "47" V 6500 4200 50  0000 C CNN
-F 2 "" H 6400 4200 50  0001 C CNN
+F 2 "Resistor_THT:R_Axial_DIN0204_L3.6mm_D1.6mm_P7.62mm_Horizontal" H 6400 4200 50  0001 C CNN
 F 3 "~" H 6400 4200 50  0001 C CNN
 	1    6400 4200
@@
 F 0 "R311" V 6300 4700 50  0000 C CNN
 F 1 "47" V 6500 4700 50  0000 C CNN
-F 2 "" H 6400 4700 50  0001 C CNN
+F 2 "Resistor_THT:R_Axial_DIN0204_L3.6mm_D1.6mm_P7.62mm_Horizontal" H 6400 4700 50  0001 C CNN
 F 3 "~" H 6400 4700 50  0001 C CNN
 	1    6400 4700
@@
 F 0 "J302" H 1750 9350 50  0000 C CNN
 F 1 "Internal FDD Power" H 1750 8850 50  0000 C CNN
-F 2 "" H 1750 9150 50  0001 C CNN
+F 2 "Connector_Molex:Molex_KK-254_AE-6410-04A_1x04_P2.54mm_Vertical" H 1750 9150 50  0001 C CNN
 F 3 "~" H 1750 9150 50  0001 C CNN
 	1    1750 9150
@@
 F 0 "J303" H 6000 7000 50  0000 C CNN
 F 1 "Internal FDD Port" H 6000 5200 50  0000 C CNN
-F 2 "" H 5950 6100 50  0001 C CNN
+F 2 "Connector_IDC:IDC-Header_2x17_P2.54mm_Vertical" H 5950 6100 50  0001 C CNN
 F 3 "~" H 5950 6100 50  0001 C CNN
 	1    5950 6100
@@
 F 0 "R302" V 1450 6850 50  0000 C CNN
 F 1 "1K" V 1650 6850 50  0000 C CNN
-F 2 "" H 1550 6850 50  0001 C CNN
+F 2 "Resistor_THT:R_Axial_DIN0204_L3.6mm_D1.6mm_P7.62mm_Horizontal" H 1550 6850 50  0001 C CNN
 F 3 "~" H 1550 6850 50  0001 C CNN
 	1    1550 6850

Commit message: [PCB] continuing footprint assignement
Parts:
- W300, W301: footprint (none) -> Connector_PinHeader_2.54mm:PinHeader_1x03_P2.54mm_Vertical
Changed lines of the file:
@@
 F 0 "W300" H 2300 6920 50  0000 C CNN
 F 1 "SW_SPDT" H 2300 6550 50  0000 C CNN
-F 2 "" H 2300 6750 50  0001 C CNN
+F 2 "Connector_PinHeader_2.54mm:PinHeader_1x03_P2.54mm_Vertical" H 2300 6750 50  0001 C CNN
 F 3 "~" H 2300 6750 50  0001 C CNN
 	1    2300 6750
@@
 F 0 "W301" H 2550 6420 50  0000 C CNN
 F 1 "SW_SPDT" H 2550 6050 50  0000 C CNN
-F 2 "" H 2550 6250 50  0001 C CNN
+F 2 "Connector_PinHeader_2.54mm:PinHeader_1x03_P2.54mm_Vertical" H 2550 6250 50  0001 C CNN
 F 3 "~" H 2550 6250 50  0001 C CNN
 	1    2550 6250

Commit message: Resolves #41 : [PCB] custom footprint library for passives
Parts:
- L300, L301, L302, L303, L304, L305, L306, L307, L308, L309, L310, L311: footprint (none) -> commons_passives_THT:Passive_THT_EMI_filter_W5.08mm_L7.62mm
- R300, R301, R302, R304, R305, R306, R307, R308, R309, R310, R311: footprint Resistor_THT:R_Axial_DIN0204_L3.6mm_D1.6mm_P7.62mm_Horizontal -> commons_passives_THT:Passive_THT_resistor_W2.54mm_L12.70mm
Changed lines of the file:
@@
 F 0 "R304" V 4900 2000 50  0000 C CNN
 F 1 "1K" V 5100 2000 50  0000 C CNN
-F 2 "Resistor_THT:R_Axial_DIN0204_L3.6mm_D1.6mm_P7.62mm_Horizontal" H 5000 2000 50  0001 C CNN
+F 2 "commons_passives_THT:Passive_THT_resistor_W2.54mm_L12.70mm" H 5000 2000 50  0001 C CNN
 F 3 "~" H 5000 2000 50  0001 C CNN
 	1    5000 2000
@@
 F 0 "R307" V 6150 2500 50  0000 C CNN
 F 1 "220" V 6350 2500 50  0000 C CNN
-F 2 "Resistor_THT:R_Axial_DIN0204_L3.6mm_D1.6mm_P7.62mm_Horizontal" H 6250 2500 50  0001 C CNN
+F 2 "commons_passives_THT:Passive_THT_resistor_W2.54mm_L12.70mm" H 6250 2500 50  0001 C CNN
 F 3 "~" H 6250 2500 50  0001 C CNN
 	1    6250 2500
@@
 F 0 "R305" V 6150 2000 50  0000 C CNN
 F 1 "1K" V 6350 2000 50  0000 C CNN
-F 2 "Resistor_THT:R_Axial_DIN0204_L3.6mm_D1.6mm_P7.62mm_Horizontal" H 6250 2000 50  0001 C CNN
+F 2 "commons_passives_THT:Passive_THT_resistor_W2.54mm_L12.70mm" H 6250 2000 50  0001 C CNN
 F 3 "~" H 6250 2000 50  0001 C CNN
 	1    6250 2000
@@
 F 0 "R306" V 4900 2500 50  0000 C CNN
 F 1 "1K" V 5100 2500 50  0000 C CNN
-F 2 "Resistor_THT:R_Axial_DIN0204_L3.6mm_D1.6mm_P7.62mm_Horizontal" H 5000 2500 50  0001 C CNN
+F 2 "commons_passives_THT:Passive_THT_resistor_W2.54mm_L12.70mm" H 5000 2500 50  0001 C CNN
 F 3 "~" H 5000 2500 50  0001 C CNN
 	1    5000 2500
@@
 F 0 "R301" V 6100 3700 50  0000 C CNN
 F 1 "1K" V 6300 3700 50  0000 C CNN
-F 2 "Resistor_THT:R_Axial_DIN0204_L3.6mm_D1.6mm_P7.62mm_Horizontal" H 6200 3700 50  0001 C CNN
+F 2 "commons_passives_THT:Passive_THT_resistor_W2.54mm_L12.70mm" H 6200 3700 50  0001 C CNN
 F 3 "~" H 6200 3700 50  0001 C CNN
 	1    6200 3700
@@
 F 0 "R300" V 4800 3700 50  0000 C CNN
 F 1 "1K" V 5000 3700 50  0000 C CNN
-F 2 "Resistor_THT:R_Axial_DIN0204_L3.6mm_D1.6mm_P7.62mm_Horizontal" H 4900 3700 50  0001 C CNN
+F 2 "commons_passives_THT:Passive_THT_resistor_W2.54mm_L12.70mm" H 4900 3700 50  0001 C CNN
 F 3 "~" H 4900 3700 50  0001 C CNN
 	1    4900 3700
@@
 F 0 "R308" V 5000 4200 50  0000 C CNN
 F 1 "47" V 5200 4200 50  0000 C CNN
-F 2 "Resistor_THT:R_Axial_DIN0204_L3.6mm_D1.6mm_P7.62mm_Horizontal" H 5100 4200 50  0001 C CNN
+F 2 "commons_passives_THT:Passive_THT_resistor_W2.54mm_L12.70mm" H 5100 4200 50  0001 C CNN
 F 3 "~" H 5100 4200 50  0001 C CNN
 	1    5100 4200
@@
 F 0 "R310" V 5000 4700 50  0000 C CNN
 F 1 "47" V 5200 4700 50  0000 C CNN
-F 2 "Resistor_THT:R_Axial_DIN0204_L3.6mm_D1.6mm_P7.62mm_Horizontal" H 5100 4700 50  0001 C CNN
+F 2 "commons_passives_THT:Passive_THT_resistor_W2.54mm_L12.70mm" H 5100 4700 50  0001 C CNN
 F 3 "~" H 5100 4700 50  0001 C CNN
 	1    5100 4700
@@
 F 0 "R309" V 6300 4200 50  0000 C CNN
 F 1 "47" V 6500 4200 50  0000 C CNN
-F 2 "Resistor_THT:R_Axial_DIN0204_L3.6mm_D1.6mm_P7.62mm_Horizontal" H 6400 4200 50  0001 C CNN
+F 2 "commons_passives_THT:Passive_THT_resistor_W2.54mm_L12.70mm" H 6400 4200 50  0001 C CNN
 F 3 "~" H 6400 4200 50  0001 C CNN
 	1    6400 4200
@@
 F 0 "R311" V 6300 4700 50  0000 C CNN
 F 1 "47" V 6500 4700 50  0000 C CNN
-F 2 "Resistor_THT:R_Axial_DIN0204_L3.6mm_D1.6mm_P7.62mm_Horizontal" H 6400 4700 50  0001 C CNN
+F 2 "commons_passives_THT:Passive_THT_resistor_W2.54mm_L12.70mm" H 6400 4700 50  0001 C CNN
 F 3 "~" H 6400 4700 50  0001 C CNN
 	1    6400 4700
@@
 F 0 "L311" H 3500 5875 50  0000 C CNN
 F 1 "EMI_Filter_LCL" H 3500 5800 50  0000 C CNN
-F 2 "" V 3500 5600 50  0001 C CNN
+F 2 "commons_passives_THT:Passive_THT_EMI_filter_W5.08mm_L7.62mm" V 3500 5600 50  0001 C CNN
 F 3 "http://www.murata.com/~/media/webrenewal/support/library/catalog/products/emc/emifil/c31e.ashx?la=en-gb" V 3500 5600 50  0001 C CNN
 	1    3500 5600
@@
 F 0 "L309" H 3500 6375 50  0000 C CNN
 F 1 "EMI_Filter_LCL" H 3500 6300 50  0000 C CNN
-F 2 "" V 3500 6100 50  0001 C CNN
+F 2 "commons_passives_THT:Passive_THT_EMI_filter_W5.08mm_L7.62mm" V 3500 6100 50  0001 C CNN
 F 3 "http://www.murata.com/~/media/webrenewal/support/library/catalog/products/emc/emifil/c31e.ashx?la=en-gb" V 3500 6100 50  0001 C CNN
 	1    3500 6100
@@
 F 0 "L307" H 3500 7125 50  0000 C CNN
 F 1 "EMI_Filter_LCL" H 3500 7050 50  0000 C CNN
-F 2 "" V 3500 6850 50  0001 C CNN
+F 2 "commons_passives_THT:Passive_THT_EMI_filter_W5.08mm_L7.62mm" V 3500 6850 50  0001 C CNN
 F 3 "http://www.murata.com/~/media/webrenewal/support/library/catalog/products/emc/emifil/c31e.ashx?la=en-gb" V 3500 6850 50  0001 C CNN
 	1    3500 6850
@@
 F 0 "L305" H 3500 7625 50  0000 C CNN
 F 1 "EMI_Filter_LCL" H 3500 7550 50  0000 C CNN
-F 2 "" V 3500 7350 50  0001 C CNN
+F 2 "commons_passives_THT:Passive_THT_EMI_filter_W5.08mm_L7.62mm" V 3500 7350 50  0001 C CNN
 F 3 "http://www.murata.com/~/media/webrenewal/support/library/catalog/products/emc/emifil/c31e.ashx?la=en-gb" V 3500 7350 50  0001 C CNN
 	1    3500 7350
@@
 F 0 "L303" H 3500 8125 50  0000 C CNN
 F 1 "EMI_Filter_LCL" H 3500 8050 50  0000 C CNN
-F 2 "" V 3500 7850 50  0001 C CNN
+F 2 "commons_passives_THT:Passive_THT_EMI_filter_W5.08mm_L7.62mm" V 3500 7850 50  0001 C CNN
 F 3 "http://www.murata.com/~/media/webrenewal/support/library/catalog/products/emc/emifil/c31e.ashx?la=en-gb" V 3500 7850 50  0001 C CNN
 	1    3500 7850
@@
 F 0 "L301" H 3500 8625 50  0000 C CNN
 F 1 "EMI_Filter_LCL" H 3500 8550 50  0000 C CNN
-F 2 "" V 3500 8350 50  0001 C CNN
+F 2 "commons_passives_THT:Passive_THT_EMI_filter_W5.08mm_L7.62mm" V 3500 8350 50  0001 C CNN
 F 3 "http://www.murata.com/~/media/webrenewal/support/library/catalog/products/emc/emifil/c31e.ashx?la=en-gb" V 3500 8350 50  0001 C CNN
 	1    3500 8350
@@
 F 0 "L310" H 4250 6125 50  0000 C CNN
 F 1 "EMI_Filter_LCL" H 4250 6050 50  0000 C CNN
-F 2 "" V 4250 5850 50  0001 C CNN
+F 2 "commons_passives_THT:Passive_THT_EMI_filter_W5.08mm_L7.62mm" V 4250 5850 50  0001 C CNN
 F 3 "http://www.murata.com/~/media/webrenewal/support/library/catalog/products/emc/emifil/c31e.ashx?la=en-gb" V 4250 5850 50  0001 C CNN
 	1    4250 5850
@@
 F 0 "L308" H 4250 6625 50  0000 C CNN
 F 1 "EMI_Filter_LCL" H 4250 6550 50  0000 C CNN
-F 2 "" V 4250 6350 50  0001 C CNN
+F 2 "commons_passives_THT:Passive_THT_EMI_filter_W5.08mm_L7.62mm" V 4250 6350 50  0001 C CNN
 F 3 "http://www.murata.com/~/media/webrenewal/support/library/catalog/products/emc/emifil/c31e.ashx?la=en-gb" V 4250 6350 50  0001 C CNN
 	1    4250 6350
@@
 F 0 "L306" H 4250 7375 50  0000 C CNN
 F 1 "EMI_Filter_LCL" H 4250 7300 50  0000 C CNN
-F 2 "" V 4250 7100 50  0001 C CNN
+F 2 "commons_passives_THT:Passive_THT_EMI_filter_W5.08mm_L7.62mm" V 4250 7100 50  0001 C CNN
 F 3 "http://www.murata.com/~/media/webrenewal/support/library/catalog/products/emc/emifil/c31e.ashx?la=en-gb" V 4250 7100 50  0001 C CNN
 	1    4250 7100
@@
 F 0 "L304" H 4250 7875 50  0000 C CNN
 F 1 "EMI_Filter_LCL" H 4250 7800 50  0000 C CNN
-F 2 "" V 4250 7600 50  0001 C CNN
+F 2 "commons_passives_THT:Passive_THT_EMI_filter_W5.08mm_L7.62mm" V 4250 7600 50  0001 C CNN
 F 3 "http://www.murata.com/~/media/webrenewal/support/library/catalog/products/emc/emifil/c31e.ashx?la=en-gb" V 4250 7600 50  0001 C CNN
 	1    4250 7600
@@
 F 0 "L302" H 4250 8375 50  0000 C CNN
 F 1 "EMI_Filter_LCL" H 4250 8300 50  0000 C CNN
-F 2 "" V 4250 8100 50  0001 C CNN
+F 2 "commons_passives_THT:Passive_THT_EMI_filter_W5.08mm_L7.62mm" V 4250 8100 50  0001 C CNN
 F 3 "http://www.murata.com/~/media/webrenewal/support/library/catalog/products/emc/emifil/c31e.ashx?la=en-gb" V 4250 8100 50  0001 C CNN
 	1    4250 8100
@@
 F 0 "L300" H 4250 8875 50  0000 C CNN
 F 1 "EMI_Filter_LCL" H 4250 8800 50  0000 C CNN
-F 2 "" V 4250 8600 50  0001 C CNN
+F 2 "commons_passives_THT:Passive_THT_EMI_filter_W5.08mm_L7.62mm" V 4250 8600 50  0001 C CNN
 F 3 "http://www.murata.com/~/media/webrenewal/support/library/catalog/products/emc/emifil/c31e.ashx?la=en-gb" V 4250 8600 50  0001 C CNN
 	1    4250 8600
@@
 F 0 "R302" V 1450 6850 50  0000 C CNN
 F 1 "1K" V 1650 6850 50  0000 C CNN
-F 2 "Resistor_THT:R_Axial_DIN0204_L3.6mm_D1.6mm_P7.62mm_Horizontal" H 1550 6850 50  0001 C CNN
+F 2 "commons_passives_THT:Passive_THT_resistor_W2.54mm_L12.70mm" H 1550 6850 50  0001 C CNN
 F 3 "~" H 1550 6850 50  0001 C CNN
 	1    1550 6850

Commit message: [PCB] continue footprint assignation
Parts:
- C304, C305: footprint (none) -> commons_passives_THT:Passive_THT_capacitor_ceramic_radial_W5.08mm_L6.35mm_X11.43mm
Changed lines of the file:
@@
 F 0 "C305" H 1275 2450 50  0000 L CNN
 F 1 "0.1uF" H 1275 2250 50  0000 L CNN
-F 2 "" H 1288 2200 50  0001 C CNN
+F 2 "commons_passives_THT:Passive_THT_capacitor_ceramic_radial_W5.08mm_L6.35mm_X11.43mm" H 1288 2200 50  0001 C CNN
 F 3 "~" H 1250 2350 50  0001 C CNN
 	1    1250 2350
@@
 F 0 "C304" H 1275 4100 50  0000 L CNN
 F 1 "0.1uF" H 1275 3900 50  0000 L CNN
-F 2 "" H 1288 3850 50  0001 C CNN
+F 2 "commons_passives_THT:Passive_THT_capacitor_ceramic_radial_W5.08mm_L6.35mm_X11.43mm" H 1288 3850 50  0001 C CNN
 F 3 "~" H 1250 4000 50  0001 C CNN
 	1    1250 4000

Commit message: [PCB] continue assigning footprints + special libraries of special holes referenced in the measurement schema of the field service manual
Parts:
- J304: footprint (none) -> atari-interconnect:socket-din-14
Changed lines of the file:
@@
 F 0 "J304" H 6500 8700 50  0000 C CNN
 F 1 "DIN 14 — External FDD Port" H 6500 7200 50  0000 C CNN
-F 2 "" H 6500 8000 50  0001 C CNN
+F 2 "atari-interconnect:socket-din-14" H 6500 8000 50  0001 C CNN
 F 3 "~" H 6500 8000 50  0001 C CNN
 	1    6500 8000

Commit message: Resolves #45 : [Atari STE]Use shielded connectors
Parts:
- J304: value DIN 14 — External FDD Port -> DIN-14S — External FDD Port; symbol Connector_Generic:Conn_01x14 -> Connector_Generic_Shielded:Conn_01x14_Shielded
Connections:
- wire segments 161 -> 162
Changed lines of the file:
@@
 $EndComp
 $Comp
-L Connector_Generic:Conn_01x14 J304
+L Connector_Generic_Shielded:Conn_01x14_Shielded J304
 U 1 1 60B2F41A
 P 6500 8000
 F 0 "J304" H 6500 8700 50  0000 C CNN
-F 1 "DIN 14 — External FDD Port" H 6500 7200 50  0000 C CNN
+F 1 "DIN-14S — External FDD Port" H 6500 8800 50  0000 C CNN
 F 2 "atari-interconnect:socket-din-14" H 6500 8000 50  0001 C CNN
 F 3 "~" H 6500 8000 50  0001 C CNN
@@
 Wire Wire Line
 	1200 9050 1550 9050
+Text Label 6500 9100 1    50   ~ 0
+GND
+Wire Wire Line
+	6500 9100 6500 8900
 $EndSCHEMATC
