File: atari-16-32-bits/motherboards/c300780-001/subsheet_400.sch (KiCad schematic (older format))
At the start: 1 part

Commit message: done subsheet 400 : GSTMCU
Parts:
- added C402, C403, C404, C405, C406: 0.1uF, symbol Device:C
- added R421: 1K, symbol Device:R_Small_US
- added R443, R444, R445, R446, R449, R450, R453: 33, symbol Device:R_Small_US
- added R454, R455, R457, R458, R460, R461, R462, R464, R465, R466: 68, symbol Device:R_Small_US
- gave numbers to parts that had none: 1
Connections:
- net GND: now reaches U400.1 (GND)
- net GND: now also U400.109 (GND), U400.128 (GND), U400.37 (GND), U400.73 (GND), U400.74 (TEST), C402.2, C403.2, C404.2, C405.2, C406.2
- net XROM3: now reaches U400.10 (~ROM3~)
- net XJOYRL: now reaches U400.100 (~JOYRL~)
- net XJOYWE: now reaches U400.101 (~JOYWE~)
- net JOYWL: now reaches U400.102 (JOYWL)
- net XBUTTON: now reaches U400.103 (~BUTTON~)
- net XSINT: now reaches U400.105 (~SINT~)
- net MCU_SLOAD: now reaches U400.106 (~SLOAD~)
- net SHIFTER_SREQ: now reaches U400.107 (SREQ)
- net VCC: now reaches U400.108 (VCC)
- net VCC: now also U400.120 (VCC), U400.144 (VCC), U400.30 (~EINT3~), U400.31 (~EINT5~), U400.32 (~EINT7~), U400.36 (VCC), U400.72 (VCC), C402.1, C403.1, C404.1, C405.1, C406.1, R421.1
- net XROM4: now reaches U400.11 (~ROM4~)
- net ma0: now reaches U400.110 (MAD0)
- net ma0: now also R466.2
- net ma1: now reaches U400.111 (MAD1)
- net ma1: now also R465.2
- net ma2: now reaches U400.112 (MAD2)
- net ma2: now also R464.2
- net ma3: now reaches U400.113 (MAD3)
- net ma3: now also R462.2
- net ma4: now reaches U400.114 (MAD4)
- net ma4: now also R461.2
- net ma5: now reaches U400.115 (MAD5)
- net ma5: now also R460.2
- net ma6: now reaches U400.116 (MAD6)
- net ma6: now also R458.2
- net ma7: now reaches U400.117 (MAD7)
- net ma7: now also R457.2
- net ma8: now reaches U400.118 (MAD8)
- net ma8: now also R455.2
- net ma9: now reaches U400.119 (MAD9)
- net ma9: now also R454.2
- net we: now reaches U400.121 (~WE~)
- net we: now also R453.2
- net cas1l: now reaches U400.122 (~CAS1L~)
- net cas1l: now also R450.2
- net cas1h: now reaches U400.123 (~CAS1H~)
- net cas1h: now also R449.2
- net ras1: now reaches U400.124 (~RAS1~)
- net ras1: now also R446.2
- net cas0l: now reaches U400.125 (~CAS0L~)
- net cas0l: now also R445.2
- net cas0h: now reaches U400.126 (~CAS0H~)
- net cas0h: now also R444.2
- net ras0: now reaches U400.127 (~RAS0~)
- net ras0: now also R443.2
- net MCU_WDAT: now reaches U400.129 (~WDAT~)
- net MCU_RDAT: now reaches U400.130 (~RDAT~)
- net MCU_LATCH: now reaches U400.131 (LATCH)
- net RDY: now reaches U400.135 (~RDY~)
- net XFCS: now reaches U400.136 (~FCS~)
- net XPEN: now reaches U400.137 (~PEN~)
- net MCU_DCYC: now reaches U400.138 (~DCYC~)
- net MCU_CMPCS: now reaches U400.139 (~CMPCS~)
- net MCU_BLANK: now reaches U400.140 (~BLANK~)
- net MCU_DE: now reaches U400.141 (DE)
- net VSYNC: now reaches U400.142 (~VSYNC~)
- net HSYNC: now reaches U400.143 (~HSYNC~)
- net XHDINT: now reaches U400.15 (~HDINT~)
- net XHDINT: now also R421.2
- net FDINT: now reaches U400.16 (FDINT)
- net XDISKINT: now reaches U400.17 (~DISKINT~)
- net SNDCS: now reaches U400.18 (SNDCS)
- net SNDIR: now reaches U400.19 (SNDIR)
- net SHIFTER_16MHZ: now reaches U400.2 (CLK16)
- net XBERR: now reaches U400.23 (~BERR~)
- net XVMA: now reaches U400.24 (~VMA~)
- net XVPA: now reaches U400.25 (~VPA~)
- net XBGK: now reaches U400.26 (~BGACK~)
- net XBLTBG: now reaches U400.28 (~BGI~)
- net XBR: now reaches U400.29 (~BR~)
- net CLK8: now reaches U400.3 (CLK8)
- net IPL0: now reaches U400.33 (~IPL0~)
- net IPL1: now reaches U400.34 (~IPL1~)
- net IPL2: now reaches U400.35 (~IPL2~)
- net FC2: now reaches U400.38 (FC2)
- net FC1: now reaches U400.39 (FC1)
- net CLK4: now reaches U400.4 (CLK4)
- net FC0: now reaches U400.40 (FC0)
- net A23: now reaches U400.41 (A23)
- net A22: now reaches U400.42 (A22)
- net A21: now reaches U400.43 (A21)
- net A20: now reaches U400.44 (A20)
- net A19: now reaches U400.45 (A19)
- net A18: now reaches U400.46 (A18)
- net A17: now reaches U400.47 (A17)
- net A16: now reaches U400.48 (A16)
- net N6850: now reaches U400.49 (6850)
- net A15: now reaches U400.50 (A15)
- net A14: now reaches U400.51 (A14)
- net A13: now reaches U400.52 (A13)
- net A12: now reaches U400.53 (A12)
- net A11: now reaches U400.54 (A11)
- net A10: now reaches U400.55 (A10)
- net A9: now reaches U400.56 (A9)
- net A8: now reaches U400.57 (A8)
- net A7: now reaches U400.58 (A7)
- net A6: now reaches U400.59 (A6)
- net KHZ500: now reaches U400.6 (CLK0.5)
- net XBLTINT: now reaches U400.60 (~BINT~)
- net A5: now reaches U400.61 (A5)
- net A4: now reaches U400.62 (A4)
- net A3: now reaches U400.63 (A3)
- net A2: now reaches U400.64 (A2)
- net A1: now reaches U400.65 (A1)
- net XRESET: now reaches U400.66 (~RESET~)
- net XAS: now reaches U400.67 (~AS~)
- net XUDS: now reaches U400.68 (~UDS~)
- net XLDS: now reaches U400.69 (~LDS~)
- net RXW: now reaches U400.70 (R/~W~)
- net XDTACK: now reaches U400.71 (~DTACK~)
- net D15: now reaches U400.75 (D15)
- net D14: now reaches U400.76 (D14)
- net D13: now reaches U400.77 (D13)
- net D12: now reaches U400.78 (D12)
- net D11: now reaches U400.79 (D11)
- net D10: now reaches U400.80 (D10)
- net D9: now reaches U400.81 (D9)
- net D8: now reaches U400.82 (D8)
- net XIACK: now reaches U400.83 (~IACK~)
- net D7: now reaches U400.84 (D7)
- net D6: now reaches U400.85 (D6)
- net D5: now reaches U400.86 (D5)
- net D4: now reaches U400.87 (D4)
- net D3: now reaches U400.88 (D3)
- net D2: now reaches U400.89 (D2)
- net XROM2: now reaches U400.9 (~ROM2~)
- net D1: now reaches U400.90 (D1)
- net D0: now reaches U400.91 (D0)
- net XMFPCS: now reaches U400.92 (~MFPCS~)
- net XMFPINT: now reaches U400.93 (~MFPINT~)
- net XPAD0X: now reaches U400.94 (~PAD0X~)
- net XPAD0Y: now reaches U400.95 (~PAD0Y~)
- net XPAD1X: now reaches U400.96 (~PAD1X~)
- net XPAD1Y: now reaches U400.97 (~PAD1Y~)
- net XPADRST: now reaches U400.98 (~PADRST~)
- net XJOYRH: now reaches U400.99 (~JOYRH~)
- new net MAD0: R466.1
- new net MAD1: R465.1
- new net MAD2: R464.1
- new net MAD3: R462.1
- new net MAD4: R461.1
- new net MAD5: R460.1
- new net MAD6: R458.1
- new net MAD7: R457.1
- new net MAD8: R455.1
- new net MAD9: R454.1
- new net XCAS0H: R444.1
- new net XCAS0L: R445.1
- new net XCAS1H: R449.1
- new net XCAS1L: R450.1
- new net XRAS0: R443.1
- new net XRAS1: R446.1
- new net XWE: R453.1
- no-connect marks 0 -> 12
Other:
- moved on the sheet: U400
