File: atari-16-32-bits/motherboards/c300780-001/subsheet_400.sch (KiCad schematic (older format))
At the start: 24 parts, among them U400 STE_GSTMCU_PHY

Commit message: [PCB] Assign builtins footprint when possible - resistors, ports
Parts:
- R421, R443, R444, R445, R446, R449, R450, R453, R454, R455, R457, R458, R460, R461, R462, R464, R465, R466: footprint (none) -> Resistor_THT:R_Axial_DIN0204_L3.6mm_D1.6mm_P7.62mm_Horizontal
Changed lines of the file:
@@
 F 0 "R443" V 2850 8250 50  0000 C CNN
 F 1 "33" V 3050 8250 50  0000 C CNN
-F 2 "" H 2950 8250 50  0001 C CNN
+F 2 "Resistor_THT:R_Axial_DIN0204_L3.6mm_D1.6mm_P7.62mm_Horizontal" H 2950 8250 50  0001 C CNN
 F 3 "~" H 2950 8250 50  0001 C CNN
 	1    2950 8250
@@
 F 0 "R454" V 5200 8250 50  0000 C CNN
 F 1 "68" V 5400 8250 50  0000 C CNN
-F 2 "" H 5300 8250 50  0001 C CNN
+F 2 "Resistor_THT:R_Axial_DIN0204_L3.6mm_D1.6mm_P7.62mm_Horizontal" H 5300 8250 50  0001 C CNN
 F 3 "~" H 5300 8250 50  0001 C CNN
 	1    5300 8250
@@
 F 0 "R444" V 2850 8750 50  0000 C CNN
 F 1 "33" V 3050 8750 50  0000 C CNN
-F 2 "" H 2950 8750 50  0001 C CNN
+F 2 "Resistor_THT:R_Axial_DIN0204_L3.6mm_D1.6mm_P7.62mm_Horizontal" H 2950 8750 50  0001 C CNN
 F 3 "~" H 2950 8750 50  0001 C CNN
 	1    2950 8750
@@
 F 0 "R445" V 2850 9250 50  0000 C CNN
 F 1 "33" V 3050 9250 50  0000 C CNN
-F 2 "" H 2950 9250 50  0001 C CNN
+F 2 "Resistor_THT:R_Axial_DIN0204_L3.6mm_D1.6mm_P7.62mm_Horizontal" H 2950 9250 50  0001 C CNN
 F 3 "~" H 2950 9250 50  0001 C CNN
 	1    2950 9250
@@
 F 0 "R446" V 3850 8250 50  0000 C CNN
 F 1 "33" V 4050 8250 50  0000 C CNN
-F 2 "" H 3950 8250 50  0001 C CNN
+F 2 "Resistor_THT:R_Axial_DIN0204_L3.6mm_D1.6mm_P7.62mm_Horizontal" H 3950 8250 50  0001 C CNN
 F 3 "~" H 3950 8250 50  0001 C CNN
 	1    3950 8250
@@
 F 0 "R449" V 3850 8750 50  0000 C CNN
 F 1 "33" V 4050 8750 50  0000 C CNN
-F 2 "" H 3950 8750 50  0001 C CNN
+F 2 "Resistor_THT:R_Axial_DIN0204_L3.6mm_D1.6mm_P7.62mm_Horizontal" H 3950 8750 50  0001 C CNN
 F 3 "~" H 3950 8750 50  0001 C CNN
 	1    3950 8750
@@
 F 0 "R450" V 3850 9250 50  0000 C CNN
 F 1 "33" V 4050 9250 50  0000 C CNN
-F 2 "" H 3950 9250 50  0001 C CNN
+F 2 "Resistor_THT:R_Axial_DIN0204_L3.6mm_D1.6mm_P7.62mm_Horizontal" H 3950 9250 50  0001 C CNN
 F 3 "~" H 3950 9250 50  0001 C CNN
 	1    3950 9250
@@
 F 0 "R453" V 2850 9750 50  0000 C CNN
 F 1 "33" V 3050 9750 50  0000 C CNN
-F 2 "" H 2950 9750 50  0001 C CNN
+F 2 "Resistor_THT:R_Axial_DIN0204_L3.6mm_D1.6mm_P7.62mm_Horizontal" H 2950 9750 50  0001 C CNN
 F 3 "~" H 2950 9750 50  0001 C CNN
 	1    2950 9750
@@
 F 0 "R455" V 5200 8750 50  0000 C CNN
 F 1 "68" V 5400 8750 50  0000 C CNN
-F 2 "" H 5300 8750 50  0001 C CNN
+F 2 "Resistor_THT:R_Axial_DIN0204_L3.6mm_D1.6mm_P7.62mm_Horizontal" H 5300 8750 50  0001 C CNN
 F 3 "~" H 5300 8750 50  0001 C CNN
 	1    5300 8750
@@
 F 0 "R457" V 5200 9250 50  0000 C CNN
 F 1 "68" V 5400 9250 50  0000 C CNN
-F 2 "" H 5300 9250 50  0001 C CNN
+F 2 "Resistor_THT:R_Axial_DIN0204_L3.6mm_D1.6mm_P7.62mm_Horizontal" H 5300 9250 50  0001 C CNN
 F 3 "~" H 5300 9250 50  0001 C CNN
 	1    5300 9250
@@
 F 0 "R458" V 5200 9750 50  0000 C CNN
 F 1 "68" V 5400 9750 50  0000 C CNN
-F 2 "" H 5300 9750 50  0001 C CNN
+F 2 "Resistor_THT:R_Axial_DIN0204_L3.6mm_D1.6mm_P7.62mm_Horizontal" H 5300 9750 50  0001 C CNN
 F 3 "~" H 5300 9750 50  0001 C CNN
 	1    5300 9750
@@
 F 0 "R460" V 6000 8250 50  0000 C CNN
 F 1 "68" V 6200 8250 50  0000 C CNN
-F 2 "" H 6100 8250 50  0001 C CNN
+F 2 "Resistor_THT:R_Axial_DIN0204_L3.6mm_D1.6mm_P7.62mm_Horizontal" H 6100 8250 50  0001 C CNN
 F 3 "~" H 6100 8250 50  0001 C CNN
 	1    6100 8250
@@
 F 0 "R461" V 6000 8750 50  0000 C CNN
 F 1 "68" V 6200 8750 50  0000 C CNN
-F 2 "" H 6100 8750 50  0001 C CNN
+F 2 "Resistor_THT:R_Axial_DIN0204_L3.6mm_D1.6mm_P7.62mm_Horizontal" H 6100 8750 50  0001 C CNN
 F 3 "~" H 6100 8750 50  0001 C CNN
 	1    6100 8750
@@
 F 0 "R462" V 6000 9250 50  0000 C CNN
 F 1 "68" V 6200 9250 50  0000 C CNN
-F 2 "" H 6100 9250 50  0001 C CNN
+F 2 "Resistor_THT:R_Axial_DIN0204_L3.6mm_D1.6mm_P7.62mm_Horizontal" H 6100 9250 50  0001 C CNN
 F 3 "~" H 6100 9250 50  0001 C CNN
 	1    6100 9250
@@
 F 0 "R464" V 6000 9750 50  0000 C CNN
 F 1 "68" V 6200 9750 50  0000 C CNN
-F 2 "" H 6100 9750 50  0001 C CNN
+F 2 "Resistor_THT:R_Axial_DIN0204_L3.6mm_D1.6mm_P7.62mm_Horizontal" H 6100 9750 50  0001 C CNN
 F 3 "~" H 6100 9750 50  0001 C CNN
 	1    6100 9750
@@
 F 0 "R465" V 6800 9250 50  0000 C CNN
 F 1 "68" V 7000 9250 50  0000 C CNN
-F 2 "" H 6900 9250 50  0001 C CNN
+F 2 "Resistor_THT:R_Axial_DIN0204_L3.6mm_D1.6mm_P7.62mm_Horizontal" H 6900 9250 50  0001 C CNN
 F 3 "~" H 6900 9250 50  0001 C CNN
 	1    6900 9250
@@
 F 0 "R466" V 6800 9750 50  0000 C CNN
 F 1 "68" V 7000 9750 50  0000 C CNN
-F 2 "" H 6900 9750 50  0001 C CNN
+F 2 "Resistor_THT:R_Axial_DIN0204_L3.6mm_D1.6mm_P7.62mm_Horizontal" H 6900 9750 50  0001 C CNN
 F 3 "~" H 6900 9750 50  0001 C CNN
 	1    6900 9750
@@
 F 0 "R421" V 6800 7500 50  0000 C CNN
 F 1 "1K" V 7000 7500 50  0000 C CNN
-F 2 "" H 6900 7500 50  0001 C CNN
+F 2 "Resistor_THT:R_Axial_DIN0204_L3.6mm_D1.6mm_P7.62mm_Horizontal" H 6900 7500 50  0001 C CNN
 F 3 "~" H 6900 7500 50  0001 C CNN
 	1    6900 7500

Commit message: Resolves #41 : [PCB] custom footprint library for passives
Parts:
- R421, R443, R444, R445, R446, R449, R450, R453, R454, R455, R457, R458, R460, R461, R462, R464, R465, R466: footprint Resistor_THT:R_Axial_DIN0204_L3.6mm_D1.6mm_P7.62mm_Horizontal -> commons_passives_THT:Passive_THT_resistor_W2.54mm_L12.70mm
Changed lines of the file:
@@
 F 0 "R443" V 2850 8250 50  0000 C CNN
 F 1 "33" V 3050 8250 50  0000 C CNN
-F 2 "Resistor_THT:R_Axial_DIN0204_L3.6mm_D1.6mm_P7.62mm_Horizontal" H 2950 8250 50  0001 C CNN
+F 2 "commons_passives_THT:Passive_THT_resistor_W2.54mm_L12.70mm" H 2950 8250 50  0001 C CNN
 F 3 "~" H 2950 8250 50  0001 C CNN
 	1    2950 8250
@@
 F 0 "R454" V 5200 8250 50  0000 C CNN
 F 1 "68" V 5400 8250 50  0000 C CNN
-F 2 "Resistor_THT:R_Axial_DIN0204_L3.6mm_D1.6mm_P7.62mm_Horizontal" H 5300 8250 50  0001 C CNN
+F 2 "commons_passives_THT:Passive_THT_resistor_W2.54mm_L12.70mm" H 5300 8250 50  0001 C CNN
 F 3 "~" H 5300 8250 50  0001 C CNN
 	1    5300 8250
@@
 F 0 "R444" V 2850 8750 50  0000 C CNN
 F 1 "33" V 3050 8750 50  0000 C CNN
-F 2 "Resistor_THT:R_Axial_DIN0204_L3.6mm_D1.6mm_P7.62mm_Horizontal" H 2950 8750 50  0001 C CNN
+F 2 "commons_passives_THT:Passive_THT_resistor_W2.54mm_L12.70mm" H 2950 8750 50  0001 C CNN
 F 3 "~" H 2950 8750 50  0001 C CNN
 	1    2950 8750
@@
 F 0 "R445" V 2850 9250 50  0000 C CNN
 F 1 "33" V 3050 9250 50  0000 C CNN
-F 2 "Resistor_THT:R_Axial_DIN0204_L3.6mm_D1.6mm_P7.62mm_Horizontal" H 2950 9250 50  0001 C CNN
+F 2 "commons_passives_THT:Passive_THT_resistor_W2.54mm_L12.70mm" H 2950 9250 50  0001 C CNN
 F 3 "~" H 2950 9250 50  0001 C CNN
 	1    2950 9250
@@
 F 0 "R446" V 3850 8250 50  0000 C CNN
 F 1 "33" V 4050 8250 50  0000 C CNN
-F 2 "Resistor_THT:R_Axial_DIN0204_L3.6mm_D1.6mm_P7.62mm_Horizontal" H 3950 8250 50  0001 C CNN
+F 2 "commons_passives_THT:Passive_THT_resistor_W2.54mm_L12.70mm" H 3950 8250 50  0001 C CNN
 F 3 "~" H 3950 8250 50  0001 C CNN
 	1    3950 8250
@@
 F 0 "R449" V 3850 8750 50  0000 C CNN
 F 1 "33" V 4050 8750 50  0000 C CNN
-F 2 "Resistor_THT:R_Axial_DIN0204_L3.6mm_D1.6mm_P7.62mm_Horizontal" H 3950 8750 50  0001 C CNN
+F 2 "commons_passives_THT:Passive_THT_resistor_W2.54mm_L12.70mm" H 3950 8750 50  0001 C CNN
 F 3 "~" H 3950 8750 50  0001 C CNN
 	1    3950 8750
@@
 F 0 "R450" V 3850 9250 50  0000 C CNN
 F 1 "33" V 4050 9250 50  0000 C CNN
-F 2 "Resistor_THT:R_Axial_DIN0204_L3.6mm_D1.6mm_P7.62mm_Horizontal" H 3950 9250 50  0001 C CNN
+F 2 "commons_passives_THT:Passive_THT_resistor_W2.54mm_L12.70mm" H 3950 9250 50  0001 C CNN
 F 3 "~" H 3950 9250 50  0001 C CNN
 	1    3950 9250
@@
 F 0 "R453" V 2850 9750 50  0000 C CNN
 F 1 "33" V 3050 9750 50  0000 C CNN
-F 2 "Resistor_THT:R_Axial_DIN0204_L3.6mm_D1.6mm_P7.62mm_Horizontal" H 2950 9750 50  0001 C CNN
+F 2 "commons_passives_THT:Passive_THT_resistor_W2.54mm_L12.70mm" H 2950 9750 50  0001 C CNN
 F 3 "~" H 2950 9750 50  0001 C CNN
 	1    2950 9750
@@
 F 0 "R455" V 5200 8750 50  0000 C CNN
 F 1 "68" V 5400 8750 50  0000 C CNN
-F 2 "Resistor_THT:R_Axial_DIN0204_L3.6mm_D1.6mm_P7.62mm_Horizontal" H 5300 8750 50  0001 C CNN
+F 2 "commons_passives_THT:Passive_THT_resistor_W2.54mm_L12.70mm" H 5300 8750 50  0001 C CNN
 F 3 "~" H 5300 8750 50  0001 C CNN
 	1    5300 8750
@@
 F 0 "R457" V 5200 9250 50  0000 C CNN
 F 1 "68" V 5400 9250 50  0000 C CNN
-F 2 "Resistor_THT:R_Axial_DIN0204_L3.6mm_D1.6mm_P7.62mm_Horizontal" H 5300 9250 50  0001 C CNN
+F 2 "commons_passives_THT:Passive_THT_resistor_W2.54mm_L12.70mm" H 5300 9250 50  0001 C CNN
 F 3 "~" H 5300 9250 50  0001 C CNN
 	1    5300 9250
@@
 F 0 "R458" V 5200 9750 50  0000 C CNN
 F 1 "68" V 5400 9750 50  0000 C CNN
-F 2 "Resistor_THT:R_Axial_DIN0204_L3.6mm_D1.6mm_P7.62mm_Horizontal" H 5300 9750 50  0001 C CNN
+F 2 "commons_passives_THT:Passive_THT_resistor_W2.54mm_L12.70mm" H 5300 9750 50  0001 C CNN
 F 3 "~" H 5300 9750 50  0001 C CNN
 	1    5300 9750
@@
 F 0 "R460" V 6000 8250 50  0000 C CNN
 F 1 "68" V 6200 8250 50  0000 C CNN
-F 2 "Resistor_THT:R_Axial_DIN0204_L3.6mm_D1.6mm_P7.62mm_Horizontal" H 6100 8250 50  0001 C CNN
+F 2 "commons_passives_THT:Passive_THT_resistor_W2.54mm_L12.70mm" H 6100 8250 50  0001 C CNN
 F 3 "~" H 6100 8250 50  0001 C CNN
 	1    6100 8250
@@
 F 0 "R461" V 6000 8750 50  0000 C CNN
 F 1 "68" V 6200 8750 50  0000 C CNN
-F 2 "Resistor_THT:R_Axial_DIN0204_L3.6mm_D1.6mm_P7.62mm_Horizontal" H 6100 8750 50  0001 C CNN
+F 2 "commons_passives_THT:Passive_THT_resistor_W2.54mm_L12.70mm" H 6100 8750 50  0001 C CNN
 F 3 "~" H 6100 8750 50  0001 C CNN
 	1    6100 8750
@@
 F 0 "R462" V 6000 9250 50  0000 C CNN
 F 1 "68" V 6200 9250 50  0000 C CNN
-F 2 "Resistor_THT:R_Axial_DIN0204_L3.6mm_D1.6mm_P7.62mm_Horizontal" H 6100 9250 50  0001 C CNN
+F 2 "commons_passives_THT:Passive_THT_resistor_W2.54mm_L12.70mm" H 6100 9250 50  0001 C CNN
 F 3 "~" H 6100 9250 50  0001 C CNN
 	1    6100 9250
@@
 F 0 "R464" V 6000 9750 50  0000 C CNN
 F 1 "68" V 6200 9750 50  0000 C CNN
-F 2 "Resistor_THT:R_Axial_DIN0204_L3.6mm_D1.6mm_P7.62mm_Horizontal" H 6100 9750 50  0001 C CNN
+F 2 "commons_passives_THT:Passive_THT_resistor_W2.54mm_L12.70mm" H 6100 9750 50  0001 C CNN
 F 3 "~" H 6100 9750 50  0001 C CNN
 	1    6100 9750
@@
 F 0 "R465" V 6800 9250 50  0000 C CNN
 F 1 "68" V 7000 9250 50  0000 C CNN
-F 2 "Resistor_THT:R_Axial_DIN0204_L3.6mm_D1.6mm_P7.62mm_Horizontal" H 6900 9250 50  0001 C CNN
+F 2 "commons_passives_THT:Passive_THT_resistor_W2.54mm_L12.70mm" H 6900 9250 50  0001 C CNN
 F 3 "~" H 6900 9250 50  0001 C CNN
 	1    6900 9250
@@
 F 0 "R466" V 6800 9750 50  0000 C CNN
 F 1 "68" V 7000 9750 50  0000 C CNN
-F 2 "Resistor_THT:R_Axial_DIN0204_L3.6mm_D1.6mm_P7.62mm_Horizontal" H 6900 9750 50  0001 C CNN
+F 2 "commons_passives_THT:Passive_THT_resistor_W2.54mm_L12.70mm" H 6900 9750 50  0001 C CNN
 F 3 "~" H 6900 9750 50  0001 C CNN
 	1    6900 9750
@@
 F 0 "R421" V 6800 7500 50  0000 C CNN
 F 1 "1K" V 7000 7500 50  0000 C CNN
-F 2 "Resistor_THT:R_Axial_DIN0204_L3.6mm_D1.6mm_P7.62mm_Horizontal" H 6900 7500 50  0001 C CNN
+F 2 "commons_passives_THT:Passive_THT_resistor_W2.54mm_L12.70mm" H 6900 7500 50  0001 C CNN
 F 3 "~" H 6900 7500 50  0001 C CNN
 	1    6900 7500

Commit message: [PCB] continue footprint assignation
Parts:
- C402, C403, C404, C405, C406: footprint (none) -> commons_passives_THT:Passive_THT_capacitor_ceramic_radial_W5.08mm_L6.35mm_X11.43mm
Changed lines of the file:
@@
 F 0 "C402" H 1125 7350 50  0000 L CNN
 F 1 "0.1uF" H 1125 7150 50  0000 L CNN
-F 2 "" H 1138 7100 50  0001 C CNN
+F 2 "commons_passives_THT:Passive_THT_capacitor_ceramic_radial_W5.08mm_L6.35mm_X11.43mm" H 1138 7100 50  0001 C CNN
 F 3 "~" H 1100 7250 50  0001 C CNN
 	1    1100 7250
@@
 F 0 "C403" H 1625 7350 50  0000 L CNN
 F 1 "0.1uF" H 1625 7150 50  0000 L CNN
-F 2 "" H 1638 7100 50  0001 C CNN
+F 2 "commons_passives_THT:Passive_THT_capacitor_ceramic_radial_W5.08mm_L6.35mm_X11.43mm" H 1638 7100 50  0001 C CNN
 F 3 "~" H 1600 7250 50  0001 C CNN
 	1    1600 7250
@@
 F 0 "C404" H 1125 8350 50  0000 L CNN
 F 1 "0.1uF" H 1125 8150 50  0000 L CNN
-F 2 "" H 1138 8100 50  0001 C CNN
+F 2 "commons_passives_THT:Passive_THT_capacitor_ceramic_radial_W5.08mm_L6.35mm_X11.43mm" H 1138 8100 50  0001 C CNN
 F 3 "~" H 1100 8250 50  0001 C CNN
 	1    1100 8250
@@
 F 0 "C405" H 1625 8350 50  0000 L CNN
 F 1 "0.1uF" H 1625 8150 50  0000 L CNN
-F 2 "" H 1638 8100 50  0001 C CNN
+F 2 "commons_passives_THT:Passive_THT_capacitor_ceramic_radial_W5.08mm_L6.35mm_X11.43mm" H 1638 8100 50  0001 C CNN
 F 3 "~" H 1600 8250 50  0001 C CNN
 	1    1600 8250
@@
 F 0 "C406" H 1125 9350 50  0000 L CNN
 F 1 "0.1uF" H 1125 9150 50  0000 L CNN
-F 2 "" H 1138 9100 50  0001 C CNN
+F 2 "commons_passives_THT:Passive_THT_capacitor_ceramic_radial_W5.08mm_L6.35mm_X11.43mm" H 1138 9100 50  0001 C CNN
 F 3 "~" H 1100 9250 50  0001 C CNN
 	1    1100 9250
