File: atari-16-32-bits/motherboards/c300780-001/subsheet_402.sch (KiCad schematic (older format))
At the start: 39 parts, among them J400 DIN 13 — Video Port, Q400 2N3904, Q401 2N3904, Q402 2N3904, Q403 2N3904, U405 74S257_PHY

Commit message: completed subsheet 402
Parts:
- removed R?: 4K7, symbol Device:R_Small_US
- added R472: 4K7, symbol Device:R_Small_US
- gave numbers to parts that had none: 28
Connections:
- net labels added: B, G
Other:
- note added: "Genlock is active low. \n -> When asserted (low), vid4 is the external video clock of the genlock,\n and sent as the main clock MC to the shifter ; MONOMON is forced to high (color display).\n -> When negated (high), the 32MHz clock is sent as the main clock MC to the shifter ; vid4 is \n the detection of monochrome displays and sent as MONOMON."
- note removed: "Genlock is active low. \n -> When asserted (low), vid4 is the external video clock of the genlock,\n and sent as main clock to the shifter ; Monomon is forced to high (color display).\n -> When negated (high), the 32MHz clock is sent as main clock to the shifter ; vid4 is \n the detection of monochrome displays."
