File: atari-16-32-bits/motherboards/c300780-001/subsheet_402.sch (KiCad schematic (older format))
At the start: 39 parts, among them J400 DIN 13 — Video Port, Q400 2N3904, Q401 2N3904, Q402 2N3904, Q403 2N3904, U405 74S257_PHY

Commit message: [PCB] Assign builtins footprint when possible - resistors, ports
Parts:
- R406, R407, R408, R409, R410, R413, R420, R423, R425, R427, R429, R431, R432, R433, R434, R435, R436, R437, R438, R440, R441, R472: footprint (none) -> Resistor_THT:R_Axial_DIN0204_L3.6mm_D1.6mm_P7.62mm_Horizontal
Changed lines of the file:
@@
 F 0 "R406" V 3650 3400 50  0000 C CNN
 F 1 "1K" V 3850 3400 50  0000 C CNN
-F 2 "" H 3750 3400 50  0001 C CNN
+F 2 "Resistor_THT:R_Axial_DIN0204_L3.6mm_D1.6mm_P7.62mm_Horizontal" H 3750 3400 50  0001 C CNN
 F 3 "~" H 3750 3400 50  0001 C CNN
 	1    3750 3400
@@
 F 0 "R407" V 4150 4000 50  0000 C CNN
 F 1 "75" V 4350 4000 50  0000 C CNN
-F 2 "" H 4250 4000 50  0001 C CNN
+F 2 "Resistor_THT:R_Axial_DIN0204_L3.6mm_D1.6mm_P7.62mm_Horizontal" H 4250 4000 50  0001 C CNN
 F 3 "~" H 4250 4000 50  0001 C CNN
 	1    4250 4000
@@
 F 0 "R409" H 4030 4320 50  0000 L CNN
 F 1 "75" H 4030 4260 50  0000 L CNN
-F 2 "" H 4000 4300 50  0001 C CNN
+F 2 "Resistor_THT:R_Axial_DIN0204_L3.6mm_D1.6mm_P7.62mm_Horizontal" H 4000 4300 50  0001 C CNN
 F 3 "~" H 4000 4300 50  0001 C CNN
 	1    4000 4300
@@
 F 0 "R410" H 4030 4820 50  0000 L CNN
 F 1 "75" H 4030 4760 50  0000 L CNN
-F 2 "" H 4000 4800 50  0001 C CNN
+F 2 "Resistor_THT:R_Axial_DIN0204_L3.6mm_D1.6mm_P7.62mm_Horizontal" H 4000 4800 50  0001 C CNN
 F 3 "~" H 4000 4800 50  0001 C CNN
 	1    4000 4800
@@
 F 0 "R408" H 3530 3970 50  0000 L CNN
 F 1 "2K" H 3530 3910 50  0000 L CNN
-F 2 "" H 3500 3950 50  0001 C CNN
+F 2 "Resistor_THT:R_Axial_DIN0204_L3.6mm_D1.6mm_P7.62mm_Horizontal" H 3500 3950 50  0001 C CNN
 F 3 "~" H 3500 3950 50  0001 C CNN
 	1    3500 3950
@@
 F 0 "R413" V 6150 3400 50  0000 C CNN
 F 1 "1K" V 6350 3400 50  0000 C CNN
-F 2 "" H 6250 3400 50  0001 C CNN
+F 2 "Resistor_THT:R_Axial_DIN0204_L3.6mm_D1.6mm_P7.62mm_Horizontal" H 6250 3400 50  0001 C CNN
 F 3 "~" H 6250 3400 50  0001 C CNN
 	1    6250 3400
@@
 F 0 "R423" H 6030 3970 50  0000 L CNN
 F 1 "2K" H 6030 3910 50  0000 L CNN
-F 2 "" H 6000 3950 50  0001 C CNN
+F 2 "Resistor_THT:R_Axial_DIN0204_L3.6mm_D1.6mm_P7.62mm_Horizontal" H 6000 3950 50  0001 C CNN
 F 3 "~" H 6000 3950 50  0001 C CNN
 	1    6000 3950
@@
 F 0 "R420" V 6650 4000 50  0000 C CNN
 F 1 "75" V 6850 4000 50  0000 C CNN
-F 2 "" H 6750 4000 50  0001 C CNN
+F 2 "Resistor_THT:R_Axial_DIN0204_L3.6mm_D1.6mm_P7.62mm_Horizontal" H 6750 4000 50  0001 C CNN
 F 3 "~" H 6750 4000 50  0001 C CNN
 	1    6750 4000
@@
 F 0 "R425" H 6530 4320 50  0000 L CNN
 F 1 "75" H 6530 4260 50  0000 L CNN
-F 2 "" H 6500 4300 50  0001 C CNN
+F 2 "Resistor_THT:R_Axial_DIN0204_L3.6mm_D1.6mm_P7.62mm_Horizontal" H 6500 4300 50  0001 C CNN
 F 3 "~" H 6500 4300 50  0001 C CNN
 	1    6500 4300
@@
 F 0 "R427" H 6530 4820 50  0000 L CNN
 F 1 "75" H 6530 4760 50  0000 L CNN
-F 2 "" H 6500 4800 50  0001 C CNN
+F 2 "Resistor_THT:R_Axial_DIN0204_L3.6mm_D1.6mm_P7.62mm_Horizontal" H 6500 4800 50  0001 C CNN
 F 3 "~" H 6500 4800 50  0001 C CNN
 	1    6500 4800
@@
 F 0 "R429" V 2400 5400 50  0000 C CNN
 F 1 "1K" V 2600 5400 50  0000 C CNN
-F 2 "" H 2500 5400 50  0001 C CNN
+F 2 "Resistor_THT:R_Axial_DIN0204_L3.6mm_D1.6mm_P7.62mm_Horizontal" H 2500 5400 50  0001 C CNN
 F 3 "~" H 2500 5400 50  0001 C CNN
 	1    2500 5400
@@
 F 0 "R433" H 2280 5970 50  0000 L CNN
 F 1 "2K" H 2280 5910 50  0000 L CNN
-F 2 "" H 2250 5950 50  0001 C CNN
+F 2 "Resistor_THT:R_Axial_DIN0204_L3.6mm_D1.6mm_P7.62mm_Horizontal" H 2250 5950 50  0001 C CNN
 F 3 "~" H 2250 5950 50  0001 C CNN
 	1    2250 5950
@@
 F 0 "R432" V 2900 6000 50  0000 C CNN
 F 1 "75" V 3100 6000 50  0000 C CNN
-F 2 "" H 3000 6000 50  0001 C CNN
+F 2 "Resistor_THT:R_Axial_DIN0204_L3.6mm_D1.6mm_P7.62mm_Horizontal" H 3000 6000 50  0001 C CNN
 F 3 "~" H 3000 6000 50  0001 C CNN
 	1    3000 6000
@@
 F 0 "R434" H 2780 6320 50  0000 L CNN
 F 1 "75" H 2780 6260 50  0000 L CNN
-F 2 "" H 2750 6300 50  0001 C CNN
+F 2 "Resistor_THT:R_Axial_DIN0204_L3.6mm_D1.6mm_P7.62mm_Horizontal" H 2750 6300 50  0001 C CNN
 F 3 "~" H 2750 6300 50  0001 C CNN
 	1    2750 6300
@@
 F 0 "R436" H 2780 6820 50  0000 L CNN
 F 1 "75" H 2780 6760 50  0000 L CNN
-F 2 "" H 2750 6800 50  0001 C CNN
+F 2 "Resistor_THT:R_Axial_DIN0204_L3.6mm_D1.6mm_P7.62mm_Horizontal" H 2750 6800 50  0001 C CNN
 F 3 "~" H 2750 6800 50  0001 C CNN
 	1    2750 6800
@@
 F 0 "R440" H 4780 5970 50  0000 L CNN
 F 1 "1K" H 4780 5910 50  0000 L CNN
-F 2 "" H 4750 5950 50  0001 C CNN
+F 2 "Resistor_THT:R_Axial_DIN0204_L3.6mm_D1.6mm_P7.62mm_Horizontal" H 4750 5950 50  0001 C CNN
 F 3 "~" H 4750 5950 50  0001 C CNN
 	1    4750 5950
@@
 F 0 "R438" V 5400 6000 50  0000 C CNN
 F 1 "27" V 5600 6000 50  0000 C CNN
-F 2 "" H 5500 6000 50  0001 C CNN
+F 2 "Resistor_THT:R_Axial_DIN0204_L3.6mm_D1.6mm_P7.62mm_Horizontal" H 5500 6000 50  0001 C CNN
 F 3 "~" H 5500 6000 50  0001 C CNN
 	1    5500 6000
@@
 F 0 "R441" H 5280 6320 50  0000 L CNN
 F 1 "100" H 5280 6260 50  0000 L CNN
-F 2 "" H 5250 6300 50  0001 C CNN
+F 2 "Resistor_THT:R_Axial_DIN0204_L3.6mm_D1.6mm_P7.62mm_Horizontal" H 5250 6300 50  0001 C CNN
 F 3 "~" H 5250 6300 50  0001 C CNN
 	1    5250 6300
@@
 F 0 "R431" V 3450 2100 50  0000 C CNN
 F 1 "1K2" V 3650 2100 50  0000 C CNN
-F 2 "" H 3550 2100 50  0001 C CNN
+F 2 "Resistor_THT:R_Axial_DIN0204_L3.6mm_D1.6mm_P7.62mm_Horizontal" H 3550 2100 50  0001 C CNN
 F 3 "~" H 3550 2100 50  0001 C CNN
 	1    3550 2100
@@
 F 0 "R437" V 1450 2600 50  0000 C CNN
 F 1 "33" V 1650 2600 50  0000 C CNN
-F 2 "" H 1550 2600 50  0001 C CNN
+F 2 "Resistor_THT:R_Axial_DIN0204_L3.6mm_D1.6mm_P7.62mm_Horizontal" H 1550 2600 50  0001 C CNN
 F 3 "~" H 1550 2600 50  0001 C CNN
 	1    1550 2600
@@
 F 0 "R435" V 3450 2600 50  0000 C CNN
 F 1 "33" V 3650 2600 50  0000 C CNN
-F 2 "" H 3550 2600 50  0001 C CNN
+F 2 "Resistor_THT:R_Axial_DIN0204_L3.6mm_D1.6mm_P7.62mm_Horizontal" H 3550 2600 50  0001 C CNN
 F 3 "~" H 3550 2600 50  0001 C CNN
 	1    3550 2600
@@
 F 0 "R472" H 3680 1320 50  0000 L CNN
 F 1 "4K7" H 3680 1260 50  0000 L CNN
-F 2 "" H 3650 1300 50  0001 C CNN
+F 2 "Resistor_THT:R_Axial_DIN0204_L3.6mm_D1.6mm_P7.62mm_Horizontal" H 3650 1300 50  0001 C CNN
 F 3 "~" H 3650 1300 50  0001 C CNN
 	1    3650 1300

Commit message: [PCB] continuing footprint assignement
Parts:
- Q400, Q401, Q402, Q403: footprint Package_TO_SOT_THT:TO-92_Inline -> Package_TO_SOT_THT:TO-92_Inline_Wide
Changed lines of the file:
@@
 F 0 "Q400" H 4100 3775 50  0000 L CNN
 F 1 "2N3904" H 4100 3700 50  0000 L CNN
-F 2 "Package_TO_SOT_THT:TO-92_Inline" H 4100 3625 50  0001 L CIN
+F 2 "Package_TO_SOT_THT:TO-92_Inline_Wide" H 4100 3625 50  0001 L CIN
 F 3 "https://www.onsemi.com/pub/Collateral/2N3903-D.PDF" H 3900 3700 50  0001 L CNN
 	1    3900 3700
@@
 F 0 "Q402" H 2850 5775 50  0000 L CNN
 F 1 "2N3904" H 2850 5700 50  0000 L CNN
-F 2 "Package_TO_SOT_THT:TO-92_Inline" H 2850 5625 50  0001 L CIN
+F 2 "Package_TO_SOT_THT:TO-92_Inline_Wide" H 2850 5625 50  0001 L CIN
 F 3 "https://www.onsemi.com/pub/Collateral/2N3903-D.PDF" H 2650 5700 50  0001 L CNN
 	1    2650 5700
@@
 F 0 "Q401" H 6600 3775 50  0000 L CNN
 F 1 "2N3904" H 6600 3700 50  0000 L CNN
-F 2 "Package_TO_SOT_THT:TO-92_Inline" H 6600 3625 50  0001 L CIN
+F 2 "Package_TO_SOT_THT:TO-92_Inline_Wide" H 6600 3625 50  0001 L CIN
 F 3 "https://www.onsemi.com/pub/Collateral/2N3903-D.PDF" H 6400 3700 50  0001 L CNN
 	1    6400 3700
@@
 F 0 "Q403" H 5350 5775 50  0000 L CNN
 F 1 "2N3904" H 5350 5700 50  0000 L CNN
-F 2 "Package_TO_SOT_THT:TO-92_Inline" H 5350 5625 50  0001 L CIN
+F 2 "Package_TO_SOT_THT:TO-92_Inline_Wide" H 5350 5625 50  0001 L CIN
 F 3 "https://www.onsemi.com/pub/Collateral/2N3903-D.PDF" H 5150 5700 50  0001 L CNN
 	1    5150 5700

Commit message: Resolves #41 : [PCB] custom footprint library for passives
Parts:
- L401, L402: footprint (none) -> commons_passives_THT:Passive_THT_ferrite_bead_W3.81mm_L15.24mm
- L404, L405, L406, L407, L408, L409: footprint (none) -> commons_passives_THT:Passive_THT_EMI_filter_W5.08mm_L7.62mm
- R406, R407, R408, R409, R410, R413, R420, R423, R425, R427, R429, R431, R432, R433, R434, R435, R436, R437, R438, R440, R441, R472: footprint Resistor_THT:R_Axial_DIN0204_L3.6mm_D1.6mm_P7.62mm_Horizontal -> commons_passives_THT:Passive_THT_resistor_W2.54mm_L12.70mm
Changed lines of the file:
@@
 F 0 "L401" H 1325 3750 50  0000 L CNN
 F 1 "Ferrite Bead" H 1325 3650 50  0000 L CNN
-F 2 "" V 1180 3700 50  0001 C CNN
+F 2 "commons_passives_THT:Passive_THT_ferrite_bead_W3.81mm_L15.24mm" V 1180 3700 50  0001 C CNN
 F 3 "~" H 1250 3700 50  0001 C CNN
 	1    1250 3700
@@
 F 0 "L402" H 2075 3750 50  0000 L CNN
 F 1 "Ferrite Bead" H 2075 3650 50  0000 L CNN
-F 2 "" V 1930 3700 50  0001 C CNN
+F 2 "commons_passives_THT:Passive_THT_ferrite_bead_W3.81mm_L15.24mm" V 1930 3700 50  0001 C CNN
 F 3 "~" H 2000 3700 50  0001 C CNN
 	1    2000 3700
@@
 F 0 "R406" V 3650 3400 50  0000 C CNN
 F 1 "1K" V 3850 3400 50  0000 C CNN
-F 2 "Resistor_THT:R_Axial_DIN0204_L3.6mm_D1.6mm_P7.62mm_Horizontal" H 3750 3400 50  0001 C CNN
+F 2 "commons_passives_THT:Passive_THT_resistor_W2.54mm_L12.70mm" H 3750 3400 50  0001 C CNN
 F 3 "~" H 3750 3400 50  0001 C CNN
 	1    3750 3400
@@
 F 0 "R407" V 4150 4000 50  0000 C CNN
 F 1 "75" V 4350 4000 50  0000 C CNN
-F 2 "Resistor_THT:R_Axial_DIN0204_L3.6mm_D1.6mm_P7.62mm_Horizontal" H 4250 4000 50  0001 C CNN
+F 2 "commons_passives_THT:Passive_THT_resistor_W2.54mm_L12.70mm" H 4250 4000 50  0001 C CNN
 F 3 "~" H 4250 4000 50  0001 C CNN
 	1    4250 4000
@@
 F 0 "R409" H 4030 4320 50  0000 L CNN
 F 1 "75" H 4030 4260 50  0000 L CNN
-F 2 "Resistor_THT:R_Axial_DIN0204_L3.6mm_D1.6mm_P7.62mm_Horizontal" H 4000 4300 50  0001 C CNN
+F 2 "commons_passives_THT:Passive_THT_resistor_W2.54mm_L12.70mm" H 4000 4300 50  0001 C CNN
 F 3 "~" H 4000 4300 50  0001 C CNN
 	1    4000 4300
@@
 F 0 "R410" H 4030 4820 50  0000 L CNN
 F 1 "75" H 4030 4760 50  0000 L CNN
-F 2 "Resistor_THT:R_Axial_DIN0204_L3.6mm_D1.6mm_P7.62mm_Horizontal" H 4000 4800 50  0001 C CNN
+F 2 "commons_passives_THT:Passive_THT_resistor_W2.54mm_L12.70mm" H 4000 4800 50  0001 C CNN
 F 3 "~" H 4000 4800 50  0001 C CNN
 	1    4000 4800
@@
 F 0 "R408" H 3530 3970 50  0000 L CNN
 F 1 "2K" H 3530 3910 50  0000 L CNN
-F 2 "Resistor_THT:R_Axial_DIN0204_L3.6mm_D1.6mm_P7.62mm_Horizontal" H 3500 3950 50  0001 C CNN
+F 2 "commons_passives_THT:Passive_THT_resistor_W2.54mm_L12.70mm" H 3500 3950 50  0001 C CNN
 F 3 "~" H 3500 3950 50  0001 C CNN
 	1    3500 3950
@@
 F 0 "R413" V 6150 3400 50  0000 C CNN
 F 1 "1K" V 6350 3400 50  0000 C CNN
-F 2 "Resistor_THT:R_Axial_DIN0204_L3.6mm_D1.6mm_P7.62mm_Horizontal" H 6250 3400 50  0001 C CNN
+F 2 "commons_passives_THT:Passive_THT_resistor_W2.54mm_L12.70mm" H 6250 3400 50  0001 C CNN
 F 3 "~" H 6250 3400 50  0001 C CNN
 	1    6250 3400
@@
 F 0 "R423" H 6030 3970 50  0000 L CNN
 F 1 "2K" H 6030 3910 50  0000 L CNN
-F 2 "Resistor_THT:R_Axial_DIN0204_L3.6mm_D1.6mm_P7.62mm_Horizontal" H 6000 3950 50  0001 C CNN
+F 2 "commons_passives_THT:Passive_THT_resistor_W2.54mm_L12.70mm" H 6000 3950 50  0001 C CNN
 F 3 "~" H 6000 3950 50  0001 C CNN
 	1    6000 3950
@@
 F 0 "R420" V 6650 4000 50  0000 C CNN
 F 1 "75" V 6850 4000 50  0000 C CNN
-F 2 "Resistor_THT:R_Axial_DIN0204_L3.6mm_D1.6mm_P7.62mm_Horizontal" H 6750 4000 50  0001 C CNN
+F 2 "commons_passives_THT:Passive_THT_resistor_W2.54mm_L12.70mm" H 6750 4000 50  0001 C CNN
 F 3 "~" H 6750 4000 50  0001 C CNN
 	1    6750 4000
@@
 F 0 "R425" H 6530 4320 50  0000 L CNN
 F 1 "75" H 6530 4260 50  0000 L CNN
-F 2 "Resistor_THT:R_Axial_DIN0204_L3.6mm_D1.6mm_P7.62mm_Horizontal" H 6500 4300 50  0001 C CNN
+F 2 "commons_passives_THT:Passive_THT_resistor_W2.54mm_L12.70mm" H 6500 4300 50  0001 C CNN
 F 3 "~" H 6500 4300 50  0001 C CNN
 	1    6500 4300
@@
 F 0 "R427" H 6530 4820 50  0000 L CNN
 F 1 "75" H 6530 4760 50  0000 L CNN
-F 2 "Resistor_THT:R_Axial_DIN0204_L3.6mm_D1.6mm_P7.62mm_Horizontal" H 6500 4800 50  0001 C CNN
+F 2 "commons_passives_THT:Passive_THT_resistor_W2.54mm_L12.70mm" H 6500 4800 50  0001 C CNN
 F 3 "~" H 6500 4800 50  0001 C CNN
 	1    6500 4800
@@
 F 0 "R429" V 2400 5400 50  0000 C CNN
 F 1 "1K" V 2600 5400 50  0000 C CNN
-F 2 "Resistor_THT:R_Axial_DIN0204_L3.6mm_D1.6mm_P7.62mm_Horizontal" H 2500 5400 50  0001 C CNN
+F 2 "commons_passives_THT:Passive_THT_resistor_W2.54mm_L12.70mm" H 2500 5400 50  0001 C CNN
 F 3 "~" H 2500 5400 50  0001 C CNN
 	1    2500 5400
@@
 F 0 "R433" H 2280 5970 50  0000 L CNN
 F 1 "2K" H 2280 5910 50  0000 L CNN
-F 2 "Resistor_THT:R_Axial_DIN0204_L3.6mm_D1.6mm_P7.62mm_Horizontal" H 2250 5950 50  0001 C CNN
+F 2 "commons_passives_THT:Passive_THT_resistor_W2.54mm_L12.70mm" H 2250 5950 50  0001 C CNN
 F 3 "~" H 2250 5950 50  0001 C CNN
 	1    2250 5950
@@
 F 0 "R432" V 2900 6000 50  0000 C CNN
 F 1 "75" V 3100 6000 50  0000 C CNN
-F 2 "Resistor_THT:R_Axial_DIN0204_L3.6mm_D1.6mm_P7.62mm_Horizontal" H 3000 6000 50  0001 C CNN
+F 2 "commons_passives_THT:Passive_THT_resistor_W2.54mm_L12.70mm" H 3000 6000 50  0001 C CNN
 F 3 "~" H 3000 6000 50  0001 C CNN
 	1    3000 6000
@@
 F 0 "R434" H 2780 6320 50  0000 L CNN
 F 1 "75" H 2780 6260 50  0000 L CNN
-F 2 "Resistor_THT:R_Axial_DIN0204_L3.6mm_D1.6mm_P7.62mm_Horizontal" H 2750 6300 50  0001 C CNN
+F 2 "commons_passives_THT:Passive_THT_resistor_W2.54mm_L12.70mm" H 2750 6300 50  0001 C CNN
 F 3 "~" H 2750 6300 50  0001 C CNN
 	1    2750 6300
@@
 F 0 "R436" H 2780 6820 50  0000 L CNN
 F 1 "75" H 2780 6760 50  0000 L CNN
-F 2 "Resistor_THT:R_Axial_DIN0204_L3.6mm_D1.6mm_P7.62mm_Horizontal" H 2750 6800 50  0001 C CNN
+F 2 "commons_passives_THT:Passive_THT_resistor_W2.54mm_L12.70mm" H 2750 6800 50  0001 C CNN
 F 3 "~" H 2750 6800 50  0001 C CNN
 	1    2750 6800
@@
 F 0 "R440" H 4780 5970 50  0000 L CNN
 F 1 "1K" H 4780 5910 50  0000 L CNN
-F 2 "Resistor_THT:R_Axial_DIN0204_L3.6mm_D1.6mm_P7.62mm_Horizontal" H 4750 5950 50  0001 C CNN
+F 2 "commons_passives_THT:Passive_THT_resistor_W2.54mm_L12.70mm" H 4750 5950 50  0001 C CNN
 F 3 "~" H 4750 5950 50  0001 C CNN
 	1    4750 5950
@@
 F 0 "R438" V 5400 6000 50  0000 C CNN
 F 1 "27" V 5600 6000 50  0000 C CNN
-F 2 "Resistor_THT:R_Axial_DIN0204_L3.6mm_D1.6mm_P7.62mm_Horizontal" H 5500 6000 50  0001 C CNN
+F 2 "commons_passives_THT:Passive_THT_resistor_W2.54mm_L12.70mm" H 5500 6000 50  0001 C CNN
 F 3 "~" H 5500 6000 50  0001 C CNN
 	1    5500 6000
@@
 F 0 "R441" H 5280 6320 50  0000 L CNN
 F 1 "100" H 5280 6260 50  0000 L CNN
-F 2 "Resistor_THT:R_Axial_DIN0204_L3.6mm_D1.6mm_P7.62mm_Horizontal" H 5250 6300 50  0001 C CNN
+F 2 "commons_passives_THT:Passive_THT_resistor_W2.54mm_L12.70mm" H 5250 6300 50  0001 C CNN
 F 3 "~" H 5250 6300 50  0001 C CNN
 	1    5250 6300
@@
 F 0 "L409" H 2100 1975 50  0000 C CNN
 F 1 "EMI_Filter_LCL" H 2100 1900 50  0000 C CNN
-F 2 "" V 2100 1700 50  0001 C CNN
+F 2 "commons_passives_THT:Passive_THT_EMI_filter_W5.08mm_L7.62mm" V 2100 1700 50  0001 C CNN
 F 3 "http://www.murata.com/~/media/webrenewal/support/library/catalog/products/emc/emifil/c31e.ashx?la=en-gb" V 2100 1700 50  0001 C CNN
 	1    2100 1700
@@
 F 0 "L407" H 2100 2475 50  0000 C CNN
 F 1 "EMI_Filter_LCL" H 2100 2400 50  0000 C CNN
-F 2 "" V 2100 2200 50  0001 C CNN
+F 2 "commons_passives_THT:Passive_THT_EMI_filter_W5.08mm_L7.62mm" V 2100 2200 50  0001 C CNN
 F 3 "http://www.murata.com/~/media/webrenewal/support/library/catalog/products/emc/emifil/c31e.ashx?la=en-gb" V 2100 2200 50  0001 C CNN
 	1    2100 2200
@@
 F 0 "L406" H 4100 2475 50  0000 C CNN
 F 1 "EMI_Filter_LCL" H 4100 2400 50  0000 C CNN
-F 2 "" V 4100 2200 50  0001 C CNN
+F 2 "commons_passives_THT:Passive_THT_EMI_filter_W5.08mm_L7.62mm" V 4100 2200 50  0001 C CNN
 F 3 "http://www.murata.com/~/media/webrenewal/support/library/catalog/products/emc/emifil/c31e.ashx?la=en-gb" V 4100 2200 50  0001 C CNN
 	1    4100 2200
@@
 F 0 "R431" V 3450 2100 50  0000 C CNN
 F 1 "1K2" V 3650 2100 50  0000 C CNN
-F 2 "Resistor_THT:R_Axial_DIN0204_L3.6mm_D1.6mm_P7.62mm_Horizontal" H 3550 2100 50  0001 C CNN
+F 2 "commons_passives_THT:Passive_THT_resistor_W2.54mm_L12.70mm" H 3550 2100 50  0001 C CNN
 F 3 "~" H 3550 2100 50  0001 C CNN
 	1    3550 2100
@@
 F 0 "L405" H 2100 2975 50  0000 C CNN
 F 1 "EMI_Filter_LCL" H 2100 2900 50  0000 C CNN
-F 2 "" V 2100 2700 50  0001 C CNN
+F 2 "commons_passives_THT:Passive_THT_EMI_filter_W5.08mm_L7.62mm" V 2100 2700 50  0001 C CNN
 F 3 "http://www.murata.com/~/media/webrenewal/support/library/catalog/products/emc/emifil/c31e.ashx?la=en-gb" V 2100 2700 50  0001 C CNN
 	1    2100 2700
@@
 F 0 "R437" V 1450 2600 50  0000 C CNN
 F 1 "33" V 1650 2600 50  0000 C CNN
-F 2 "Resistor_THT:R_Axial_DIN0204_L3.6mm_D1.6mm_P7.62mm_Horizontal" H 1550 2600 50  0001 C CNN
+F 2 "commons_passives_THT:Passive_THT_resistor_W2.54mm_L12.70mm" H 1550 2600 50  0001 C CNN
 F 3 "~" H 1550 2600 50  0001 C CNN
 	1    1550 2600
@@
 F 0 "L404" H 4100 2975 50  0000 C CNN
 F 1 "EMI_Filter_LCL" H 4100 2900 50  0000 C CNN
-F 2 "" V 4100 2700 50  0001 C CNN
+F 2 "commons_passives_THT:Passive_THT_EMI_filter_W5.08mm_L7.62mm" V 4100 2700 50  0001 C CNN
 F 3 "http://www.murata.com/~/media/webrenewal/support/library/catalog/products/emc/emifil/c31e.ashx?la=en-gb" V 4100 2700 50  0001 C CNN
 	1    4100 2700
@@
 F 0 "R435" V 3450 2600 50  0000 C CNN
 F 1 "33" V 3650 2600 50  0000 C CNN
-F 2 "Resistor_THT:R_Axial_DIN0204_L3.6mm_D1.6mm_P7.62mm_Horizontal" H 3550 2600 50  0001 C CNN
+F 2 "commons_passives_THT:Passive_THT_resistor_W2.54mm_L12.70mm" H 3550 2600 50  0001 C CNN
 F 3 "~" H 3550 2600 50  0001 C CNN
 	1    3550 2600
@@
 F 0 "L408" H 4100 1975 50  0000 C CNN
 F 1 "EMI_Filter_LCL" H 4100 1900 50  0000 C CNN
-F 2 "" V 4100 1700 50  0001 C CNN
+F 2 "commons_passives_THT:Passive_THT_EMI_filter_W5.08mm_L7.62mm" V 4100 1700 50  0001 C CNN
 F 3 "http://www.murata.com/~/media/webrenewal/support/library/catalog/products/emc/emifil/c31e.ashx?la=en-gb" V 4100 1700 50  0001 C CNN
 	1    4100 1700
@@
 F 0 "R472" H 3680 1320 50  0000 L CNN
 F 1 "4K7" H 3680 1260 50  0000 L CNN
-F 2 "Resistor_THT:R_Axial_DIN0204_L3.6mm_D1.6mm_P7.62mm_Horizontal" H 3650 1300 50  0001 C CNN
+F 2 "commons_passives_THT:Passive_THT_resistor_W2.54mm_L12.70mm" H 3650 1300 50  0001 C CNN
 F 3 "~" H 3650 1300 50  0001 C CNN
 	1    3650 1300

Commit message: [PCB] continue footprint assignation
Parts:
- C411, C414: footprint (none) -> commons_passives_THT:Passive_THT_capacitor_ceramic_radial_W5.08mm_L6.35mm_X11.43mm
Changed lines of the file:
@@
 F 0 "C411" H 1275 4450 50  0000 L CNN
 F 1 "0.1uF" H 1275 4250 50  0000 L CNN
-F 2 "" H 1288 4200 50  0001 C CNN
+F 2 "commons_passives_THT:Passive_THT_capacitor_ceramic_radial_W5.08mm_L6.35mm_X11.43mm" H 1288 4200 50  0001 C CNN
 F 3 "~" H 1250 4350 50  0001 C CNN
 	1    1250 4350
@@
 F 0 "C414" H 2025 4450 50  0000 L CNN
 F 1 "0.1uF" H 2025 4250 50  0000 L CNN
-F 2 "" H 2038 4200 50  0001 C CNN
+F 2 "commons_passives_THT:Passive_THT_capacitor_ceramic_radial_W5.08mm_L6.35mm_X11.43mm" H 2038 4200 50  0001 C CNN
 F 3 "~" H 2000 4350 50  0001 C CNN
 	1    2000 4350

Commit message: [PCB] continue assigning footprints - done all fixed capacitors
Parts:
- C416: footprint (none) -> commons_passives_THT:Passive_THT_capacitor_polarized_rad_D5.08mm_P2.54mm_H12.70mm
Changed lines of the file:
@@
 F 0 "C416" V 1700 1550 50  0000 L CNN
 F 1 "47uF" V 1400 1500 50  0000 L CNN
-F 2 "" H 1550 1600 50  0001 C CNN
+F 2 "commons_passives_THT:Passive_THT_capacitor_polarized_rad_D5.08mm_P2.54mm_H12.70mm" H 1550 1600 50  0001 C CNN
 F 3 "~" H 1550 1600 50  0001 C CNN
 	1    1550 1600

Commit message: [PCB] Done assigning footprint
Parts:
- J400: footprint (none) -> atari-interconnect:socket-din-13
Changed lines of the file:
@@
 F 0 "J400" H 6350 2600 50  0000 C CNN
 F 1 "DIN 13 — Video Port" H 6350 1200 50  0000 C CNN
-F 2 "" H 6350 1900 50  0001 C CNN
+F 2 "atari-interconnect:socket-din-13" H 6350 1900 50  0001 C CNN
 F 3 "~" H 6350 1900 50  0001 C CNN
 	1    6350 1900

Commit message: Resolves #45 : [Atari STE]Use shielded connectors
Parts:
- J400: value DIN 13 — Video Port -> DIN-13S — Video Port; symbol Connector_Generic:Conn_01x13 -> Connector_Generic_Shielded:Conn_01x13_Shielded
Connections:
- wire segments 121 -> 122
Changed lines of the file:
@@
 $EndDescr
 $Comp
-L Connector_Generic:Conn_01x13 J400
+L Connector_Generic_Shielded:Conn_01x13_Shielded J400
 U 1 1 60B3F5D5
 P 6350 1900
 F 0 "J400" H 6350 2600 50  0000 C CNN
-F 1 "DIN 13 — Video Port" H 6350 1200 50  0000 C CNN
+F 1 "DIN-13S — Video Port" H 6350 2700 50  0000 C CNN
 F 2 "atari-interconnect:socket-din-13" H 6350 1900 50  0001 C CNN
 F 3 "~" H 6350 1900 50  0001 C CNN
@@
 Text Notes 4300 7650 0    50   ~ 0
 It may also be a 74F257
+Text Label 6350 2900 1    50   ~ 0
+GND
+Wire Wire Line
+	6350 2900 6350 2700
 $EndSCHEMATC
