File: atari-16-32-bits/motherboards/c300780-001/subsheet_504.sch (KiCad schematic (older format))
At the start: 36 parts, among them J502 Phono LEFT, J503 Phono RIGHT, U504 LF347N_mu, U508 LMC1992CCN_PHY

Commit message: [PCB] Assign builtins footprint when possible - resistors, ports
Parts:
- R520, R524, R525, R527, R530, R531, R533, R537, R538, R539, R540, R541, R590, R591: footprint (none) -> Resistor_THT:R_Axial_DIN0204_L3.6mm_D1.6mm_P7.62mm_Horizontal
Changed lines of the file:
@@
 F 0 "R530" H 4050 2150 50  0000 L CNN
 F 1 "10K" H 4050 2050 50  0000 L CNN
-F 2 "" H 4000 2100 50  0001 C CNN
+F 2 "Resistor_THT:R_Axial_DIN0204_L3.6mm_D1.6mm_P7.62mm_Horizontal" H 4000 2100 50  0001 C CNN
 F 3 "~" H 4000 2100 50  0001 C CNN
 	1    4000 2100
@@
 F 0 "R525" H 4550 1350 50  0000 L CNN
 F 1 "10K" H 4550 1250 50  0000 L CNN
-F 2 "" H 4500 1300 50  0001 C CNN
+F 2 "Resistor_THT:R_Axial_DIN0204_L3.6mm_D1.6mm_P7.62mm_Horizontal" H 4500 1300 50  0001 C CNN
 F 3 "~" H 4500 1300 50  0001 C CNN
 	1    4500 1300
@@
 F 0 "R531" V 4200 1400 50  0000 L CNN
 F 1 "51K" V 4000 1450 50  0000 L CNN
-F 2 "" H 4100 1500 50  0001 C CNN
+F 2 "Resistor_THT:R_Axial_DIN0204_L3.6mm_D1.6mm_P7.62mm_Horizontal" H 4100 1500 50  0001 C CNN
 F 3 "~" H 4100 1500 50  0001 C CNN
 	1    4100 1500
@@
 F 0 "R539" V 5000 1500 50  0000 L CNN
 F 1 "51K" V 4800 1500 50  0000 L CNN
-F 2 "" H 4900 1600 50  0001 C CNN
+F 2 "Resistor_THT:R_Axial_DIN0204_L3.6mm_D1.6mm_P7.62mm_Horizontal" H 4900 1600 50  0001 C CNN
 F 3 "~" H 4900 1600 50  0001 C CNN
 	1    4900 1600
@@
 F 0 "R520" H 1900 5450 50  0000 C CNN
 F 1 "1K" H 1900 5550 50  0000 C CNN
-F 2 "" H 1750 5500 50  0001 C CNN
+F 2 "Resistor_THT:R_Axial_DIN0204_L3.6mm_D1.6mm_P7.62mm_Horizontal" H 1750 5500 50  0001 C CNN
 F 3 "~" H 1750 5500 50  0001 C CNN
 	1    1750 5500
@@
 F 0 "R590" V 1400 7400 50  0000 L CNN
 F 1 "270K" V 1600 7400 50  0000 L CNN
-F 2 "" H 1500 7500 50  0001 C CNN
+F 2 "Resistor_THT:R_Axial_DIN0204_L3.6mm_D1.6mm_P7.62mm_Horizontal" H 1500 7500 50  0001 C CNN
 F 3 "~" H 1500 7500 50  0001 C CNN
 	1    1500 7500
@@
 F 0 "R533" H 6350 5450 50  0000 C CNN
 F 1 "1K" H 6350 5550 50  0000 C CNN
-F 2 "" H 6500 5500 50  0001 C CNN
+F 2 "Resistor_THT:R_Axial_DIN0204_L3.6mm_D1.6mm_P7.62mm_Horizontal" H 6500 5500 50  0001 C CNN
 F 3 "~" H 6500 5500 50  0001 C CNN
 	1    6500 5500
@@
 F 0 "R591" V 6150 7400 50  0000 L CNN
 F 1 "270K" V 6350 7400 50  0000 L CNN
-F 2 "" H 6250 7500 50  0001 C CNN
+F 2 "Resistor_THT:R_Axial_DIN0204_L3.6mm_D1.6mm_P7.62mm_Horizontal" H 6250 7500 50  0001 C CNN
 F 3 "~" H 6250 7500 50  0001 C CNN
 	1    6250 7500
@@
 F 0 "R527" H 2100 5700 50  0000 C CNN
 F 1 "10K" H 2100 5800 50  0000 C CNN
-F 2 "" H 2250 5750 50  0001 C CNN
+F 2 "Resistor_THT:R_Axial_DIN0204_L3.6mm_D1.6mm_P7.62mm_Horizontal" H 2250 5750 50  0001 C CNN
 F 3 "~" H 2250 5750 50  0001 C CNN
 	1    2250 5750
@@
 F 0 "R524" V 2850 5750 50  0000 L CNN
 F 1 "3K6" V 2850 6150 50  0000 L CNN
-F 2 "" H 2900 6050 50  0001 C CNN
+F 2 "Resistor_THT:R_Axial_DIN0204_L3.6mm_D1.6mm_P7.62mm_Horizontal" H 2900 6050 50  0001 C CNN
 F 3 "~" H 2900 6050 50  0001 C CNN
 	1    2900 6050
@@
 F 0 "R540" H 3400 6700 50  0000 C CNN
 F 1 "1K" H 3400 6800 50  0000 C CNN
-F 2 "" H 3550 6750 50  0001 C CNN
+F 2 "Resistor_THT:R_Axial_DIN0204_L3.6mm_D1.6mm_P7.62mm_Horizontal" H 3550 6750 50  0001 C CNN
 F 3 "~" H 3550 6750 50  0001 C CNN
 	1    3550 6750
@@
 F 0 "R538" H 5850 5700 50  0000 C CNN
 F 1 "10K" H 5850 5800 50  0000 C CNN
-F 2 "" H 6000 5750 50  0001 C CNN
+F 2 "Resistor_THT:R_Axial_DIN0204_L3.6mm_D1.6mm_P7.62mm_Horizontal" H 6000 5750 50  0001 C CNN
 F 3 "~" H 6000 5750 50  0001 C CNN
 	1    6000 5750
@@
 F 0 "R537" V 5400 6150 50  0000 L CNN
 F 1 "3K6" V 5400 5800 50  0000 L CNN
-F 2 "" H 5350 6050 50  0001 C CNN
+F 2 "Resistor_THT:R_Axial_DIN0204_L3.6mm_D1.6mm_P7.62mm_Horizontal" H 5350 6050 50  0001 C CNN
 F 3 "~" H 5350 6050 50  0001 C CNN
 	1    5350 6050
@@
 F 0 "R541" H 4550 6700 50  0000 C CNN
 F 1 "1K" H 4550 6800 50  0000 C CNN
-F 2 "" H 4700 6750 50  0001 C CNN
+F 2 "Resistor_THT:R_Axial_DIN0204_L3.6mm_D1.6mm_P7.62mm_Horizontal" H 4700 6750 50  0001 C CNN
 F 3 "~" H 4700 6750 50  0001 C CNN
 	1    4700 6750

Commit message: Resolves #41 : [PCB] custom footprint library for passives
Parts:
- L504, L505: footprint (none) -> commons_passives_THT:Passive_THT_EMI_filter_W5.08mm_L7.62mm
- R520, R524, R525, R527, R530, R531, R533, R537, R538, R539, R540, R541, R590, R591: footprint Resistor_THT:R_Axial_DIN0204_L3.6mm_D1.6mm_P7.62mm_Horizontal -> commons_passives_THT:Passive_THT_resistor_W2.54mm_L12.70mm
Changed lines of the file:
@@
 F 0 "R530" H 4050 2150 50  0000 L CNN
 F 1 "10K" H 4050 2050 50  0000 L CNN
-F 2 "Resistor_THT:R_Axial_DIN0204_L3.6mm_D1.6mm_P7.62mm_Horizontal" H 4000 2100 50  0001 C CNN
+F 2 "commons_passives_THT:Passive_THT_resistor_W2.54mm_L12.70mm" H 4000 2100 50  0001 C CNN
 F 3 "~" H 4000 2100 50  0001 C CNN
 	1    4000 2100
@@
 F 0 "R525" H 4550 1350 50  0000 L CNN
 F 1 "10K" H 4550 1250 50  0000 L CNN
-F 2 "Resistor_THT:R_Axial_DIN0204_L3.6mm_D1.6mm_P7.62mm_Horizontal" H 4500 1300 50  0001 C CNN
+F 2 "commons_passives_THT:Passive_THT_resistor_W2.54mm_L12.70mm" H 4500 1300 50  0001 C CNN
 F 3 "~" H 4500 1300 50  0001 C CNN
 	1    4500 1300
@@
 F 0 "R531" V 4200 1400 50  0000 L CNN
 F 1 "51K" V 4000 1450 50  0000 L CNN
-F 2 "Resistor_THT:R_Axial_DIN0204_L3.6mm_D1.6mm_P7.62mm_Horizontal" H 4100 1500 50  0001 C CNN
+F 2 "commons_passives_THT:Passive_THT_resistor_W2.54mm_L12.70mm" H 4100 1500 50  0001 C CNN
 F 3 "~" H 4100 1500 50  0001 C CNN
 	1    4100 1500
@@
 F 0 "R539" V 5000 1500 50  0000 L CNN
 F 1 "51K" V 4800 1500 50  0000 L CNN
-F 2 "Resistor_THT:R_Axial_DIN0204_L3.6mm_D1.6mm_P7.62mm_Horizontal" H 4900 1600 50  0001 C CNN
+F 2 "commons_passives_THT:Passive_THT_resistor_W2.54mm_L12.70mm" H 4900 1600 50  0001 C CNN
 F 3 "~" H 4900 1600 50  0001 C CNN
 	1    4900 1600
@@
 F 0 "R520" H 1900 5450 50  0000 C CNN
 F 1 "1K" H 1900 5550 50  0000 C CNN
-F 2 "Resistor_THT:R_Axial_DIN0204_L3.6mm_D1.6mm_P7.62mm_Horizontal" H 1750 5500 50  0001 C CNN
+F 2 "commons_passives_THT:Passive_THT_resistor_W2.54mm_L12.70mm" H 1750 5500 50  0001 C CNN
 F 3 "~" H 1750 5500 50  0001 C CNN
 	1    1750 5500
@@
 F 0 "L504" V 1750 6450 50  0000 C CNN
 F 1 "EMI_Filter_LCL" V 1850 6450 50  0000 C CNN
-F 2 "" V 1650 6750 50  0001 C CNN
+F 2 "commons_passives_THT:Passive_THT_EMI_filter_W5.08mm_L7.62mm" V 1650 6750 50  0001 C CNN
 F 3 "http://www.murata.com/~/media/webrenewal/support/library/catalog/products/emc/emifil/c31e.ashx?la=en-gb" V 1650 6750 50  0001 C CNN
 	1    1650 6750
@@
 F 0 "R590" V 1400 7400 50  0000 L CNN
 F 1 "270K" V 1600 7400 50  0000 L CNN
-F 2 "Resistor_THT:R_Axial_DIN0204_L3.6mm_D1.6mm_P7.62mm_Horizontal" H 1500 7500 50  0001 C CNN
+F 2 "commons_passives_THT:Passive_THT_resistor_W2.54mm_L12.70mm" H 1500 7500 50  0001 C CNN
 F 3 "~" H 1500 7500 50  0001 C CNN
 	1    1500 7500
@@
 F 0 "R533" H 6350 5450 50  0000 C CNN
 F 1 "1K" H 6350 5550 50  0000 C CNN
-F 2 "Resistor_THT:R_Axial_DIN0204_L3.6mm_D1.6mm_P7.62mm_Horizontal" H 6500 5500 50  0001 C CNN
+F 2 "commons_passives_THT:Passive_THT_resistor_W2.54mm_L12.70mm" H 6500 5500 50  0001 C CNN
 F 3 "~" H 6500 5500 50  0001 C CNN
 	1    6500 5500
@@
 F 0 "L505" V 6500 6450 50  0000 C CNN
 F 1 "EMI_Filter_LCL" V 6600 6450 50  0000 C CNN
-F 2 "" V 6400 6750 50  0001 C CNN
+F 2 "commons_passives_THT:Passive_THT_EMI_filter_W5.08mm_L7.62mm" V 6400 6750 50  0001 C CNN
 F 3 "http://www.murata.com/~/media/webrenewal/support/library/catalog/products/emc/emifil/c31e.ashx?la=en-gb" V 6400 6750 50  0001 C CNN
 	1    6400 6750
@@
 F 0 "R591" V 6150 7400 50  0000 L CNN
 F 1 "270K" V 6350 7400 50  0000 L CNN
-F 2 "Resistor_THT:R_Axial_DIN0204_L3.6mm_D1.6mm_P7.62mm_Horizontal" H 6250 7500 50  0001 C CNN
+F 2 "commons_passives_THT:Passive_THT_resistor_W2.54mm_L12.70mm" H 6250 7500 50  0001 C CNN
 F 3 "~" H 6250 7500 50  0001 C CNN
 	1    6250 7500
@@
 F 0 "R527" H 2100 5700 50  0000 C CNN
 F 1 "10K" H 2100 5800 50  0000 C CNN
-F 2 "Resistor_THT:R_Axial_DIN0204_L3.6mm_D1.6mm_P7.62mm_Horizontal" H 2250 5750 50  0001 C CNN
+F 2 "commons_passives_THT:Passive_THT_resistor_W2.54mm_L12.70mm" H 2250 5750 50  0001 C CNN
 F 3 "~" H 2250 5750 50  0001 C CNN
 	1    2250 5750
@@
 F 0 "R524" V 2850 5750 50  0000 L CNN
 F 1 "3K6" V 2850 6150 50  0000 L CNN
-F 2 "Resistor_THT:R_Axial_DIN0204_L3.6mm_D1.6mm_P7.62mm_Horizontal" H 2900 6050 50  0001 C CNN
+F 2 "commons_passives_THT:Passive_THT_resistor_W2.54mm_L12.70mm" H 2900 6050 50  0001 C CNN
 F 3 "~" H 2900 6050 50  0001 C CNN
 	1    2900 6050
@@
 F 0 "R540" H 3400 6700 50  0000 C CNN
 F 1 "1K" H 3400 6800 50  0000 C CNN
-F 2 "Resistor_THT:R_Axial_DIN0204_L3.6mm_D1.6mm_P7.62mm_Horizontal" H 3550 6750 50  0001 C CNN
+F 2 "commons_passives_THT:Passive_THT_resistor_W2.54mm_L12.70mm" H 3550 6750 50  0001 C CNN
 F 3 "~" H 3550 6750 50  0001 C CNN
 	1    3550 6750
@@
 F 0 "R538" H 5850 5700 50  0000 C CNN
 F 1 "10K" H 5850 5800 50  0000 C CNN
-F 2 "Resistor_THT:R_Axial_DIN0204_L3.6mm_D1.6mm_P7.62mm_Horizontal" H 6000 5750 50  0001 C CNN
+F 2 "commons_passives_THT:Passive_THT_resistor_W2.54mm_L12.70mm" H 6000 5750 50  0001 C CNN
 F 3 "~" H 6000 5750 50  0001 C CNN
 	1    6000 5750
@@
 F 0 "R537" V 5400 6150 50  0000 L CNN
 F 1 "3K6" V 5400 5800 50  0000 L CNN
-F 2 "Resistor_THT:R_Axial_DIN0204_L3.6mm_D1.6mm_P7.62mm_Horizontal" H 5350 6050 50  0001 C CNN
+F 2 "commons_passives_THT:Passive_THT_resistor_W2.54mm_L12.70mm" H 5350 6050 50  0001 C CNN
 F 3 "~" H 5350 6050 50  0001 C CNN
 	1    5350 6050
@@
 F 0 "R541" H 4550 6700 50  0000 C CNN
 F 1 "1K" H 4550 6800 50  0000 C CNN
-F 2 "Resistor_THT:R_Axial_DIN0204_L3.6mm_D1.6mm_P7.62mm_Horizontal" H 4700 6750 50  0001 C CNN
+F 2 "commons_passives_THT:Passive_THT_resistor_W2.54mm_L12.70mm" H 4700 6750 50  0001 C CNN
 F 3 "~" H 4700 6750 50  0001 C CNN
 	1    4700 6750

Commit message: [PCB] continue footprint assignation
Parts:
- C524, C536: footprint (none) -> commons_passives_THT:Passive_THT_capacitor_ceramic_radial_W5.08mm_L6.35mm_X11.43mm
Changed lines of the file:
@@
 F 0 "C536" H 5050 2200 50  0000 L CNN
 F 1 "0.1uF" H 5050 2000 50  0000 L CNN
-F 2 "" H 5000 2100 50  0001 C CNN
+F 2 "commons_passives_THT:Passive_THT_capacitor_ceramic_radial_W5.08mm_L6.35mm_X11.43mm" H 5000 2100 50  0001 C CNN
 F 3 "~" H 5000 2100 50  0001 C CNN
 	1    5000 2100
@@
 F 0 "C524" H 825 3100 50  0000 L CNN
 F 1 "0.1uF" H 825 2900 50  0000 L CNN
-F 2 "" H 838 2850 50  0001 C CNN
+F 2 "commons_passives_THT:Passive_THT_capacitor_ceramic_radial_W5.08mm_L6.35mm_X11.43mm" H 838 2850 50  0001 C CNN
 F 3 "~" H 800 3000 50  0001 C CNN
 	1    800  3000

Commit message: [PCB] continue assigning footprints - done all fixed capacitors
Parts:
- C525, C529, C535, C537, C541, C543, C544, C546, C547: footprint (none) -> commons_passives_THT:Passive_THT_capacitor_polarized_W6.35mm_L20.32mm
- C528, C531, C534, C538: footprint (none) -> commons_passives_THT:Passive_THT_capacitor_mlcc_W2.54mm_L10.16mm
- C542: footprint (none) -> commons_passives_THT:Passive_THT_capacitor_polarized_W5.08mm_L17.78mm
Changed lines of the file:
@@
 F 0 "C535" H 4550 2200 50  0000 L CNN
 F 1 "47uF" H 4550 2000 50  0000 L CNN
-F 2 "" H 4500 2100 50  0001 C CNN
+F 2 "commons_passives_THT:Passive_THT_capacitor_polarized_W6.35mm_L20.32mm" H 4500 2100 50  0001 C CNN
 F 3 "~" H 4500 2100 50  0001 C CNN
 	1    4500 2100
@@
 F 0 "C541" V 2350 1150 50  0000 L CNN
 F 1 "47uF" V 2650 1150 50  0000 L CNN
-F 2 "" H 2500 1250 50  0001 C CNN
+F 2 "commons_passives_THT:Passive_THT_capacitor_polarized_W6.35mm_L20.32mm" H 2500 1250 50  0001 C CNN
 F 3 "~" H 2500 1250 50  0001 C CNN
 	1    2500 1250
@@
 F 0 "C546" V 2350 1650 50  0000 L CNN
 F 1 "47uF" V 2650 1650 50  0000 L CNN
-F 2 "" H 2500 1750 50  0001 C CNN
+F 2 "commons_passives_THT:Passive_THT_capacitor_polarized_W6.35mm_L20.32mm" H 2500 1750 50  0001 C CNN
 F 3 "~" H 2500 1750 50  0001 C CNN
 	1    2500 1750
@@
 F 0 "C544" V 1350 3500 50  0000 L CNN
 F 1 "47uF" V 1350 3950 50  0000 L CNN
-F 2 "" H 1400 3800 50  0001 C CNN
+F 2 "commons_passives_THT:Passive_THT_capacitor_polarized_W6.35mm_L20.32mm" H 1400 3800 50  0001 C CNN
 F 3 "~" H 1400 3800 50  0001 C CNN
 	1    1400 3800
@@
 F 0 "C547" V 6850 3800 50  0000 L CNN
 F 1 "47uF" V 6850 3450 50  0000 L CNN
-F 2 "" H 6800 3700 50  0001 C CNN
+F 2 "commons_passives_THT:Passive_THT_capacitor_polarized_W6.35mm_L20.32mm" H 6800 3700 50  0001 C CNN
 F 3 "~" H 6800 3700 50  0001 C CNN
 	1    6800 3700
@@
 F 0 "C528" V 1950 4050 50  0000 L CNN
 F 1 "0.0082uF" V 1850 3950 50  0000 L CNN
-F 2 "" H 2038 3850 50  0001 C CNN
+F 2 "commons_passives_THT:Passive_THT_capacitor_mlcc_W2.54mm_L10.16mm" H 2038 3850 50  0001 C CNN
 F 3 "~" H 2000 4000 50  0001 C CNN
 	1    2000 4000
@@
 F 0 "C531" H 500 4950 50  0000 L CNN
 F 1 "0.0082uF" H 350 5050 50  0000 L CNN
-F 2 "" H 838 4850 50  0001 C CNN
+F 2 "commons_passives_THT:Passive_THT_capacitor_mlcc_W2.54mm_L10.16mm" H 838 4850 50  0001 C CNN
 F 3 "~" H 800 5000 50  0001 C CNN
 	1    800  5000
@@
 F 0 "C534" H 7600 4950 50  0000 L CNN
 F 1 "0.0082uF" H 7550 5050 50  0000 L CNN
-F 2 "" H 7488 4850 50  0001 C CNN
+F 2 "commons_passives_THT:Passive_THT_capacitor_mlcc_W2.54mm_L10.16mm" H 7488 4850 50  0001 C CNN
 F 3 "~" H 7450 5000 50  0001 C CNN
 	1    7450 5000
@@
 F 0 "C538" V 6300 3950 50  0000 L CNN
 F 1 "0.0082uF" V 6400 3900 50  0000 L CNN
-F 2 "" H 6288 3750 50  0001 C CNN
+F 2 "commons_passives_THT:Passive_THT_capacitor_mlcc_W2.54mm_L10.16mm" H 6288 3750 50  0001 C CNN
 F 3 "~" H 6250 3900 50  0001 C CNN
 	1    6250 3900
@@
 F 0 "C525" H 1450 6050 50  0000 L CNN
 F 1 "47uF" H 1450 5950 50  0000 L CNN
-F 2 "" H 1750 6000 50  0001 C CNN
+F 2 "commons_passives_THT:Passive_THT_capacitor_polarized_W6.35mm_L20.32mm" H 1750 6000 50  0001 C CNN
 F 3 "~" H 1750 6000 50  0001 C CNN
 	1    1750 6000
@@
 F 0 "C537" H 6600 6050 50  0000 L CNN
 F 1 "47uF" H 6600 5950 50  0000 L CNN
-F 2 "" H 6500 6000 50  0001 C CNN
+F 2 "commons_passives_THT:Passive_THT_capacitor_polarized_W6.35mm_L20.32mm" H 6500 6000 50  0001 C CNN
 F 3 "~" H 6500 6000 50  0001 C CNN
 	1    6500 6000
@@
 F 0 "C529" H 2350 5300 50  0000 L CNN
 F 1 "47uF" H 2350 5200 50  0000 L CNN
-F 2 "" H 2250 5250 50  0001 C CNN
+F 2 "commons_passives_THT:Passive_THT_capacitor_polarized_W6.35mm_L20.32mm" H 2250 5250 50  0001 C CNN
 F 3 "~" H 2250 5250 50  0001 C CNN
 	1    2250 5250
@@
 F 0 "C543" H 6100 5300 50  0000 L CNN
 F 1 "47uF" H 6100 5200 50  0000 L CNN
-F 2 "" H 6000 5250 50  0001 C CNN
+F 2 "commons_passives_THT:Passive_THT_capacitor_polarized_W6.35mm_L20.32mm" H 6000 5250 50  0001 C CNN
 F 3 "~" H 6000 5250 50  0001 C CNN
 	1    6000 5250
@@
 F 0 "C542" V 6150 2900 50  0000 L CNN
 F 1 "10uF" V 6050 2900 50  0000 L CNN
-F 2 "" H 6100 3200 50  0001 C CNN
+F 2 "commons_passives_THT:Passive_THT_capacitor_polarized_W5.08mm_L17.78mm" H 6100 3200 50  0001 C CNN
 F 3 "~" H 6100 3200 50  0001 C CNN
 	1    6100 3200

Commit message: [PCB] continue assigning footprints + special libraries of special holes referenced in the measurement schema of the field service manual
Parts:
- J502, J503: footprint (none) -> atari-interconnect:socket-rca-5-pins
Changed lines of the file:
@@
 F 0 "J502" V 1900 8000 50  0000 C CNN
 F 1 "Phono LEFT" V 2000 8000 50  0000 C CNN
-F 2 "" H 1750 8000 50  0001 C CNN
+F 2 "atari-interconnect:socket-rca-5-pins" H 1750 8000 50  0001 C CNN
 F 3 " ~" H 1750 8000 50  0001 C CNN
 	1    1750 8000
@@
 F 0 "J503" V 6650 8000 50  0000 C CNN
 F 1 "Phono RIGHT" V 6750 8000 50  0000 C CNN
-F 2 "" H 6500 8000 50  0001 C CNN
+F 2 "atari-interconnect:socket-rca-5-pins" H 6500 8000 50  0001 C CNN
 F 3 " ~" H 6500 8000 50  0001 C CNN
 	1    6500 8000
