File: atari-16-32-bits/motherboards/c300780-001/subsheet_303.sch (KiCad schematic (older format))
At the start: 4 parts, among them U303 8.010613 MHz, U304 74LS74_PHY

Commit message: general cleanup
Connections:
- net GND: now also U304.7 (GND)
Changed lines of the file:
@@
 Text Notes 5850 2200 0    50   ~ 0
 To YM2149\nand MFP 68901
+Wire Wire Line
+	3900 2000 4150 2000
 $EndSCHEMATC
