File: atari-16-32-bits/motherboards/c300780-001/subsheet_303.sch (KiCad schematic (older format))
At the start: 4 parts, among them U303 8.010613 MHz, U304 74LS74_PHY

Commit message: Fixes #51 : [bug][schematics] fix the association of mlcc capacitors and their footprint in schematics to match the association done in the pcb
Parts:
- C300, C301: footprint commons_passives_THT:Passive_THT_capacitor_ceramic_radial_W5.08mm_L6.35mm_X11.43mm -> commons_passives_THT:Passive_THT_capacitor_mlcc_W2.54mm_L7.62mm
Changed lines of the file:
@@
 F 0 "C300" H 6575 1800 50  0000 L CNN
 F 1 "0.1uF" H 6575 1600 50  0000 L CNN
-F 2 "commons_passives_THT:Passive_THT_capacitor_ceramic_radial_W5.08mm_L6.35mm_X11.43mm" H 6588 1550 50  0001 C CNN
+F 2 "commons_passives_THT:Passive_THT_capacitor_mlcc_W2.54mm_L7.62mm" H 6588 1550 50  0001 C CNN
 F 3 "~" H 6550 1700 50  0001 C CNN
 	1    6550 1700
@@
 F 0 "C301" H 1575 1700 50  0000 L CNN
 F 1 "0.1uF" H 1575 1500 50  0000 L CNN
-F 2 "commons_passives_THT:Passive_THT_capacitor_ceramic_radial_W5.08mm_L6.35mm_X11.43mm" H 1588 1450 50  0001 C CNN
+F 2 "commons_passives_THT:Passive_THT_capacitor_mlcc_W2.54mm_L7.62mm" H 1588 1450 50  0001 C CNN
 F 3 "~" H 1550 1600 50  0001 C CNN
 	1    1550 1600
