File: atari-16-32-bits/motherboards/c300780-001/subsheet_500.sch (KiCad schematic (older format))
At the start: 48 parts, among them J500 DM-15S — JOY0, J501 DM-15S — JOY1, U513 LM556_DUAL_TIMER_PHY, U514 LM556_DUAL_TIMER_PHY

Commit message: Fixed : [ERC] duplicate C528, was C528 and C526
Parts:
- renumbered C528 to C526
Changed lines of the file:
@@
 $EndComp
 $Comp
-L Device:C_Small C528
+L Device:C_Small C526
 U 1 1 60CD0365
 P 1850 2750
-F 0 "C528" H 1860 2820 50  0000 L CNN
+F 0 "C526" H 1860 2820 50  0000 L CNN
 F 1 "800pF" H 1860 2670 50  0000 L CNN
 F 2 "" H 1850 2750 50  0001 C CNN

Commit message: Fixed : [ERC] ambiguous labels joy* vs JOY*
Connections:
- net labels added: j0_1, j0_10, j0_11, j0_12, j0_13, j0_14, j0_15, j0_2, j0_3, j0_4, j0_5, j0_6, j0_7, j1_1, j1_10, j1_11, j1_12, j1_13, j1_14, j1_15, j1_2, j1_3, j1_4, j1_5, j1_6, j1_7
- net labels removed: joy0_1, joy0_10, joy0_11, joy0_12, joy0_13, joy0_14, joy0_15, joy0_2, joy0_3, joy0_4, joy0_5, joy0_6, joy0_7, joy1_1, joy1_10, joy1_11, joy1_12, joy1_13, joy1_14, joy1_15, joy1_2, joy1_3, joy1_4, joy1_5, joy1_6, joy1_7
Changed lines of the file:
@@
 	1    0    0    -1
 $EndComp
-Text Label 3250 1100 0    50   ~ 0
-joy0_1
 Text Label 3250 1200 0    50   ~ 0
-joy0_2
+j0_2
 Text Label 3250 1400 0    50   ~ 0
-joy0_4
+j0_4
 Text Label 3250 1600 0    50   ~ 0
-joy0_6
+j0_6
 Text Label 3250 1700 0    50   ~ 0
-joy0_7
+j0_7
 Text Label 3250 2000 0    50   ~ 0
-joy0_10
+j0_10
 Text Label 3250 2100 0    50   ~ 0
-joy0_11
+j0_11
 Text Label 3250 2200 0    50   ~ 0
-joy0_12
+j0_12
 Text Label 3250 2300 0    50   ~ 0
-joy0_13
+j0_13
 Text Label 3250 2400 0    50   ~ 0
-joy0_14
+j0_14
 Text Label 1500 2500 0    50   ~ 0
-joy0_15
+j0_15
 Text Label 3400 1900 0    50   ~ 0
 GND
@@
 NoConn ~ 3650 1800
 Text Label 6250 1100 0    50   ~ 0
-joy1_1
+j1_1
 Text Label 6250 1200 0    50   ~ 0
-joy1_2
+j1_2
 Text Label 6250 1300 0    50   ~ 0
-joy1_3
+j1_3
 Text Label 6250 1400 0    50   ~ 0
-joy1_4
+j1_4
 Text Label 4500 1500 0    50   ~ 0
-joy1_5
+j1_5
 Text Label 6250 1600 0    50   ~ 0
-joy1_6
+j1_6
 Text Label 6250 1700 0    50   ~ 0
-joy1_7
+j1_7
 Text Label 6250 2000 0    50   ~ 0
-joy1_10
+j1_10
 Text Label 6250 2100 0    50   ~ 0
-joy1_11
+j1_11
 Text Label 6250 2200 0    50   ~ 0
-joy1_12
+j1_12
 Text Label 6250 2300 0    50   ~ 0
-joy1_13
+j1_13
 Text Label 6250 2400 0    50   ~ 0
-joy1_14
+j1_14
 Text Label 4500 2500 0    50   ~ 0
-joy1_15
+j1_15
 Wire Wire Line
 	6250 1100 6650 1100
@@
 	1850 1500 2150 1500
 Text Label 1500 1500 0    50   ~ 0
-joy0_5
+j0_5
 Wire Wire Line
 	1500 1500 1850 1500
@@
 	3350 3800 3250 3800
 Text Label 3700 3700 2    50   ~ 0
-joy0_5
+j0_5
 Text Label 1000 3600 0    50   ~ 0
-joy0_15
+j0_15
 Text Label 4500 3600 0    50   ~ 0
-joy1_5
+j1_5
 Text Label 7200 3700 2    50   ~ 0
-joy1_15
+j1_15
 Wire Wire Line
 	1000 3600 1350 3600
@@
 GND
 Text Label 3350 5700 2    50   ~ 0
-joy0_1
+j0_1
 Text Label 3350 6000 2    50   ~ 0
-joy0_2
+j0_2
 Text Label 3250 1300 0    50   ~ 0
-joy0_3
+j0_3
 Text Label 3350 6300 2    50   ~ 0
-joy0_3
+j0_3
 Text Label 3350 6600 2    50   ~ 0
-joy0_4
+j0_4
 Text Label 3350 7200 2    50   ~ 0
-joy0_7
+j0_7
 Wire Wire Line
 	3050 6000 3350 6000
@@
 	6550 8400 6850 8400
 Text Label 3350 7500 2    50   ~ 0
-joy0_10
+j0_10
 Text Label 3350 7800 2    50   ~ 0
-joy0_11
+j0_11
 Text Label 3350 8100 2    50   ~ 0
-joy0_12
+j0_12
 Text Label 3350 8700 2    50   ~ 0
-joy0_14
+j0_14
 Text Label 3350 8400 2    50   ~ 0
-joy0_13
+j0_13
 Text Label 6850 5700 2    50   ~ 0
-joy1_1
+j1_1
 Text Label 6850 6000 2    50   ~ 0
-joy1_2
+j1_2
 Text Label 6850 6300 2    50   ~ 0
-joy1_3
+j1_3
 Text Label 6850 6600 2    50   ~ 0
-joy1_4
+j1_4
 Text Label 6850 7200 2    50   ~ 0
-joy1_7
+j1_7
 Text Label 6850 7500 2    50   ~ 0
-joy1_10
+j1_10
 Text Label 6850 7800 2    50   ~ 0
-joy1_11
+j1_11
 Text Label 6850 8100 2    50   ~ 0
-joy1_12
+j1_12
 Text Label 6850 8400 2    50   ~ 0
-joy1_13
+j1_13
 Text Label 6850 8700 2    50   ~ 0
-joy1_14
+j1_14
 $Comp
 L Device:EMI_Filter_LCL L?
@@
 GND
 Text Label 6850 6900 2    50   ~ 0
-joy1_6
+j1_6
 Wire Wire Line
 	2550 5700 3350 5700
@@
 $EndComp
 Text Label 3350 6900 2    50   ~ 0
-joy0_6
+j0_6
 Text GLabel 1750 6900 0    50   BiDi ~ 0
 XPEN
@@
 Wire Wire Line
 	6700 4900 6700 5100
+Text Label 3250 1100 0    50   ~ 0
+j0_1
 $EndSCHEMATC
