File: atari-16-32-bits/motherboards/c300780-001/subsheet_500.sch (KiCad schematic (older format))
At the start: 48 parts, among them J500 DM-15S — JOY0, J501 DM-15S — JOY1, U513 LM556_DUAL_TIMER_PHY, U514 LM556_DUAL_TIMER_PHY

Commit message: [PCB] Assign builtins footprint when possible - resistors, ports
Parts:
- J500, J501: footprint (none) -> Connector_Dsub:DSUB-15-HD_Female_Horizontal_P2.29x1.98mm_EdgePinOffset3.03mm_Housed_MountingHolesOffset4.94mm
- R518, R519, R521, R523, R528, R529, R535, R536: footprint (none) -> Resistor_THT:R_Axial_DIN0204_L3.6mm_D1.6mm_P7.62mm_Horizontal
Changed lines of the file:
@@
 F 0 "J501" H 6850 2600 50  0000 C CNN
 F 1 "DM-15S — JOY1" H 6850 1000 50  0000 C CNN
-F 2 "" H 6850 1800 50  0001 C CNN
+F 2 "Connector_Dsub:DSUB-15-HD_Female_Horizontal_P2.29x1.98mm_EdgePinOffset3.03mm_Housed_MountingHolesOffset4.94mm" H 6850 1800 50  0001 C CNN
 F 3 "~" H 6850 1800 50  0001 C CNN
 	1    6850 1800
@@
 F 0 "J500" H 3850 2600 50  0000 C CNN
 F 1 "DM-15S — JOY0" H 3850 1000 50  0000 C CNN
-F 2 "" H 3850 1800 50  0001 C CNN
+F 2 "Connector_Dsub:DSUB-15-HD_Female_Horizontal_P2.29x1.98mm_EdgePinOffset3.03mm_Housed_MountingHolesOffset4.94mm" H 3850 1800 50  0001 C CNN
 F 3 "~" H 3850 1800 50  0001 C CNN
 	1    3850 1800
@@
 F 0 "R521" H 2680 1270 50  0000 L CNN
 F 1 "1M" H 2680 1210 50  0000 L CNN
-F 2 "" H 2650 1250 50  0001 C CNN
+F 2 "Resistor_THT:R_Axial_DIN0204_L3.6mm_D1.6mm_P7.62mm_Horizontal" H 2650 1250 50  0001 C CNN
 F 3 "~" H 2650 1250 50  0001 C CNN
 	1    2650 1250
@@
 F 0 "R518" H 2680 2270 50  0000 L CNN
 F 1 "1M" H 2680 2210 50  0000 L CNN
-F 2 "" H 2650 2250 50  0001 C CNN
+F 2 "Resistor_THT:R_Axial_DIN0204_L3.6mm_D1.6mm_P7.62mm_Horizontal" H 2650 2250 50  0001 C CNN
 F 3 "~" H 2650 2250 50  0001 C CNN
 	1    2650 2250
@@
 F 0 "R528" H 5680 1270 50  0000 L CNN
 F 1 "1M" H 5680 1210 50  0000 L CNN
-F 2 "" H 5650 1250 50  0001 C CNN
+F 2 "Resistor_THT:R_Axial_DIN0204_L3.6mm_D1.6mm_P7.62mm_Horizontal" H 5650 1250 50  0001 C CNN
 F 3 "~" H 5650 1250 50  0001 C CNN
 	1    5650 1250
@@
 F 0 "R535" H 5680 2270 50  0000 L CNN
 F 1 "1M" H 5680 2210 50  0000 L CNN
-F 2 "" H 5650 2250 50  0001 C CNN
+F 2 "Resistor_THT:R_Axial_DIN0204_L3.6mm_D1.6mm_P7.62mm_Horizontal" H 5650 2250 50  0001 C CNN
 F 3 "~" H 5650 2250 50  0001 C CNN
 	1    5650 2250
@@
 F 0 "R523" V 2150 1500 50  0000 C CNN
 F 1 "470" V 2350 1500 50  0000 C CNN
-F 2 "" H 2250 1500 50  0001 C CNN
+F 2 "Resistor_THT:R_Axial_DIN0204_L3.6mm_D1.6mm_P7.62mm_Horizontal" H 2250 1500 50  0001 C CNN
 F 3 "~" H 2250 1500 50  0001 C CNN
 	1    2250 1500
@@
 F 0 "R519" V 2150 2500 50  0000 C CNN
 F 1 "470" V 2350 2500 50  0000 C CNN
-F 2 "" H 2250 2500 50  0001 C CNN
+F 2 "Resistor_THT:R_Axial_DIN0204_L3.6mm_D1.6mm_P7.62mm_Horizontal" H 2250 2500 50  0001 C CNN
 F 3 "~" H 2250 2500 50  0001 C CNN
 	1    2250 2500
@@
 F 0 "R529" V 5150 1500 50  0000 C CNN
 F 1 "470" V 5350 1500 50  0000 C CNN
-F 2 "" H 5250 1500 50  0001 C CNN
+F 2 "Resistor_THT:R_Axial_DIN0204_L3.6mm_D1.6mm_P7.62mm_Horizontal" H 5250 1500 50  0001 C CNN
 F 3 "~" H 5250 1500 50  0001 C CNN
 	1    5250 1500
@@
 F 0 "R536" V 5150 2500 50  0000 C CNN
 F 1 "470" V 5350 2500 50  0000 C CNN
-F 2 "" H 5250 2500 50  0001 C CNN
+F 2 "Resistor_THT:R_Axial_DIN0204_L3.6mm_D1.6mm_P7.62mm_Horizontal" H 5250 2500 50  0001 C CNN
 F 3 "~" H 5250 2500 50  0001 C CNN
 	1    5250 2500

Commit message: Resolves #41 : [PCB] custom footprint library for passives
Parts:
- L500, L501, L502, L503, L508: footprint (none) -> commons_passives_THT:Passive_THT_ferrite_bead_W3.81mm_L15.24mm
- L506, L507, L509, L510, L511, L512, L513, L514, L515, L516, L517, L518, L519, L520, L521, L522, L523, L524, L525, L526, L527: footprint (none) -> commons_passives_THT:Passive_THT_EMI_filter_W5.08mm_L7.62mm
- R518, R519, R521, R523, R528, R529, R535, R536: footprint Resistor_THT:R_Axial_DIN0204_L3.6mm_D1.6mm_P7.62mm_Horizontal -> commons_passives_THT:Passive_THT_resistor_W2.54mm_L12.70mm

Commit message: [PCB] continue footprint assignation
Parts:
- C554, C555: footprint (none) -> commons_passives_THT:Passive_THT_capacitor_ceramic_radial_W5.08mm_L6.35mm_X11.43mm
Changed lines of the file:
@@
 F 0 "C554" H 3225 4850 50  0000 L CNN
 F 1 "0.1uF" H 3225 4650 50  0000 L CNN
-F 2 "" H 3238 4600 50  0001 C CNN
+F 2 "commons_passives_THT:Passive_THT_capacitor_ceramic_radial_W5.08mm_L6.35mm_X11.43mm" H 3238 4600 50  0001 C CNN
 F 3 "~" H 3200 4750 50  0001 C CNN
 	1    3200 4750
@@
 F 0 "C555" H 6725 4850 50  0000 L CNN
 F 1 "0.1uF" H 6725 4650 50  0000 L CNN
-F 2 "" H 6738 4600 50  0001 C CNN
+F 2 "commons_passives_THT:Passive_THT_capacitor_ceramic_radial_W5.08mm_L6.35mm_X11.43mm" H 6738 4600 50  0001 C CNN
 F 3 "~" H 6700 4750 50  0001 C CNN
 	1    6700 4750

Commit message: [PCB] continue assigning footprints - done all fixed capacitors
Parts:
- C526, C532, C539, C548: footprint (none) -> commons_passives_THT:Passive_THT_capacitor_ceramic_radial_W5.08mm_L6.35mm_X11.43mm
- C527, C533, C540, C549: footprint (none) -> commons_passives_THT:Passive_THT_capacitor_W2.54mm_L10.16mm
Changed lines of the file:
@@
 F 0 "C532" H 1860 1820 50  0000 L CNN
 F 1 "800pF" H 1860 1670 50  0000 L CNN
-F 2 "" H 1850 1750 50  0001 C CNN
+F 2 "commons_passives_THT:Passive_THT_capacitor_ceramic_radial_W5.08mm_L6.35mm_X11.43mm" H 1850 1750 50  0001 C CNN
 F 3 "~" H 1850 1750 50  0001 C CNN
 	1    1850 1750
@@
 F 0 "C526" H 1860 2820 50  0000 L CNN
 F 1 "800pF" H 1860 2670 50  0000 L CNN
-F 2 "" H 1850 2750 50  0001 C CNN
+F 2 "commons_passives_THT:Passive_THT_capacitor_ceramic_radial_W5.08mm_L6.35mm_X11.43mm" H 1850 2750 50  0001 C CNN
 F 3 "~" H 1850 2750 50  0001 C CNN
 	1    1850 2750
@@
 F 0 "C539" H 4860 1820 50  0000 L CNN
 F 1 "800pF" H 4860 1670 50  0000 L CNN
-F 2 "" H 4850 1750 50  0001 C CNN
+F 2 "commons_passives_THT:Passive_THT_capacitor_ceramic_radial_W5.08mm_L6.35mm_X11.43mm" H 4850 1750 50  0001 C CNN
 F 3 "~" H 4850 1750 50  0001 C CNN
 	1    4850 1750
@@
 F 0 "C548" H 4860 2820 50  0000 L CNN
 F 1 "800pF" H 4860 2670 50  0000 L CNN
-F 2 "" H 4850 2750 50  0001 C CNN
+F 2 "commons_passives_THT:Passive_THT_capacitor_ceramic_radial_W5.08mm_L6.35mm_X11.43mm" H 4850 2750 50  0001 C CNN
 F 3 "~" H 4850 2750 50  0001 C CNN
 	1    4850 2750
@@
 F 0 "C527" V 1000 3550 50  0000 L CNN
 F 1 "0.01uF" V 1000 3850 50  0000 L CNN
-F 2 "" H 1050 3800 50  0001 C CNN
+F 2 "commons_passives_THT:Passive_THT_capacitor_W2.54mm_L10.16mm" H 1050 3800 50  0001 C CNN
 F 3 "~" H 1050 3800 50  0001 C CNN
 	1    1050 3800
@@
 F 0 "C533" V 3650 3650 50  0000 L CNN
 F 1 "0.01uF" V 3650 3950 50  0000 L CNN
-F 2 "" H 3700 3900 50  0001 C CNN
+F 2 "commons_passives_THT:Passive_THT_capacitor_W2.54mm_L10.16mm" H 3700 3900 50  0001 C CNN
 F 3 "~" H 3700 3900 50  0001 C CNN
 	1    3700 3900
@@
 F 0 "C540" V 4500 3550 50  0000 L CNN
 F 1 "0.01uF" V 4500 3850 50  0000 L CNN
-F 2 "" H 4550 3800 50  0001 C CNN
+F 2 "commons_passives_THT:Passive_THT_capacitor_W2.54mm_L10.16mm" H 4550 3800 50  0001 C CNN
 F 3 "~" H 4550 3800 50  0001 C CNN
 	1    4550 3800
@@
 F 0 "C549" V 7250 3950 50  0000 L CNN
 F 1 "0.01uF" V 7250 3600 50  0000 L CNN
-F 2 "" H 7200 3900 50  0001 C CNN
+F 2 "commons_passives_THT:Passive_THT_capacitor_W2.54mm_L10.16mm" H 7200 3900 50  0001 C CNN
 F 3 "~" H 7200 3900 50  0001 C CNN
 	1    7200 3900

Commit message: Resolves #45 : [Atari STE]Use shielded connectors
Parts:
- J500, J501: symbol Connector_Generic:Conn_01x15 -> Connector_Generic_Shielded:Conn_01x15_Shielded
Connections:
- wire segments 152 -> 154
Changed lines of the file:
@@
 $EndComp
 $Comp
-L Connector_Generic:Conn_01x15 J501
+L Connector_Generic_Shielded:Conn_01x15_Shielded J501
 U 1 1 60C69D74
 P 6850 1800
 F 0 "J501" H 6850 2600 50  0000 C CNN
-F 1 "DM-15S — JOY1" H 6850 1000 50  0000 C CNN
+F 1 "DM-15S — JOY1" H 6850 2700 50  0000 C CNN
 F 2 "Connector_Dsub:DSUB-15-HD_Female_Horizontal_P2.29x1.98mm_EdgePinOffset3.03mm_Housed_MountingHolesOffset4.94mm" H 6850 1800 50  0001 C CNN
 F 3 "~" H 6850 1800 50  0001 C CNN
@@
 $EndComp
 $Comp
-L Connector_Generic:Conn_01x15 J500
+L Connector_Generic_Shielded:Conn_01x15_Shielded J500
 U 1 1 60C6DE62
 P 3850 1800
 F 0 "J500" H 3850 2600 50  0000 C CNN
-F 1 "DM-15S — JOY0" H 3850 1000 50  0000 C CNN
+F 1 "DM-15S — JOY0" H 3850 2700 50  0000 C CNN
 F 2 "Connector_Dsub:DSUB-15-HD_Female_Horizontal_P2.29x1.98mm_EdgePinOffset3.03mm_Housed_MountingHolesOffset4.94mm" H 3850 1800 50  0001 C CNN
 F 3 "~" H 3850 1800 50  0001 C CNN
@@
 Text Label 3250 1100 0    50   ~ 0
 j0_1
+Text Label 3850 2900 1    50   ~ 0
+GND
+Wire Wire Line
+	3850 2900 3850 2700
+Text Label 6850 2900 1    50   ~ 0
+GND
+Wire Wire Line
+	6850 2900 6850 2700
 $EndSCHEMATC

Commit message: Resolves #46 : [PCB] Footprints for shielded ports should have pins named 'SH'
Parts:
- J500, J501: footprint Connector_Dsub:DSUB-15-HD_Female_Horizontal_P2.29x1.98mm_EdgePinOffset3.03mm_Housed_MountingHolesOffset4.94mm -> commons-interconnect_THT:DSUB-15-HD_Female_Horizontal_P2.29x1.98mm_EdgePinOffset8.35mm_Housed_MountingHolesOffset10.89mm
Changed lines of the file:
@@
 F 0 "J501" H 6850 2600 50  0000 C CNN
 F 1 "DM-15S — JOY1" H 6850 2700 50  0000 C CNN
-F 2 "Connector_Dsub:DSUB-15-HD_Female_Horizontal_P2.29x1.98mm_EdgePinOffset3.03mm_Housed_MountingHolesOffset4.94mm" H 6850 1800 50  0001 C CNN
+F 2 "commons-interconnect_THT:DSUB-15-HD_Female_Horizontal_P2.29x1.98mm_EdgePinOffset8.35mm_Housed_MountingHolesOffset10.89mm" H 6850 1800 50  0001 C CNN
 F 3 "~" H 6850 1800 50  0001 C CNN
 	1    6850 1800
@@
 F 0 "J500" H 3850 2600 50  0000 C CNN
 F 1 "DM-15S — JOY0" H 3850 2700 50  0000 C CNN
-F 2 "Connector_Dsub:DSUB-15-HD_Female_Horizontal_P2.29x1.98mm_EdgePinOffset3.03mm_Housed_MountingHolesOffset4.94mm" H 3850 1800 50  0001 C CNN
+F 2 "commons-interconnect_THT:DSUB-15-HD_Female_Horizontal_P2.29x1.98mm_EdgePinOffset8.35mm_Housed_MountingHolesOffset10.89mm" H 3850 1800 50  0001 C CNN
 F 3 "~" H 3850 1800 50  0001 C CNN
 	1    3850 1800
