File: atari-16-32-bits/motherboards/c300780-001/motherboard.kicad_pcb (KiCad board)
At the start: 2 copper layers, 440 x 252 mm, 0 parts

Commit message: [PCB] Placed reference solder mask and silkscreen
Parts:
- added G***: LOGO, pcb-masks:silkscreen, F.Cu at (302.3, 201.7)
- added G***: LOGO, pcb-masks:soldermask-componentside, F.Cu at (302.3, 201.2)
