File: atari-16-32-bits/motherboards/c300780-001/motherboard.kicad_pcb (KiCad board)
At the start: 2 copper layers, 440 x 252 mm, 2 parts

Commit message: [PCB] places mounting holes (precisely when possible)
Parts:
- added REF**: hole_K, atari-motherboard-holes-ste:hole_K, F.Cu at (86.0, 323.7)
- added REF**: hole_U, atari-motherboard-holes-ste:hole_U, F.Cu at (240.7, 191.5)
- added REF**: hole_U, atari-motherboard-holes-ste:hole_U, F.Cu at (109.3, 105.2)
- added REF**: hole_U, atari-motherboard-holes-ste:hole_U, F.Cu at (111.8, 191.5)
- added REF**: hole_U, atari-motherboard-holes-ste:hole_U, F.Cu at (244.3, 112.2)
- added REF**: hole_E, atari-motherboard-holes-ste:hole_E, F.Cu at (244.3, 106.2)
- added REF**: hole_E, atari-motherboard-holes-ste:hole_E, F.Cu at (109.3, 99.2)
- added REF**: hole_Q, atari-motherboard-holes-ste:hole_Q, F.Cu at (437.3, 321.7)
- added REF**: hole_X, atari-motherboard-holes-ste:hole_X, F.Cu at (302.3, 252.7)
- added REF**: hole_K, atari-motherboard-holes-ste:hole_K, F.Cu at (262.0, 322.1)
- added REF**: hole_S, atari-motherboard-holes-ste:hole_S, F.Cu at (412.8, 317.9)
- added REF**: hole_U, atari-motherboard-holes-ste:hole_U, F.Cu at (461.0, 85.0)
- added REF**: hole_V, atari-motherboard-holes-ste:hole_V, F.Cu at (501.0, 191.5)
- added REF**: hole_V, atari-motherboard-holes-ste:hole_V, F.Cu at (431.2, 191.9)
- added REF**: hole_V, atari-motherboard-holes-ste:hole_V, F.Cu at (500.9, 97.2)
- added REF**: hole_V, atari-motherboard-holes-ste:hole_V, F.Cu at (431.0, 97.4)
- added REF**: hole_U, atari-motherboard-holes-ste:hole_U, F.Cu at (352.0, 94.1)
Other:
- outline, holes or cut-outs redrawn
