File: atari-16-32-bits/motherboards/c300780-001/subsheet_100.sch (KiCad schematic (older format))
At the start: 16 parts, among them P100 1K2 ×8, P101 4K7 ×8, P102 4K7 ×8, P103 4K7 ×8, P104 10K ×8, P105 10K ×8, U100 MC68000_PLCC_68_PHY

Commit message: [PCB] Assign builtins footprint when possible - resistors, ports
Parts:
- R102, R103, R104, R105, R107, R109, R110: footprint (none) -> Resistor_THT:R_Axial_DIN0204_L3.6mm_D1.6mm_P7.62mm_Horizontal
Changed lines of the file:
@@
 F 0 "R102" V 6700 5850 50  0000 C CNN
 F 1 "1K" V 6500 5850 50  0000 C CNN
-F 2 "" V 6640 5840 50  0001 C CNN
+F 2 "Resistor_THT:R_Axial_DIN0204_L3.6mm_D1.6mm_P7.62mm_Horizontal" V 6640 5840 50  0001 C CNN
 F 3 "~" H 6600 5850 50  0001 C CNN
 	1    6600 5850
@@
 F 0 "R103" V 5700 5850 50  0000 C CNN
 F 1 "10K" V 5500 5850 50  0000 C CNN
-F 2 "" V 5640 5840 50  0001 C CNN
+F 2 "Resistor_THT:R_Axial_DIN0204_L3.6mm_D1.6mm_P7.62mm_Horizontal" V 5640 5840 50  0001 C CNN
 F 3 "~" H 5600 5850 50  0001 C CNN
 	1    5600 5850
@@
 F 0 "R104" V 5700 6250 50  0000 C CNN
 F 1 "10K" V 5500 6250 50  0000 C CNN
-F 2 "" V 5640 6240 50  0001 C CNN
+F 2 "Resistor_THT:R_Axial_DIN0204_L3.6mm_D1.6mm_P7.62mm_Horizontal" V 5640 6240 50  0001 C CNN
 F 3 "~" H 5600 6250 50  0001 C CNN
 	1    5600 6250
@@
 F 0 "R105" V 5700 6650 50  0000 C CNN
 F 1 "10K" V 5500 6650 50  0000 C CNN
-F 2 "" V 5640 6640 50  0001 C CNN
+F 2 "Resistor_THT:R_Axial_DIN0204_L3.6mm_D1.6mm_P7.62mm_Horizontal" V 5640 6640 50  0001 C CNN
 F 3 "~" H 5600 6650 50  0001 C CNN
 	1    5600 6650
@@
 F 0 "R107" V 6700 6250 50  0000 C CNN
 F 1 "1K" V 6500 6250 50  0000 C CNN
-F 2 "" V 6640 6240 50  0001 C CNN
+F 2 "Resistor_THT:R_Axial_DIN0204_L3.6mm_D1.6mm_P7.62mm_Horizontal" V 6640 6240 50  0001 C CNN
 F 3 "~" H 6600 6250 50  0001 C CNN
 	1    6600 6250
@@
 F 0 "R109" V 6700 6650 50  0000 C CNN
 F 1 "2K2" V 6500 6650 50  0000 C CNN
-F 2 "" V 6640 6640 50  0001 C CNN
+F 2 "Resistor_THT:R_Axial_DIN0204_L3.6mm_D1.6mm_P7.62mm_Horizontal" V 6640 6640 50  0001 C CNN
 F 3 "~" H 6600 6650 50  0001 C CNN
 	1    6600 6650
@@
 F 0 "R110" V 6700 7050 50  0000 C CNN
 F 1 "4K7" V 6500 7050 50  0000 C CNN
-F 2 "" V 6640 7040 50  0001 C CNN
+F 2 "Resistor_THT:R_Axial_DIN0204_L3.6mm_D1.6mm_P7.62mm_Horizontal" V 6640 7040 50  0001 C CNN
 F 3 "~" H 6600 7050 50  0001 C CNN
 	1    6600 7050

Commit message: Resolves #41 : [PCB] custom footprint library for passives
Parts:
- R102, R103, R104, R105, R107, R109, R110: footprint Resistor_THT:R_Axial_DIN0204_L3.6mm_D1.6mm_P7.62mm_Horizontal -> commons_passives_THT:Passive_THT_resistor_W2.54mm_L12.70mm
Changed lines of the file:
@@
 F 0 "R102" V 6700 5850 50  0000 C CNN
 F 1 "1K" V 6500 5850 50  0000 C CNN
-F 2 "Resistor_THT:R_Axial_DIN0204_L3.6mm_D1.6mm_P7.62mm_Horizontal" V 6640 5840 50  0001 C CNN
+F 2 "commons_passives_THT:Passive_THT_resistor_W2.54mm_L12.70mm" V 6640 5840 50  0001 C CNN
 F 3 "~" H 6600 5850 50  0001 C CNN
 	1    6600 5850
@@
 F 0 "R103" V 5700 5850 50  0000 C CNN
 F 1 "10K" V 5500 5850 50  0000 C CNN
-F 2 "Resistor_THT:R_Axial_DIN0204_L3.6mm_D1.6mm_P7.62mm_Horizontal" V 5640 5840 50  0001 C CNN
+F 2 "commons_passives_THT:Passive_THT_resistor_W2.54mm_L12.70mm" V 5640 5840 50  0001 C CNN
 F 3 "~" H 5600 5850 50  0001 C CNN
 	1    5600 5850
@@
 F 0 "R104" V 5700 6250 50  0000 C CNN
 F 1 "10K" V 5500 6250 50  0000 C CNN
-F 2 "Resistor_THT:R_Axial_DIN0204_L3.6mm_D1.6mm_P7.62mm_Horizontal" V 5640 6240 50  0001 C CNN
+F 2 "commons_passives_THT:Passive_THT_resistor_W2.54mm_L12.70mm" V 5640 6240 50  0001 C CNN
 F 3 "~" H 5600 6250 50  0001 C CNN
 	1    5600 6250
@@
 F 0 "R105" V 5700 6650 50  0000 C CNN
 F 1 "10K" V 5500 6650 50  0000 C CNN
-F 2 "Resistor_THT:R_Axial_DIN0204_L3.6mm_D1.6mm_P7.62mm_Horizontal" V 5640 6640 50  0001 C CNN
+F 2 "commons_passives_THT:Passive_THT_resistor_W2.54mm_L12.70mm" V 5640 6640 50  0001 C CNN
 F 3 "~" H 5600 6650 50  0001 C CNN
 	1    5600 6650
@@
 F 0 "R107" V 6700 6250 50  0000 C CNN
 F 1 "1K" V 6500 6250 50  0000 C CNN
-F 2 "Resistor_THT:R_Axial_DIN0204_L3.6mm_D1.6mm_P7.62mm_Horizontal" V 6640 6240 50  0001 C CNN
+F 2 "commons_passives_THT:Passive_THT_resistor_W2.54mm_L12.70mm" V 6640 6240 50  0001 C CNN
 F 3 "~" H 6600 6250 50  0001 C CNN
 	1    6600 6250
@@
 F 0 "R109" V 6700 6650 50  0000 C CNN
 F 1 "2K2" V 6500 6650 50  0000 C CNN
-F 2 "Resistor_THT:R_Axial_DIN0204_L3.6mm_D1.6mm_P7.62mm_Horizontal" V 6640 6640 50  0001 C CNN
+F 2 "commons_passives_THT:Passive_THT_resistor_W2.54mm_L12.70mm" V 6640 6640 50  0001 C CNN
 F 3 "~" H 6600 6650 50  0001 C CNN
 	1    6600 6650
@@
 F 0 "R110" V 6700 7050 50  0000 C CNN
 F 1 "4K7" V 6500 7050 50  0000 C CNN
-F 2 "Resistor_THT:R_Axial_DIN0204_L3.6mm_D1.6mm_P7.62mm_Horizontal" V 6640 7040 50  0001 C CNN
+F 2 "commons_passives_THT:Passive_THT_resistor_W2.54mm_L12.70mm" V 6640 7040 50  0001 C CNN
 F 3 "~" H 6600 7050 50  0001 C CNN
 	1    6600 7050

Commit message: [PCB] continue footprint assignation
Parts:
- C111, C112: footprint (none) -> commons_passives_THT:Passive_THT_capacitor_mlcc_W2.54mm_L10.16mm
Changed lines of the file:
@@
 F 0 "C111" H 6775 1900 50  0000 L CNN
 F 1 "0.1uF" H 6775 1700 50  0000 L CNN
-F 2 "" H 6788 1650 50  0001 C CNN
+F 2 "commons_passives_THT:Passive_THT_capacitor_mlcc_W2.54mm_L10.16mm" H 6788 1650 50  0001 C CNN
 F 3 "~" H 6750 1800 50  0001 C CNN
 	1    6750 1800
@@
 F 0 "C112" H 7275 1900 50  0000 L CNN
 F 1 "0.1uF" H 7275 1700 50  0000 L CNN
-F 2 "" H 7288 1650 50  0001 C CNN
+F 2 "commons_passives_THT:Passive_THT_capacitor_mlcc_W2.54mm_L10.16mm" H 7288 1650 50  0001 C CNN
 F 3 "~" H 7250 1800 50  0001 C CNN
 	1    7250 1800
