File: atari-16-32-bits/motherboards/c300780-001/subsheet_102.sch (KiCad schematic (older format))
At the start: 7 parts, among them U102 EPROM_32_PINS_DIP_PHY, U103 EPROM_32_PINS_DIP_PHY

Commit message: [PCB] continuing footprint assignement
Parts:
- W102, W103, W104: footprint (none) -> Connector_PinHeader_2.54mm:PinHeader_1x03_P2.54mm_Vertical
Changed lines of the file:
@@
 F 0 "W102" H 2650 4770 50  0000 C CNN
 F 1 "SW_SPDT" H 2650 4400 50  0000 C CNN
-F 2 "" H 2650 4600 50  0001 C CNN
+F 2 "Connector_PinHeader_2.54mm:PinHeader_1x03_P2.54mm_Vertical" H 2650 4600 50  0001 C CNN
 F 3 "~" H 2650 4600 50  0001 C CNN
 	1    2650 4600
@@
 F 0 "W103" H 4150 4770 50  0000 C CNN
 F 1 "SW_SPDT" H 4150 4400 50  0000 C CNN
-F 2 "" H 4150 4600 50  0001 C CNN
+F 2 "Connector_PinHeader_2.54mm:PinHeader_1x03_P2.54mm_Vertical" H 4150 4600 50  0001 C CNN
 F 3 "~" H 4150 4600 50  0001 C CNN
 	1    4150 4600
@@
 F 0 "W104" H 5650 4770 50  0000 C CNN
 F 1 "SW_SPDT" H 5650 4400 50  0000 C CNN
-F 2 "" H 5650 4600 50  0001 C CNN
+F 2 "Connector_PinHeader_2.54mm:PinHeader_1x03_P2.54mm_Vertical" H 5650 4600 50  0001 C CNN
 F 3 "~" H 5650 4600 50  0001 C CNN
 	1    5650 4600

Commit message: [PCB] continue footprint assignation
Parts:
- C113, C114: footprint (none) -> commons_passives_THT:Passive_THT_capacitor_mlcc_W2.54mm_L10.16mm
Changed lines of the file:
@@
 F 0 "C113" H 1425 3600 50  0000 L CNN
 F 1 "0.1uF" H 1425 3400 50  0000 L CNN
-F 2 "" H 1438 3350 50  0001 C CNN
+F 2 "commons_passives_THT:Passive_THT_capacitor_mlcc_W2.54mm_L10.16mm" H 1438 3350 50  0001 C CNN
 F 3 "~" H 1400 3500 50  0001 C CNN
 	1    1400 3500
@@
 F 0 "C114" H 6925 3600 50  0000 L CNN
 F 1 "0.1uF" H 6925 3400 50  0000 L CNN
-F 2 "" H 6938 3350 50  0001 C CNN
+F 2 "commons_passives_THT:Passive_THT_capacitor_mlcc_W2.54mm_L10.16mm" H 6938 3350 50  0001 C CNN
 F 3 "~" H 6900 3500 50  0001 C CNN
 	1    6900 3500
