File: atari-16-32-bits/motherboards/c300780-001/subsheet_401.sch (KiCad schematic (older format))
At the start: 16 parts, among them U401 STE_GSTSHIFTER_PHY

Commit message: [PCB] Assign builtins footprint when possible - resistors, ports
Parts:
- R411, R412, R414, R415, R416, R417, R418, R419, R422, R424, R426, R428, R430: footprint (none) -> Resistor_THT:R_Axial_DIN0204_L3.6mm_D1.6mm_P7.62mm_Horizontal
Changed lines of the file:
@@
 F 0 "R411" V 1400 7500 50  0000 C CNN
 F 1 "12K" V 1600 7500 50  0000 C CNN
-F 2 "" H 1500 7500 50  0001 C CNN
+F 2 "Resistor_THT:R_Axial_DIN0204_L3.6mm_D1.6mm_P7.62mm_Horizontal" H 1500 7500 50  0001 C CNN
 F 3 "~" H 1500 7500 50  0001 C CNN
 	1    1500 7500
@@
 F 0 "R412" V 1400 8000 50  0000 C CNN
 F 1 "1K5" V 1600 8000 50  0000 C CNN
-F 2 "" H 1500 8000 50  0001 C CNN
+F 2 "Resistor_THT:R_Axial_DIN0204_L3.6mm_D1.6mm_P7.62mm_Horizontal" H 1500 8000 50  0001 C CNN
 F 3 "~" H 1500 8000 50  0001 C CNN
 	1    1500 8000
@@
 F 0 "R414" V 1400 8500 50  0000 C CNN
 F 1 "3K" V 1600 8500 50  0000 C CNN
-F 2 "" H 1500 8500 50  0001 C CNN
+F 2 "Resistor_THT:R_Axial_DIN0204_L3.6mm_D1.6mm_P7.62mm_Horizontal" H 1500 8500 50  0001 C CNN
 F 3 "~" H 1500 8500 50  0001 C CNN
 	1    1500 8500
@@
 F 0 "R415" V 1400 9000 50  0000 C CNN
 F 1 "6K2" V 1600 9000 50  0000 C CNN
-F 2 "" H 1500 9000 50  0001 C CNN
+F 2 "Resistor_THT:R_Axial_DIN0204_L3.6mm_D1.6mm_P7.62mm_Horizontal" H 1500 9000 50  0001 C CNN
 F 3 "~" H 1500 9000 50  0001 C CNN
 	1    1500 9000
@@
 F 0 "R416" V 2900 7500 50  0000 C CNN
 F 1 "12K" V 3100 7500 50  0000 C CNN
-F 2 "" H 3000 7500 50  0001 C CNN
+F 2 "Resistor_THT:R_Axial_DIN0204_L3.6mm_D1.6mm_P7.62mm_Horizontal" H 3000 7500 50  0001 C CNN
 F 3 "~" H 3000 7500 50  0001 C CNN
 	1    3000 7500
@@
 F 0 "R417" V 2900 8000 50  0000 C CNN
 F 1 "1K5" V 3100 8000 50  0000 C CNN
-F 2 "" H 3000 8000 50  0001 C CNN
+F 2 "Resistor_THT:R_Axial_DIN0204_L3.6mm_D1.6mm_P7.62mm_Horizontal" H 3000 8000 50  0001 C CNN
 F 3 "~" H 3000 8000 50  0001 C CNN
 	1    3000 8000
@@
 F 0 "R418" V 2900 8500 50  0000 C CNN
 F 1 "3K" V 3100 8500 50  0000 C CNN
-F 2 "" H 3000 8500 50  0001 C CNN
+F 2 "Resistor_THT:R_Axial_DIN0204_L3.6mm_D1.6mm_P7.62mm_Horizontal" H 3000 8500 50  0001 C CNN
 F 3 "~" H 3000 8500 50  0001 C CNN
 	1    3000 8500
@@
 F 0 "R419" V 2900 9000 50  0000 C CNN
 F 1 "6K2" V 3100 9000 50  0000 C CNN
-F 2 "" H 3000 9000 50  0001 C CNN
+F 2 "Resistor_THT:R_Axial_DIN0204_L3.6mm_D1.6mm_P7.62mm_Horizontal" H 3000 9000 50  0001 C CNN
 F 3 "~" H 3000 9000 50  0001 C CNN
 	1    3000 9000
@@
 F 0 "R422" V 4400 7500 50  0000 C CNN
 F 1 "12K" V 4600 7500 50  0000 C CNN
-F 2 "" H 4500 7500 50  0001 C CNN
+F 2 "Resistor_THT:R_Axial_DIN0204_L3.6mm_D1.6mm_P7.62mm_Horizontal" H 4500 7500 50  0001 C CNN
 F 3 "~" H 4500 7500 50  0001 C CNN
 	1    4500 7500
@@
 F 0 "R424" V 4400 8000 50  0000 C CNN
 F 1 "1K5" V 4600 8000 50  0000 C CNN
-F 2 "" H 4500 8000 50  0001 C CNN
+F 2 "Resistor_THT:R_Axial_DIN0204_L3.6mm_D1.6mm_P7.62mm_Horizontal" H 4500 8000 50  0001 C CNN
 F 3 "~" H 4500 8000 50  0001 C CNN
 	1    4500 8000
@@
 F 0 "R426" V 4400 8500 50  0000 C CNN
 F 1 "3K" V 4600 8500 50  0000 C CNN
-F 2 "" H 4500 8500 50  0001 C CNN
+F 2 "Resistor_THT:R_Axial_DIN0204_L3.6mm_D1.6mm_P7.62mm_Horizontal" H 4500 8500 50  0001 C CNN
 F 3 "~" H 4500 8500 50  0001 C CNN
 	1    4500 8500
@@
 F 0 "R428" V 4400 9000 50  0000 C CNN
 F 1 "6K2" V 4600 9000 50  0000 C CNN
-F 2 "" H 4500 9000 50  0001 C CNN
+F 2 "Resistor_THT:R_Axial_DIN0204_L3.6mm_D1.6mm_P7.62mm_Horizontal" H 4500 9000 50  0001 C CNN
 F 3 "~" H 4500 9000 50  0001 C CNN
 	1    4500 9000
@@
 F 0 "R430" V 6000 7500 50  0000 C CNN
 F 1 "1K" V 6200 7500 50  0000 C CNN
-F 2 "" H 6100 7500 50  0001 C CNN
+F 2 "Resistor_THT:R_Axial_DIN0204_L3.6mm_D1.6mm_P7.62mm_Horizontal" H 6100 7500 50  0001 C CNN
 F 3 "~" H 6100 7500 50  0001 C CNN
 	1    6100 7500

Commit message: Resolves #41 : [PCB] custom footprint library for passives
Parts:
- R411, R412, R414, R415, R416, R417, R418, R419, R422, R424, R426, R428, R430: footprint Resistor_THT:R_Axial_DIN0204_L3.6mm_D1.6mm_P7.62mm_Horizontal -> commons_passives_THT:Passive_THT_resistor_W2.54mm_L12.70mm
Changed lines of the file:
@@
 F 0 "R411" V 1400 7500 50  0000 C CNN
 F 1 "12K" V 1600 7500 50  0000 C CNN
-F 2 "Resistor_THT:R_Axial_DIN0204_L3.6mm_D1.6mm_P7.62mm_Horizontal" H 1500 7500 50  0001 C CNN
+F 2 "commons_passives_THT:Passive_THT_resistor_W2.54mm_L12.70mm" H 1500 7500 50  0001 C CNN
 F 3 "~" H 1500 7500 50  0001 C CNN
 	1    1500 7500
@@
 F 0 "R412" V 1400 8000 50  0000 C CNN
 F 1 "1K5" V 1600 8000 50  0000 C CNN
-F 2 "Resistor_THT:R_Axial_DIN0204_L3.6mm_D1.6mm_P7.62mm_Horizontal" H 1500 8000 50  0001 C CNN
+F 2 "commons_passives_THT:Passive_THT_resistor_W2.54mm_L12.70mm" H 1500 8000 50  0001 C CNN
 F 3 "~" H 1500 8000 50  0001 C CNN
 	1    1500 8000
@@
 F 0 "R414" V 1400 8500 50  0000 C CNN
 F 1 "3K" V 1600 8500 50  0000 C CNN
-F 2 "Resistor_THT:R_Axial_DIN0204_L3.6mm_D1.6mm_P7.62mm_Horizontal" H 1500 8500 50  0001 C CNN
+F 2 "commons_passives_THT:Passive_THT_resistor_W2.54mm_L12.70mm" H 1500 8500 50  0001 C CNN
 F 3 "~" H 1500 8500 50  0001 C CNN
 	1    1500 8500
@@
 F 0 "R415" V 1400 9000 50  0000 C CNN
 F 1 "6K2" V 1600 9000 50  0000 C CNN
-F 2 "Resistor_THT:R_Axial_DIN0204_L3.6mm_D1.6mm_P7.62mm_Horizontal" H 1500 9000 50  0001 C CNN
+F 2 "commons_passives_THT:Passive_THT_resistor_W2.54mm_L12.70mm" H 1500 9000 50  0001 C CNN
 F 3 "~" H 1500 9000 50  0001 C CNN
 	1    1500 9000
@@
 F 0 "R416" V 2900 7500 50  0000 C CNN
 F 1 "12K" V 3100 7500 50  0000 C CNN
-F 2 "Resistor_THT:R_Axial_DIN0204_L3.6mm_D1.6mm_P7.62mm_Horizontal" H 3000 7500 50  0001 C CNN
+F 2 "commons_passives_THT:Passive_THT_resistor_W2.54mm_L12.70mm" H 3000 7500 50  0001 C CNN
 F 3 "~" H 3000 7500 50  0001 C CNN
 	1    3000 7500
@@
 F 0 "R417" V 2900 8000 50  0000 C CNN
 F 1 "1K5" V 3100 8000 50  0000 C CNN
-F 2 "Resistor_THT:R_Axial_DIN0204_L3.6mm_D1.6mm_P7.62mm_Horizontal" H 3000 8000 50  0001 C CNN
+F 2 "commons_passives_THT:Passive_THT_resistor_W2.54mm_L12.70mm" H 3000 8000 50  0001 C CNN
 F 3 "~" H 3000 8000 50  0001 C CNN
 	1    3000 8000
@@
 F 0 "R418" V 2900 8500 50  0000 C CNN
 F 1 "3K" V 3100 8500 50  0000 C CNN
-F 2 "Resistor_THT:R_Axial_DIN0204_L3.6mm_D1.6mm_P7.62mm_Horizontal" H 3000 8500 50  0001 C CNN
+F 2 "commons_passives_THT:Passive_THT_resistor_W2.54mm_L12.70mm" H 3000 8500 50  0001 C CNN
 F 3 "~" H 3000 8500 50  0001 C CNN
 	1    3000 8500
@@
 F 0 "R419" V 2900 9000 50  0000 C CNN
 F 1 "6K2" V 3100 9000 50  0000 C CNN
-F 2 "Resistor_THT:R_Axial_DIN0204_L3.6mm_D1.6mm_P7.62mm_Horizontal" H 3000 9000 50  0001 C CNN
+F 2 "commons_passives_THT:Passive_THT_resistor_W2.54mm_L12.70mm" H 3000 9000 50  0001 C CNN
 F 3 "~" H 3000 9000 50  0001 C CNN
 	1    3000 9000
@@
 F 0 "R422" V 4400 7500 50  0000 C CNN
 F 1 "12K" V 4600 7500 50  0000 C CNN
-F 2 "Resistor_THT:R_Axial_DIN0204_L3.6mm_D1.6mm_P7.62mm_Horizontal" H 4500 7500 50  0001 C CNN
+F 2 "commons_passives_THT:Passive_THT_resistor_W2.54mm_L12.70mm" H 4500 7500 50  0001 C CNN
 F 3 "~" H 4500 7500 50  0001 C CNN
 	1    4500 7500
@@
 F 0 "R424" V 4400 8000 50  0000 C CNN
 F 1 "1K5" V 4600 8000 50  0000 C CNN
-F 2 "Resistor_THT:R_Axial_DIN0204_L3.6mm_D1.6mm_P7.62mm_Horizontal" H 4500 8000 50  0001 C CNN
+F 2 "commons_passives_THT:Passive_THT_resistor_W2.54mm_L12.70mm" H 4500 8000 50  0001 C CNN
 F 3 "~" H 4500 8000 50  0001 C CNN
 	1    4500 8000
@@
 F 0 "R426" V 4400 8500 50  0000 C CNN
 F 1 "3K" V 4600 8500 50  0000 C CNN
-F 2 "Resistor_THT:R_Axial_DIN0204_L3.6mm_D1.6mm_P7.62mm_Horizontal" H 4500 8500 50  0001 C CNN
+F 2 "commons_passives_THT:Passive_THT_resistor_W2.54mm_L12.70mm" H 4500 8500 50  0001 C CNN
 F 3 "~" H 4500 8500 50  0001 C CNN
 	1    4500 8500
@@
 F 0 "R428" V 4400 9000 50  0000 C CNN
 F 1 "6K2" V 4600 9000 50  0000 C CNN
-F 2 "Resistor_THT:R_Axial_DIN0204_L3.6mm_D1.6mm_P7.62mm_Horizontal" H 4500 9000 50  0001 C CNN
+F 2 "commons_passives_THT:Passive_THT_resistor_W2.54mm_L12.70mm" H 4500 9000 50  0001 C CNN
 F 3 "~" H 4500 9000 50  0001 C CNN
 	1    4500 9000
@@
 F 0 "R430" V 6000 7500 50  0000 C CNN
 F 1 "1K" V 6200 7500 50  0000 C CNN
-F 2 "Resistor_THT:R_Axial_DIN0204_L3.6mm_D1.6mm_P7.62mm_Horizontal" H 6100 7500 50  0001 C CNN
+F 2 "commons_passives_THT:Passive_THT_resistor_W2.54mm_L12.70mm" H 6100 7500 50  0001 C CNN
 F 3 "~" H 6100 7500 50  0001 C CNN
 	1    6100 7500

Commit message: [PCB] continue footprint assignation
Parts:
- C412, C413: footprint (none) -> commons_passives_THT:Passive_THT_capacitor_ceramic_radial_W5.08mm_L6.35mm_X11.43mm
Changed lines of the file:
@@
 F 0 "C412" H 1275 5850 50  0000 L CNN
 F 1 "0.1uF" H 1275 5650 50  0000 L CNN
-F 2 "" H 1288 5600 50  0001 C CNN
+F 2 "commons_passives_THT:Passive_THT_capacitor_ceramic_radial_W5.08mm_L6.35mm_X11.43mm" H 1288 5600 50  0001 C CNN
 F 3 "~" H 1250 5750 50  0001 C CNN
 	1    1250 5750
@@
 F 0 "C413" H 1775 5850 50  0000 L CNN
 F 1 "0.1uF" H 1775 5650 50  0000 L CNN
-F 2 "" H 1788 5600 50  0001 C CNN
+F 2 "commons_passives_THT:Passive_THT_capacitor_ceramic_radial_W5.08mm_L6.35mm_X11.43mm" H 1788 5600 50  0001 C CNN
 F 3 "~" H 1750 5750 50  0001 C CNN
 	1    1750 5750
