File: atari-16-32-bits/motherboards/c300780-001/subsheet_205.sch (KiCad schematic (older format))
At the start: 23 parts, among them U204 TL497A_DIP-14_500MA_PEAK_STEP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, U205 TL497A_DIP-14_500MA_PEAK_STEP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

Commit message: [PCB] Assign builtins footprint when possible - resistors, ports
Parts:
- D200, D201, D203: footprint (none) -> Diode_THT:D_DO-35_SOD27_P7.62mm_Horizontal
- R203, R206, R208, R211, R213, R214: footprint (none) -> Resistor_THT:R_Axial_DIN0204_L3.6mm_D1.6mm_P7.62mm_Horizontal
Changed lines of the file:
@@
 F 0 "R208" V 4350 2500 50  0000 C CNN
 F 1 "1K2" V 4150 2500 50  0000 C CNN
-F 2 "" V 4290 2490 50  0001 C CNN
+F 2 "Resistor_THT:R_Axial_DIN0204_L3.6mm_D1.6mm_P7.62mm_Horizontal" V 4290 2490 50  0001 C CNN
 F 3 "~" H 4250 2500 50  0001 C CNN
 	1    4250 2500
@@
 F 0 "D201" V 4800 4250 50  0000 C CNN
 F 1 "1N914" V 4600 4250 50  0000 C CNN
-F 2 "" H 4700 4400 50  0001 C CNN
+F 2 "Diode_THT:D_DO-35_SOD27_P7.62mm_Horizontal" H 4700 4400 50  0001 C CNN
 F 3 "~" H 4700 4400 50  0001 C CNN
 	1    4700 4400
@@
 F 0 "D200" H 5100 4150 50  0000 C CNN
 F 1 "1N914" H 5100 3950 50  0000 C CNN
-F 2 "" H 5100 4050 50  0001 C CNN
+F 2 "Diode_THT:D_DO-35_SOD27_P7.62mm_Horizontal" H 5100 4050 50  0001 C CNN
 F 3 "~" H 5100 4050 50  0001 C CNN
 	1    5100 4050
@@
 F 0 "R206" V 5200 2500 50  0000 C CNN
 F 1 "12K" V 5000 2500 50  0000 C CNN
-F 2 "" V 5140 2490 50  0001 C CNN
+F 2 "Resistor_THT:R_Axial_DIN0204_L3.6mm_D1.6mm_P7.62mm_Horizontal" V 5140 2490 50  0001 C CNN
 F 3 "~" H 5100 2500 50  0001 C CNN
 	1    5100 2500
@@
 F 0 "R203" V 2700 4050 50  0000 C CNN
 F 1 "5.1" V 2500 4050 50  0000 C CNN
-F 2 "" V 2640 4040 50  0001 C CNN
+F 2 "Resistor_THT:R_Axial_DIN0204_L3.6mm_D1.6mm_P7.62mm_Horizontal" V 2640 4040 50  0001 C CNN
 F 3 "~" H 2600 4050 50  0001 C CNN
 	1    2600 4050
@@
 F 0 "R214" V 2700 7050 50  0000 C CNN
 F 1 "3K9" V 2500 7050 50  0000 C CNN
-F 2 "" V 2640 7040 50  0001 C CNN
+F 2 "Resistor_THT:R_Axial_DIN0204_L3.6mm_D1.6mm_P7.62mm_Horizontal" V 2640 7040 50  0001 C CNN
 F 3 "~" H 2600 7050 50  0001 C CNN
 	1    2600 7050
@@
 F 0 "R213" V 3550 7050 50  0000 C CNN
 F 1 "1K2" V 3350 7050 50  0000 C CNN
-F 2 "" V 3490 7040 50  0001 C CNN
+F 2 "Resistor_THT:R_Axial_DIN0204_L3.6mm_D1.6mm_P7.62mm_Horizontal" V 3490 7040 50  0001 C CNN
 F 3 "~" H 3450 7050 50  0001 C CNN
 	1    3450 7050
@@
 F 0 "R211" V 4250 5850 50  0000 C CNN
 F 1 "1" V 4050 5850 50  0000 C CNN
-F 2 "" V 4190 5840 50  0001 C CNN
+F 2 "Resistor_THT:R_Axial_DIN0204_L3.6mm_D1.6mm_P7.62mm_Horizontal" V 4190 5840 50  0001 C CNN
 F 3 "~" H 4150 5850 50  0001 C CNN
 	1    4150 5850
@@
 F 0 "D203" V 3900 6550 50  0000 C CNN
 F 1 "1N914" V 3700 6550 50  0000 C CNN
-F 2 "" H 3800 6700 50  0001 C CNN
+F 2 "Diode_THT:D_DO-35_SOD27_P7.62mm_Horizontal" H 3800 6700 50  0001 C CNN
 F 3 "~" H 3800 6700 50  0001 C CNN
 	1    3800 6700

Commit message: Resolves #41 : [PCB] custom footprint library for passives
Parts:
- D200, D201, D203: footprint Diode_THT:D_DO-35_SOD27_P7.62mm_Horizontal -> commons_passives_THT:Passive_THT_diode_W2.54mm_L12.70mm
- L203, L208: footprint (none) -> commons_passives_THT:Passive_THT_inductor_W5.08mm_L15.24mm
- R203, R206, R208, R211, R213, R214: footprint Resistor_THT:R_Axial_DIN0204_L3.6mm_D1.6mm_P7.62mm_Horizontal -> commons_passives_THT:Passive_THT_resistor_W2.54mm_L12.70mm
Changed lines of the file:
@@
 F 0 "R208" V 4350 2500 50  0000 C CNN
 F 1 "1K2" V 4150 2500 50  0000 C CNN
-F 2 "Resistor_THT:R_Axial_DIN0204_L3.6mm_D1.6mm_P7.62mm_Horizontal" V 4290 2490 50  0001 C CNN
+F 2 "commons_passives_THT:Passive_THT_resistor_W2.54mm_L12.70mm" V 4290 2490 50  0001 C CNN
 F 3 "~" H 4250 2500 50  0001 C CNN
 	1    4250 2500
@@
 F 0 "D201" V 4800 4250 50  0000 C CNN
 F 1 "1N914" V 4600 4250 50  0000 C CNN
-F 2 "Diode_THT:D_DO-35_SOD27_P7.62mm_Horizontal" H 4700 4400 50  0001 C CNN
+F 2 "commons_passives_THT:Passive_THT_diode_W2.54mm_L12.70mm" H 4700 4400 50  0001 C CNN
 F 3 "~" H 4700 4400 50  0001 C CNN
 	1    4700 4400
@@
 F 0 "D200" H 5100 4150 50  0000 C CNN
 F 1 "1N914" H 5100 3950 50  0000 C CNN
-F 2 "Diode_THT:D_DO-35_SOD27_P7.62mm_Horizontal" H 5100 4050 50  0001 C CNN
+F 2 "commons_passives_THT:Passive_THT_diode_W2.54mm_L12.70mm" H 5100 4050 50  0001 C CNN
 F 3 "~" H 5100 4050 50  0001 C CNN
 	1    5100 4050
@@
 F 0 "R206" V 5200 2500 50  0000 C CNN
 F 1 "12K" V 5000 2500 50  0000 C CNN
-F 2 "Resistor_THT:R_Axial_DIN0204_L3.6mm_D1.6mm_P7.62mm_Horizontal" V 5140 2490 50  0001 C CNN
+F 2 "commons_passives_THT:Passive_THT_resistor_W2.54mm_L12.70mm" V 5140 2490 50  0001 C CNN
 F 3 "~" H 5100 2500 50  0001 C CNN
 	1    5100 2500
@@
 F 0 "R203" V 2700 4050 50  0000 C CNN
 F 1 "5.1" V 2500 4050 50  0000 C CNN
-F 2 "Resistor_THT:R_Axial_DIN0204_L3.6mm_D1.6mm_P7.62mm_Horizontal" V 2640 4040 50  0001 C CNN
+F 2 "commons_passives_THT:Passive_THT_resistor_W2.54mm_L12.70mm" V 2640 4040 50  0001 C CNN
 F 3 "~" H 2600 4050 50  0001 C CNN
 	1    2600 4050
@@
 F 0 "L203" V 3400 4050 50  0000 C CNN
 F 1 "220uH" V 3525 4050 50  0000 C CNN
-F 2 "" H 3450 4050 50  0001 C CNN
+F 2 "commons_passives_THT:Passive_THT_inductor_W5.08mm_L15.24mm" H 3450 4050 50  0001 C CNN
 F 3 "~" H 3450 4050 50  0001 C CNN
 	1    3450 4050
@@
 F 0 "R214" V 2700 7050 50  0000 C CNN
 F 1 "3K9" V 2500 7050 50  0000 C CNN
-F 2 "Resistor_THT:R_Axial_DIN0204_L3.6mm_D1.6mm_P7.62mm_Horizontal" V 2640 7040 50  0001 C CNN
+F 2 "commons_passives_THT:Passive_THT_resistor_W2.54mm_L12.70mm" V 2640 7040 50  0001 C CNN
 F 3 "~" H 2600 7050 50  0001 C CNN
 	1    2600 7050
@@
 F 0 "R213" V 3550 7050 50  0000 C CNN
 F 1 "1K2" V 3350 7050 50  0000 C CNN
-F 2 "Resistor_THT:R_Axial_DIN0204_L3.6mm_D1.6mm_P7.62mm_Horizontal" V 3490 7040 50  0001 C CNN
+F 2 "commons_passives_THT:Passive_THT_resistor_W2.54mm_L12.70mm" V 3490 7040 50  0001 C CNN
 F 3 "~" H 3450 7050 50  0001 C CNN
 	1    3450 7050
@@
 F 0 "R211" V 4250 5850 50  0000 C CNN
 F 1 "1" V 4050 5850 50  0000 C CNN
-F 2 "Resistor_THT:R_Axial_DIN0204_L3.6mm_D1.6mm_P7.62mm_Horizontal" V 4190 5840 50  0001 C CNN
+F 2 "commons_passives_THT:Passive_THT_resistor_W2.54mm_L12.70mm" V 4190 5840 50  0001 C CNN
 F 3 "~" H 4150 5850 50  0001 C CNN
 	1    4150 5850
@@
 F 0 "L208" V 4100 6350 50  0000 C CNN
 F 1 "220uH" V 4225 6350 50  0000 C CNN
-F 2 "" H 4150 6350 50  0001 C CNN
+F 2 "commons_passives_THT:Passive_THT_inductor_W5.08mm_L15.24mm" H 4150 6350 50  0001 C CNN
 F 3 "~" H 4150 6350 50  0001 C CNN
 	1    4150 6350
@@
 F 0 "D203" V 3900 6550 50  0000 C CNN
 F 1 "1N914" V 3700 6550 50  0000 C CNN
-F 2 "Diode_THT:D_DO-35_SOD27_P7.62mm_Horizontal" H 3800 6700 50  0001 C CNN
+F 2 "commons_passives_THT:Passive_THT_diode_W2.54mm_L12.70mm" H 3800 6700 50  0001 C CNN
 F 3 "~" H 3800 6700 50  0001 C CNN
 	1    3800 6700

Commit message: [PCB] continue footprint assignation
Parts:
- C202, C204, C205, C215: footprint (none) -> commons_passives_THT:Passive_THT_capacitor_polarized_W5.08mm_L17.78mm
- C207, C217: footprint (none) -> commons_passives_THT:Passive_THT_capacitor_ceramic_radial_W5.08mm_L6.35mm_X11.43mm
- C208, C209, C218: footprint (none) -> commons_passives_THT:Passive_THT_capacitor_W2.54mm_L10.16mm
Changed lines of the file:
@@
 F 0 "C207" H 5425 1700 50  0000 L CNN
 F 1 "0.1uF" H 5425 1500 50  0000 L CNN
-F 2 "" H 5438 1450 50  0001 C CNN
+F 2 "commons_passives_THT:Passive_THT_capacitor_ceramic_radial_W5.08mm_L6.35mm_X11.43mm" H 5438 1450 50  0001 C CNN
 F 3 "~" H 5400 1600 50  0001 C CNN
 	1    5400 1600
@@
 F 0 "C209" H 5925 1700 50  0000 L CNN
 F 1 "330pF" H 5925 1500 50  0000 L CNN
-F 2 "" H 5938 1450 50  0001 C CNN
+F 2 "commons_passives_THT:Passive_THT_capacitor_W2.54mm_L10.16mm" H 5938 1450 50  0001 C CNN
 F 3 "~" H 5900 1600 50  0001 C CNN
 	1    5900 1600
@@
 F 0 "C205" H 5475 2950 50  0000 L CNN
 F 1 "4.7uF" H 5475 2750 50  0000 L CNN
-F 2 "" H 5450 2850 50  0001 C CNN
+F 2 "commons_passives_THT:Passive_THT_capacitor_polarized_W5.08mm_L17.78mm" H 5450 2850 50  0001 C CNN
 F 3 "~" H 5450 2850 50  0001 C CNN
 	1    5450 2850
@@
 F 0 "C204" H 5475 3800 50  0000 L CNN
 F 1 "4.7uF" H 5475 3600 50  0000 L CNN
-F 2 "" H 5450 3700 50  0001 C CNN
+F 2 "commons_passives_THT:Passive_THT_capacitor_polarized_W5.08mm_L17.78mm" H 5450 3700 50  0001 C CNN
 F 3 "~" H 5450 3700 50  0001 C CNN
 	1    5450 3700
@@
 F 0 "C202" V 4200 4000 50  0000 L CNN
 F 1 "4.7uF" V 4500 3950 50  0000 L CNN
-F 2 "" H 4350 4050 50  0001 C CNN
+F 2 "commons_passives_THT:Passive_THT_capacitor_polarized_W5.08mm_L17.78mm" H 4350 4050 50  0001 C CNN
 F 3 "~" H 4350 4050 50  0001 C CNN
 	1    4350 4050
@@
 F 0 "C208" H 2975 4500 50  0000 L CNN
 F 1 "150pF" H 2975 4300 50  0000 L CNN
-F 2 "" H 2988 4250 50  0001 C CNN
+F 2 "commons_passives_THT:Passive_THT_capacitor_W2.54mm_L10.16mm" H 2988 4250 50  0001 C CNN
 F 3 "~" H 2950 4400 50  0001 C CNN
 	1    2950 4400
@@
 F 0 "C217" H 6275 6350 50  0000 L CNN
 F 1 "0.1uF" H 6275 6150 50  0000 L CNN
-F 2 "" H 6288 6100 50  0001 C CNN
+F 2 "commons_passives_THT:Passive_THT_capacitor_ceramic_radial_W5.08mm_L6.35mm_X11.43mm" H 6288 6100 50  0001 C CNN
 F 3 "~" H 6250 6250 50  0001 C CNN
 	1    6250 6250
@@
 F 0 "C218" H 6775 6350 50  0000 L CNN
 F 1 "270pF" H 6775 6150 50  0000 L CNN
-F 2 "" H 6788 6100 50  0001 C CNN
+F 2 "commons_passives_THT:Passive_THT_capacitor_W2.54mm_L10.16mm" H 6788 6100 50  0001 C CNN
 F 3 "~" H 6750 6250 50  0001 C CNN
 	1    6750 6250
@@
 F 0 "C215" H 5275 6350 50  0000 L CNN
 F 1 "4.7uF" H 5275 6150 50  0000 L CNN
-F 2 "" H 5250 6250 50  0001 C CNN
+F 2 "commons_passives_THT:Passive_THT_capacitor_polarized_W5.08mm_L17.78mm" H 5250 6250 50  0001 C CNN
 F 3 "~" H 5250 6250 50  0001 C CNN
 	1    5250 6250

Commit message: [PCB] continue footprints assignements
Parts:
- C216: footprint (none) -> commons_passives_THT:Passive_THT_capacitor_polarized_W10.16mm_L27.94mm
Changed lines of the file:
@@
 F 0 "C216" H 5775 6350 50  0000 L CNN
 F 1 "470uF" H 5775 6150 50  0000 L CNN
-F 2 "" H 5750 6250 50  0001 C CNN
+F 2 "commons_passives_THT:Passive_THT_capacitor_polarized_W10.16mm_L27.94mm" H 5750 6250 50  0001 C CNN
 F 3 "~" H 5750 6250 50  0001 C CNN
 	1    5750 6250
