File: atari-16-32-bits/motherboards/c300780-001/subsheet_502.sch (KiCad schematic (older format))
At the start: 26 parts, among them U500 74F374_OCTAL_D-TYPE_EDGE-TRIG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, U501 74F374_OCTAL_D-TYPE_EDGE-TRIG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, U502 DAC0802LCN_PHY, U503 DAC0802LCN_PHY

Commit message: [PCB] Assign builtins footprint when possible - resistors, ports
Parts:
- R500, R505, R506, R508, R509, R514, R515, R517, R542, R543: footprint (none) -> Resistor_THT:R_Axial_DIN0204_L3.6mm_D1.6mm_P7.62mm_Horizontal
Changed lines of the file:
@@
 F 0 "R542" V 1800 1500 50  0000 C CNN
 F 1 "10" V 2000 1500 50  0000 C CNN
-F 2 "" H 1900 1500 50  0001 C CNN
+F 2 "Resistor_THT:R_Axial_DIN0204_L3.6mm_D1.6mm_P7.62mm_Horizontal" H 1900 1500 50  0001 C CNN
 F 3 "~" H 1900 1500 50  0001 C CNN
 	1    1900 1500
@@
 F 0 "R543" V 4800 1500 50  0000 C CNN
 F 1 "10" V 5000 1500 50  0000 C CNN
-F 2 "" H 4900 1500 50  0001 C CNN
+F 2 "Resistor_THT:R_Axial_DIN0204_L3.6mm_D1.6mm_P7.62mm_Horizontal" H 4900 1500 50  0001 C CNN
 F 3 "~" H 4900 1500 50  0001 C CNN
 	1    4900 1500
@@
 F 0 "R505" H 2100 5450 50  0000 L CNN
 F 1 "10K" H 2150 5350 50  0000 L CNN
-F 2 "" H 2350 5400 50  0001 C CNN
+F 2 "Resistor_THT:R_Axial_DIN0204_L3.6mm_D1.6mm_P7.62mm_Horizontal" H 2350 5400 50  0001 C CNN
 F 3 "~" H 2350 5400 50  0001 C CNN
 	1    2350 5400
@@
 F 0 "R506" H 1300 5950 50  0000 L CNN
 F 1 "10K" H 1300 5850 50  0000 L CNN
-F 2 "" H 1250 5900 50  0001 C CNN
+F 2 "Resistor_THT:R_Axial_DIN0204_L3.6mm_D1.6mm_P7.62mm_Horizontal" H 1250 5900 50  0001 C CNN
 F 3 "~" H 1250 5900 50  0001 C CNN
 	1    1250 5900
@@
 F 0 "R500" H 2200 8550 50  0000 L CNN
 F 1 "8K2" H 2250 8650 50  0000 L CNN
-F 2 "" H 2450 8600 50  0001 C CNN
+F 2 "Resistor_THT:R_Axial_DIN0204_L3.6mm_D1.6mm_P7.62mm_Horizontal" H 2450 8600 50  0001 C CNN
 F 3 "~" H 2450 8600 50  0001 C CNN
 	1    2450 8600
@@
 F 0 "R508" H 2350 8550 50  0000 L CNN
 F 1 "8K2" H 2350 8650 50  0000 L CNN
-F 2 "" H 2250 8600 50  0001 C CNN
+F 2 "Resistor_THT:R_Axial_DIN0204_L3.6mm_D1.6mm_P7.62mm_Horizontal" H 2250 8600 50  0001 C CNN
 F 3 "~" H 2250 8600 50  0001 C CNN
 	1    2250 8600
@@
 F 0 "R514" H 5600 5450 50  0000 L CNN
 F 1 "10K" H 5650 5350 50  0000 L CNN
-F 2 "" H 5850 5400 50  0001 C CNN
+F 2 "Resistor_THT:R_Axial_DIN0204_L3.6mm_D1.6mm_P7.62mm_Horizontal" H 5850 5400 50  0001 C CNN
 F 3 "~" H 5850 5400 50  0001 C CNN
 	1    5850 5400
@@
 F 0 "R515" H 4800 5950 50  0000 L CNN
 F 1 "10K" H 4800 5850 50  0000 L CNN
-F 2 "" H 4750 5900 50  0001 C CNN
+F 2 "Resistor_THT:R_Axial_DIN0204_L3.6mm_D1.6mm_P7.62mm_Horizontal" H 4750 5900 50  0001 C CNN
 F 3 "~" H 4750 5900 50  0001 C CNN
 	1    4750 5900
@@
 F 0 "R509" H 5700 8550 50  0000 L CNN
 F 1 "8K2" H 5750 8650 50  0000 L CNN
-F 2 "" H 5950 8600 50  0001 C CNN
+F 2 "Resistor_THT:R_Axial_DIN0204_L3.6mm_D1.6mm_P7.62mm_Horizontal" H 5950 8600 50  0001 C CNN
 F 3 "~" H 5950 8600 50  0001 C CNN
 	1    5950 8600
@@
 F 0 "R517" H 5800 8550 50  0000 L CNN
 F 1 "8K2" H 5800 8650 50  0000 L CNN
-F 2 "" H 5750 8600 50  0001 C CNN
+F 2 "Resistor_THT:R_Axial_DIN0204_L3.6mm_D1.6mm_P7.62mm_Horizontal" H 5750 8600 50  0001 C CNN
 F 3 "~" H 5750 8600 50  0001 C CNN
 	1    5750 8600

Commit message: Resolves #41 : [PCB] custom footprint library for passives
Parts:
- R500, R505, R506, R508, R509, R514, R515, R517, R542, R543: footprint Resistor_THT:R_Axial_DIN0204_L3.6mm_D1.6mm_P7.62mm_Horizontal -> commons_passives_THT:Passive_THT_resistor_W2.54mm_L12.70mm
Changed lines of the file:
@@
 F 0 "R542" V 1800 1500 50  0000 C CNN
 F 1 "10" V 2000 1500 50  0000 C CNN
-F 2 "Resistor_THT:R_Axial_DIN0204_L3.6mm_D1.6mm_P7.62mm_Horizontal" H 1900 1500 50  0001 C CNN
+F 2 "commons_passives_THT:Passive_THT_resistor_W2.54mm_L12.70mm" H 1900 1500 50  0001 C CNN
 F 3 "~" H 1900 1500 50  0001 C CNN
 	1    1900 1500
@@
 F 0 "R543" V 4800 1500 50  0000 C CNN
 F 1 "10" V 5000 1500 50  0000 C CNN
-F 2 "Resistor_THT:R_Axial_DIN0204_L3.6mm_D1.6mm_P7.62mm_Horizontal" H 4900 1500 50  0001 C CNN
+F 2 "commons_passives_THT:Passive_THT_resistor_W2.54mm_L12.70mm" H 4900 1500 50  0001 C CNN
 F 3 "~" H 4900 1500 50  0001 C CNN
 	1    4900 1500
@@
 F 0 "R505" H 2100 5450 50  0000 L CNN
 F 1 "10K" H 2150 5350 50  0000 L CNN
-F 2 "Resistor_THT:R_Axial_DIN0204_L3.6mm_D1.6mm_P7.62mm_Horizontal" H 2350 5400 50  0001 C CNN
+F 2 "commons_passives_THT:Passive_THT_resistor_W2.54mm_L12.70mm" H 2350 5400 50  0001 C CNN
 F 3 "~" H 2350 5400 50  0001 C CNN
 	1    2350 5400
@@
 F 0 "R506" H 1300 5950 50  0000 L CNN
 F 1 "10K" H 1300 5850 50  0000 L CNN
-F 2 "Resistor_THT:R_Axial_DIN0204_L3.6mm_D1.6mm_P7.62mm_Horizontal" H 1250 5900 50  0001 C CNN
+F 2 "commons_passives_THT:Passive_THT_resistor_W2.54mm_L12.70mm" H 1250 5900 50  0001 C CNN
 F 3 "~" H 1250 5900 50  0001 C CNN
 	1    1250 5900
@@
 F 0 "R500" H 2200 8550 50  0000 L CNN
 F 1 "8K2" H 2250 8650 50  0000 L CNN
-F 2 "Resistor_THT:R_Axial_DIN0204_L3.6mm_D1.6mm_P7.62mm_Horizontal" H 2450 8600 50  0001 C CNN
+F 2 "commons_passives_THT:Passive_THT_resistor_W2.54mm_L12.70mm" H 2450 8600 50  0001 C CNN
 F 3 "~" H 2450 8600 50  0001 C CNN
 	1    2450 8600
@@
 F 0 "R508" H 2350 8550 50  0000 L CNN
 F 1 "8K2" H 2350 8650 50  0000 L CNN
-F 2 "Resistor_THT:R_Axial_DIN0204_L3.6mm_D1.6mm_P7.62mm_Horizontal" H 2250 8600 50  0001 C CNN
+F 2 "commons_passives_THT:Passive_THT_resistor_W2.54mm_L12.70mm" H 2250 8600 50  0001 C CNN
 F 3 "~" H 2250 8600 50  0001 C CNN
 	1    2250 8600
@@
 F 0 "R514" H 5600 5450 50  0000 L CNN
 F 1 "10K" H 5650 5350 50  0000 L CNN
-F 2 "Resistor_THT:R_Axial_DIN0204_L3.6mm_D1.6mm_P7.62mm_Horizontal" H 5850 5400 50  0001 C CNN
+F 2 "commons_passives_THT:Passive_THT_resistor_W2.54mm_L12.70mm" H 5850 5400 50  0001 C CNN
 F 3 "~" H 5850 5400 50  0001 C CNN
 	1    5850 5400
@@
 F 0 "R515" H 4800 5950 50  0000 L CNN
 F 1 "10K" H 4800 5850 50  0000 L CNN
-F 2 "Resistor_THT:R_Axial_DIN0204_L3.6mm_D1.6mm_P7.62mm_Horizontal" H 4750 5900 50  0001 C CNN
+F 2 "commons_passives_THT:Passive_THT_resistor_W2.54mm_L12.70mm" H 4750 5900 50  0001 C CNN
 F 3 "~" H 4750 5900 50  0001 C CNN
 	1    4750 5900
@@
 F 0 "R509" H 5700 8550 50  0000 L CNN
 F 1 "8K2" H 5750 8650 50  0000 L CNN
-F 2 "Resistor_THT:R_Axial_DIN0204_L3.6mm_D1.6mm_P7.62mm_Horizontal" H 5950 8600 50  0001 C CNN
+F 2 "commons_passives_THT:Passive_THT_resistor_W2.54mm_L12.70mm" H 5950 8600 50  0001 C CNN
 F 3 "~" H 5950 8600 50  0001 C CNN
 	1    5950 8600
@@
 F 0 "R517" H 5800 8550 50  0000 L CNN
 F 1 "8K2" H 5800 8650 50  0000 L CNN
-F 2 "Resistor_THT:R_Axial_DIN0204_L3.6mm_D1.6mm_P7.62mm_Horizontal" H 5750 8600 50  0001 C CNN
+F 2 "commons_passives_THT:Passive_THT_resistor_W2.54mm_L12.70mm" H 5750 8600 50  0001 C CNN
 F 3 "~" H 5750 8600 50  0001 C CNN
 	1    5750 8600

Commit message: [PCB] continue footprint assignation
Parts:
- C504, C507, C516, C519, C556, C557, C559, C562: footprint (none) -> commons_passives_THT:Passive_THT_capacitor_ceramic_radial_W5.08mm_L6.35mm_X11.43mm
Changed lines of the file:
@@
 F 0 "C559" H 2925 1850 50  0000 L CNN
 F 1 "0.1uF" H 2925 1650 50  0000 L CNN
-F 2 "" H 2938 1600 50  0001 C CNN
+F 2 "commons_passives_THT:Passive_THT_capacitor_ceramic_radial_W5.08mm_L6.35mm_X11.43mm" H 2938 1600 50  0001 C CNN
 F 3 "~" H 2900 1750 50  0001 C CNN
 	1    2900 1750
@@
 F 0 "C562" H 5925 1850 50  0000 L CNN
 F 1 "0.1uF" H 5925 1650 50  0000 L CNN
-F 2 "" H 5938 1600 50  0001 C CNN
+F 2 "commons_passives_THT:Passive_THT_capacitor_ceramic_radial_W5.08mm_L6.35mm_X11.43mm" H 5938 1600 50  0001 C CNN
 F 3 "~" H 5900 1750 50  0001 C CNN
 	1    5900 1750
@@
 F 0 "C507" H 3475 6600 50  0000 L CNN
 F 1 "0.1uF" H 3475 6400 50  0000 L CNN
-F 2 "" H 3488 6350 50  0001 C CNN
+F 2 "commons_passives_THT:Passive_THT_capacitor_ceramic_radial_W5.08mm_L6.35mm_X11.43mm" H 3488 6350 50  0001 C CNN
 F 3 "~" H 3450 6500 50  0001 C CNN
 	1    3450 6500
@@
 F 0 "C504" H 3475 7200 50  0000 L CNN
 F 1 "0.1uF" H 3475 7000 50  0000 L CNN
-F 2 "" H 3488 6950 50  0001 C CNN
+F 2 "commons_passives_THT:Passive_THT_capacitor_ceramic_radial_W5.08mm_L6.35mm_X11.43mm" H 3488 6950 50  0001 C CNN
 F 3 "~" H 3450 7100 50  0001 C CNN
 	1    3450 7100
@@
 F 0 "C556" H 1025 4100 50  0000 L CNN
 F 1 "0.1uF" H 1025 3900 50  0000 L CNN
-F 2 "" H 1038 3850 50  0001 C CNN
+F 2 "commons_passives_THT:Passive_THT_capacitor_ceramic_radial_W5.08mm_L6.35mm_X11.43mm" H 1038 3850 50  0001 C CNN
 F 3 "~" H 1000 4000 50  0001 C CNN
 	1    1000 4000
@@
 F 0 "C519" H 6975 6600 50  0000 L CNN
 F 1 "0.1uF" H 6975 6400 50  0000 L CNN
-F 2 "" H 6988 6350 50  0001 C CNN
+F 2 "commons_passives_THT:Passive_THT_capacitor_ceramic_radial_W5.08mm_L6.35mm_X11.43mm" H 6988 6350 50  0001 C CNN
 F 3 "~" H 6950 6500 50  0001 C CNN
 	1    6950 6500
@@
 F 0 "C516" H 6975 7200 50  0000 L CNN
 F 1 "0.1uF" H 6975 7000 50  0000 L CNN
-F 2 "" H 6988 6950 50  0001 C CNN
+F 2 "commons_passives_THT:Passive_THT_capacitor_ceramic_radial_W5.08mm_L6.35mm_X11.43mm" H 6988 6950 50  0001 C CNN
 F 3 "~" H 6950 7100 50  0001 C CNN
 	1    6950 7100
@@
 F 0 "C557" H 7275 4100 50  0000 L CNN
 F 1 "0.1uF" H 7275 3900 50  0000 L CNN
-F 2 "" H 7288 3850 50  0001 C CNN
+F 2 "commons_passives_THT:Passive_THT_capacitor_ceramic_radial_W5.08mm_L6.35mm_X11.43mm" H 7288 3850 50  0001 C CNN
 F 3 "~" H 7250 4000 50  0001 C CNN
 	1    7250 4000

Commit message: [PCB] continue assigning footprints - done all fixed capacitors
Parts:
- C503, C515: footprint (none) -> commons_passives_THT:Passive_THT_capacitor_W2.54mm_L10.16mm
- C558, C561: footprint (none) -> commons_passives_THT:Passive_THT_capacitor_polarized_W6.35mm_L20.32mm
Changed lines of the file:
@@
 F 0 "C558" H 2425 1850 50  0000 L CNN
 F 1 "100uF" H 2425 1650 50  0000 L CNN
-F 2 "" H 2400 1750 50  0001 C CNN
+F 2 "commons_passives_THT:Passive_THT_capacitor_polarized_W6.35mm_L20.32mm" H 2400 1750 50  0001 C CNN
 F 3 "~" H 2400 1750 50  0001 C CNN
 	1    2400 1750
@@
 F 0 "C561" H 5425 1850 50  0000 L CNN
 F 1 "100uF" H 5425 1650 50  0000 L CNN
-F 2 "" H 5400 1750 50  0001 C CNN
+F 2 "commons_passives_THT:Passive_THT_capacitor_polarized_W6.35mm_L20.32mm" H 5400 1750 50  0001 C CNN
 F 3 "~" H 5400 1750 50  0001 C CNN
 	1    5400 1750
@@
 F 0 "C503" H 1675 6000 50  0000 L CNN
 F 1 "0.01uF" H 1675 5800 50  0000 L CNN
-F 2 "" H 1688 5750 50  0001 C CNN
+F 2 "commons_passives_THT:Passive_THT_capacitor_W2.54mm_L10.16mm" H 1688 5750 50  0001 C CNN
 F 3 "~" H 1650 5900 50  0001 C CNN
 	1    1650 5900
@@
 F 0 "C515" H 5175 6000 50  0000 L CNN
 F 1 "0.01uF" H 5175 5800 50  0000 L CNN
-F 2 "" H 5188 5750 50  0001 C CNN
+F 2 "commons_passives_THT:Passive_THT_capacitor_W2.54mm_L10.16mm" H 5188 5750 50  0001 C CNN
 F 3 "~" H 5150 5900 50  0001 C CNN
 	1    5150 5900
