File: atari-16-32-bits/motherboards/c300780-001/subsheet_503.sch (KiCad schematic (older format))
At the start: 39 parts, among them Q500 LM78L82_TO92, U504 LF347N_mu, U505 MF4CN-100_PHY, U506 MF4CN-100_PHY, U507 LF347N_mu

Commit message: [PCB] Assign builtins footprint when possible - resistors, ports
Parts:
- R501, R502, R503, R504, R507, R510, R511, R512, R513, R516, R545, R546: footprint (none) -> Resistor_THT:R_Axial_DIN0204_L3.6mm_D1.6mm_P7.62mm_Horizontal
Changed lines of the file:
@@
 F 0 "R545" H 3880 2570 50  0000 L CNN
 F 1 "100K" H 3880 2510 50  0000 L CNN
-F 2 "" H 3850 2550 50  0001 C CNN
+F 2 "Resistor_THT:R_Axial_DIN0204_L3.6mm_D1.6mm_P7.62mm_Horizontal" H 3850 2550 50  0001 C CNN
 F 3 "~" H 3850 2550 50  0001 C CNN
 	1    3850 2550
@@
 F 0 "R546" H 7230 3420 50  0000 L CNN
 F 1 "100K" H 7230 3360 50  0000 L CNN
-F 2 "" H 7200 3400 50  0001 C CNN
+F 2 "Resistor_THT:R_Axial_DIN0204_L3.6mm_D1.6mm_P7.62mm_Horizontal" H 7200 3400 50  0001 C CNN
 F 3 "~" H 7200 3400 50  0001 C CNN
 	1    7200 3400
@@
 F 0 "R513" H 6850 5350 50  0000 C CNN
 F 1 "10K" H 6850 5450 50  0000 C CNN
-F 2 "" H 7000 5400 50  0001 C CNN
+F 2 "Resistor_THT:R_Axial_DIN0204_L3.6mm_D1.6mm_P7.62mm_Horizontal" H 7000 5400 50  0001 C CNN
 F 3 "~" H 7000 5400 50  0001 C CNN
 	1    7000 5400
@@
 F 0 "R511" V 7150 5900 50  0000 L CNN
 F 1 "10K" V 7350 5900 50  0000 L CNN
-F 2 "" H 7250 6000 50  0001 C CNN
+F 2 "Resistor_THT:R_Axial_DIN0204_L3.6mm_D1.6mm_P7.62mm_Horizontal" H 7250 6000 50  0001 C CNN
 F 3 "~" H 7250 6000 50  0001 C CNN
 	1    7250 6000
@@
 F 0 "R512" H 6350 3700 50  0000 C CNN
 F 1 "10K" H 6350 3800 50  0000 C CNN
-F 2 "" H 6500 3750 50  0001 C CNN
+F 2 "Resistor_THT:R_Axial_DIN0204_L3.6mm_D1.6mm_P7.62mm_Horizontal" H 6500 3750 50  0001 C CNN
 F 3 "~" H 6500 3750 50  0001 C CNN
 	1    6500 3750
@@
 F 0 "R510" V 6650 4150 50  0000 L CNN
 F 1 "10K" H 6780 4210 50  0000 L CNN
-F 2 "" H 6750 4250 50  0001 C CNN
+F 2 "Resistor_THT:R_Axial_DIN0204_L3.6mm_D1.6mm_P7.62mm_Horizontal" H 6750 4250 50  0001 C CNN
 F 3 "~" H 6750 4250 50  0001 C CNN
 	1    6750 4250
@@
 F 0 "R516" V 6650 5550 50  0000 L CNN
 F 1 "1K8" V 6850 5550 50  0000 L CNN
-F 2 "" H 6750 5650 50  0001 C CNN
+F 2 "Resistor_THT:R_Axial_DIN0204_L3.6mm_D1.6mm_P7.62mm_Horizontal" H 6750 5650 50  0001 C CNN
 F 3 "~" H 6750 5650 50  0001 C CNN
 	1    6750 5650
@@
 F 0 "R504" H 3500 4350 50  0000 C CNN
 F 1 "10K" H 3500 4450 50  0000 C CNN
-F 2 "" H 3650 4400 50  0001 C CNN
+F 2 "Resistor_THT:R_Axial_DIN0204_L3.6mm_D1.6mm_P7.62mm_Horizontal" H 3650 4400 50  0001 C CNN
 F 3 "~" H 3650 4400 50  0001 C CNN
 	1    3650 4400
@@
 F 0 "R502" V 3800 4950 50  0000 L CNN
 F 1 "10K" V 4000 4950 50  0000 L CNN
-F 2 "" H 3900 5050 50  0001 C CNN
+F 2 "Resistor_THT:R_Axial_DIN0204_L3.6mm_D1.6mm_P7.62mm_Horizontal" H 3900 5050 50  0001 C CNN
 F 3 "~" H 3900 5050 50  0001 C CNN
 	1    3900 5050
@@
 F 0 "R503" H 3000 2850 50  0000 C CNN
 F 1 "10K" H 3000 2950 50  0000 C CNN
-F 2 "" H 3150 2900 50  0001 C CNN
+F 2 "Resistor_THT:R_Axial_DIN0204_L3.6mm_D1.6mm_P7.62mm_Horizontal" H 3150 2900 50  0001 C CNN
 F 3 "~" H 3150 2900 50  0001 C CNN
 	1    3150 2900
@@
 F 0 "R501" V 3300 3200 50  0000 L CNN
 F 1 "10K" V 3500 3200 50  0000 L CNN
-F 2 "" H 3400 3300 50  0001 C CNN
+F 2 "Resistor_THT:R_Axial_DIN0204_L3.6mm_D1.6mm_P7.62mm_Horizontal" H 3400 3300 50  0001 C CNN
 F 3 "~" H 3400 3300 50  0001 C CNN
 	1    3400 3300
@@
 F 0 "R507" V 3300 4600 50  0000 L CNN
 F 1 "1K8" V 3500 4600 50  0000 L CNN
-F 2 "" H 3400 4700 50  0001 C CNN
+F 2 "Resistor_THT:R_Axial_DIN0204_L3.6mm_D1.6mm_P7.62mm_Horizontal" H 3400 4700 50  0001 C CNN
 F 3 "~" H 3400 4700 50  0001 C CNN
 	1    3400 4700

Commit message: [PCB] continuing footprint assignement
Parts:
- Q500: footprint Package_TO_SOT_THT:TO-92_Inline -> Package_TO_SOT_THT:TO-92_Inline_Wide
Changed lines of the file:
@@
 F 0 "Q500" H 5700 925 50  0000 C CNN
 F 1 "LM78L82_TO92" H 5850 925 50  0000 L CNN
-F 2 "Package_TO_SOT_THT:TO-92_Inline" H 5850 1025 50  0001 C CIN
+F 2 "Package_TO_SOT_THT:TO-92_Inline_Wide" H 5850 1025 50  0001 C CIN
 F 3 "https://www.onsemi.com/pub/Collateral/MC78L06A-D.pdf" H 5850 750 50  0001 C CNN
 	1    5850 800

Commit message: Resolves #41 : [PCB] custom footprint library for passives
Parts:
- R501, R502, R503, R504, R507, R510, R511, R512, R513, R516, R545, R546: footprint Resistor_THT:R_Axial_DIN0204_L3.6mm_D1.6mm_P7.62mm_Horizontal -> commons_passives_THT:Passive_THT_resistor_W2.54mm_L12.70mm
Changed lines of the file:
@@
 F 0 "R545" H 3880 2570 50  0000 L CNN
 F 1 "100K" H 3880 2510 50  0000 L CNN
-F 2 "Resistor_THT:R_Axial_DIN0204_L3.6mm_D1.6mm_P7.62mm_Horizontal" H 3850 2550 50  0001 C CNN
+F 2 "commons_passives_THT:Passive_THT_resistor_W2.54mm_L12.70mm" H 3850 2550 50  0001 C CNN
 F 3 "~" H 3850 2550 50  0001 C CNN
 	1    3850 2550
@@
 F 0 "R546" H 7230 3420 50  0000 L CNN
 F 1 "100K" H 7230 3360 50  0000 L CNN
-F 2 "Resistor_THT:R_Axial_DIN0204_L3.6mm_D1.6mm_P7.62mm_Horizontal" H 7200 3400 50  0001 C CNN
+F 2 "commons_passives_THT:Passive_THT_resistor_W2.54mm_L12.70mm" H 7200 3400 50  0001 C CNN
 F 3 "~" H 7200 3400 50  0001 C CNN
 	1    7200 3400
@@
 F 0 "R513" H 6850 5350 50  0000 C CNN
 F 1 "10K" H 6850 5450 50  0000 C CNN
-F 2 "Resistor_THT:R_Axial_DIN0204_L3.6mm_D1.6mm_P7.62mm_Horizontal" H 7000 5400 50  0001 C CNN
+F 2 "commons_passives_THT:Passive_THT_resistor_W2.54mm_L12.70mm" H 7000 5400 50  0001 C CNN
 F 3 "~" H 7000 5400 50  0001 C CNN
 	1    7000 5400
@@
 F 0 "R511" V 7150 5900 50  0000 L CNN
 F 1 "10K" V 7350 5900 50  0000 L CNN
-F 2 "Resistor_THT:R_Axial_DIN0204_L3.6mm_D1.6mm_P7.62mm_Horizontal" H 7250 6000 50  0001 C CNN
+F 2 "commons_passives_THT:Passive_THT_resistor_W2.54mm_L12.70mm" H 7250 6000 50  0001 C CNN
 F 3 "~" H 7250 6000 50  0001 C CNN
 	1    7250 6000
@@
 F 0 "R512" H 6350 3700 50  0000 C CNN
 F 1 "10K" H 6350 3800 50  0000 C CNN
-F 2 "Resistor_THT:R_Axial_DIN0204_L3.6mm_D1.6mm_P7.62mm_Horizontal" H 6500 3750 50  0001 C CNN
+F 2 "commons_passives_THT:Passive_THT_resistor_W2.54mm_L12.70mm" H 6500 3750 50  0001 C CNN
 F 3 "~" H 6500 3750 50  0001 C CNN
 	1    6500 3750
@@
 F 0 "R510" V 6650 4150 50  0000 L CNN
 F 1 "10K" H 6780 4210 50  0000 L CNN
-F 2 "Resistor_THT:R_Axial_DIN0204_L3.6mm_D1.6mm_P7.62mm_Horizontal" H 6750 4250 50  0001 C CNN
+F 2 "commons_passives_THT:Passive_THT_resistor_W2.54mm_L12.70mm" H 6750 4250 50  0001 C CNN
 F 3 "~" H 6750 4250 50  0001 C CNN
 	1    6750 4250
@@
 F 0 "R516" V 6650 5550 50  0000 L CNN
 F 1 "1K8" V 6850 5550 50  0000 L CNN
-F 2 "Resistor_THT:R_Axial_DIN0204_L3.6mm_D1.6mm_P7.62mm_Horizontal" H 6750 5650 50  0001 C CNN
+F 2 "commons_passives_THT:Passive_THT_resistor_W2.54mm_L12.70mm" H 6750 5650 50  0001 C CNN
 F 3 "~" H 6750 5650 50  0001 C CNN
 	1    6750 5650
@@
 F 0 "R504" H 3500 4350 50  0000 C CNN
 F 1 "10K" H 3500 4450 50  0000 C CNN
-F 2 "Resistor_THT:R_Axial_DIN0204_L3.6mm_D1.6mm_P7.62mm_Horizontal" H 3650 4400 50  0001 C CNN
+F 2 "commons_passives_THT:Passive_THT_resistor_W2.54mm_L12.70mm" H 3650 4400 50  0001 C CNN
 F 3 "~" H 3650 4400 50  0001 C CNN
 	1    3650 4400
@@
 F 0 "R502" V 3800 4950 50  0000 L CNN
 F 1 "10K" V 4000 4950 50  0000 L CNN
-F 2 "Resistor_THT:R_Axial_DIN0204_L3.6mm_D1.6mm_P7.62mm_Horizontal" H 3900 5050 50  0001 C CNN
+F 2 "commons_passives_THT:Passive_THT_resistor_W2.54mm_L12.70mm" H 3900 5050 50  0001 C CNN
 F 3 "~" H 3900 5050 50  0001 C CNN
 	1    3900 5050
@@
 F 0 "R503" H 3000 2850 50  0000 C CNN
 F 1 "10K" H 3000 2950 50  0000 C CNN
-F 2 "Resistor_THT:R_Axial_DIN0204_L3.6mm_D1.6mm_P7.62mm_Horizontal" H 3150 2900 50  0001 C CNN
+F 2 "commons_passives_THT:Passive_THT_resistor_W2.54mm_L12.70mm" H 3150 2900 50  0001 C CNN
 F 3 "~" H 3150 2900 50  0001 C CNN
 	1    3150 2900
@@
 F 0 "R501" V 3300 3200 50  0000 L CNN
 F 1 "10K" V 3500 3200 50  0000 L CNN
-F 2 "Resistor_THT:R_Axial_DIN0204_L3.6mm_D1.6mm_P7.62mm_Horizontal" H 3400 3300 50  0001 C CNN
+F 2 "commons_passives_THT:Passive_THT_resistor_W2.54mm_L12.70mm" H 3400 3300 50  0001 C CNN
 F 3 "~" H 3400 3300 50  0001 C CNN
 	1    3400 3300
@@
 F 0 "R507" V 3300 4600 50  0000 L CNN
 F 1 "1K8" V 3500 4600 50  0000 L CNN
-F 2 "Resistor_THT:R_Axial_DIN0204_L3.6mm_D1.6mm_P7.62mm_Horizontal" H 3400 4700 50  0001 C CNN
+F 2 "commons_passives_THT:Passive_THT_resistor_W2.54mm_L12.70mm" H 3400 4700 50  0001 C CNN
 F 3 "~" H 3400 4700 50  0001 C CNN
 	1    3400 4700

Commit message: [PCB] continue footprint assignation
Parts:
- C500, C501, C502, C511, C512, C513, C514, C523, C565: footprint (none) -> commons_passives_THT:Passive_THT_capacitor_ceramic_radial_W5.08mm_L6.35mm_X11.43mm
Changed lines of the file:
@@
 F 0 "C501" H 1625 8400 50  0000 L CNN
 F 1 "0.1uF" H 1625 8200 50  0000 L CNN
-F 2 "" H 1638 8150 50  0001 C CNN
+F 2 "commons_passives_THT:Passive_THT_capacitor_ceramic_radial_W5.08mm_L6.35mm_X11.43mm" H 1638 8150 50  0001 C CNN
 F 3 "~" H 1600 8300 50  0001 C CNN
 	1    1600 8300
@@
 F 0 "C512" H 1625 9000 50  0000 L CNN
 F 1 "0.1uF" H 1625 8800 50  0000 L CNN
-F 2 "" H 1638 8750 50  0001 C CNN
+F 2 "commons_passives_THT:Passive_THT_capacitor_ceramic_radial_W5.08mm_L6.35mm_X11.43mm" H 1638 8750 50  0001 C CNN
 F 3 "~" H 1600 8900 50  0001 C CNN
 	1    1600 8900
@@
 F 0 "C500" H 875 8400 50  0000 L CNN
 F 1 "0.1uF" H 875 8200 50  0000 L CNN
-F 2 "" H 888 8150 50  0001 C CNN
+F 2 "commons_passives_THT:Passive_THT_capacitor_ceramic_radial_W5.08mm_L6.35mm_X11.43mm" H 888 8150 50  0001 C CNN
 F 3 "~" H 850 8300 50  0001 C CNN
 	1    850  8300
@@
 F 0 "C511" H 875 9000 50  0000 L CNN
 F 1 "0.1uF" H 875 8800 50  0000 L CNN
-F 2 "" H 888 8750 50  0001 C CNN
+F 2 "commons_passives_THT:Passive_THT_capacitor_ceramic_radial_W5.08mm_L6.35mm_X11.43mm" H 888 8750 50  0001 C CNN
 F 3 "~" H 850 8900 50  0001 C CNN
 	1    850  8900
@@
 F 0 "C502" H 3125 8400 50  0000 L CNN
 F 1 "0.1uF" H 3125 8200 50  0000 L CNN
-F 2 "" H 3138 8150 50  0001 C CNN
+F 2 "commons_passives_THT:Passive_THT_capacitor_ceramic_radial_W5.08mm_L6.35mm_X11.43mm" H 3138 8150 50  0001 C CNN
 F 3 "~" H 3100 8300 50  0001 C CNN
 	1    3100 8300
@@
 F 0 "C513" H 3125 9000 50  0000 L CNN
 F 1 "0.1uF" H 3125 8800 50  0000 L CNN
-F 2 "" H 3138 8750 50  0001 C CNN
+F 2 "commons_passives_THT:Passive_THT_capacitor_ceramic_radial_W5.08mm_L6.35mm_X11.43mm" H 3138 8750 50  0001 C CNN
 F 3 "~" H 3100 8900 50  0001 C CNN
 	1    3100 8900
@@
 F 0 "C514" H 2375 8400 50  0000 L CNN
 F 1 "0.1uF" H 2375 8200 50  0000 L CNN
-F 2 "" H 2388 8150 50  0001 C CNN
+F 2 "commons_passives_THT:Passive_THT_capacitor_ceramic_radial_W5.08mm_L6.35mm_X11.43mm" H 2388 8150 50  0001 C CNN
 F 3 "~" H 2350 8300 50  0001 C CNN
 	1    2350 8300
@@
 F 0 "C523" H 2375 9000 50  0000 L CNN
 F 1 "0.1uF" H 2375 8800 50  0000 L CNN
-F 2 "" H 2388 8750 50  0001 C CNN
+F 2 "commons_passives_THT:Passive_THT_capacitor_ceramic_radial_W5.08mm_L6.35mm_X11.43mm" H 2388 8750 50  0001 C CNN
 F 3 "~" H 2350 8900 50  0001 C CNN
 	1    2350 8900
@@
 F 0 "C565" H 6875 1150 50  0000 L CNN
 F 1 "0.1uF" H 6875 950 50  0000 L CNN
-F 2 "" H 6888 900 50  0001 C CNN
+F 2 "commons_passives_THT:Passive_THT_capacitor_ceramic_radial_W5.08mm_L6.35mm_X11.43mm" H 6888 900 50  0001 C CNN
 F 3 "~" H 6850 1050 50  0001 C CNN
 	1    6850 1050

Commit message: [PCB] continue assigning footprints - done all fixed capacitors
Parts:
- C505, C506, C509, C510, C517, C518, C521, C522: footprint (none) -> commons_passives_THT:Passive_THT_capacitor_W2.54mm_L10.16mm
- C508, C520, C564: footprint (none) -> commons_passives_THT:Passive_THT_capacitor_polarized_W6.35mm_L20.32mm
- C566, C567: footprint (none) -> commons_passives_THT:Passive_THT_capacitor_polarized_rad_D5.08mm_P2.54mm_H12.70mm
Changed lines of the file:
@@
 F 0 "C566" H 3900 2050 50  0000 L CNN
 F 1 "47uF" H 3900 1850 50  0000 L CNN
-F 2 "" H 3850 1950 50  0001 C CNN
+F 2 "commons_passives_THT:Passive_THT_capacitor_polarized_rad_D5.08mm_P2.54mm_H12.70mm" H 3850 1950 50  0001 C CNN
 F 3 "~" H 3850 1950 50  0001 C CNN
 	1    3850 1950
@@
 F 0 "C567" H 7250 2900 50  0000 L CNN
 F 1 "47uF" H 7250 2700 50  0000 L CNN
-F 2 "" H 7200 2800 50  0001 C CNN
+F 2 "commons_passives_THT:Passive_THT_capacitor_polarized_rad_D5.08mm_P2.54mm_H12.70mm" H 7200 2800 50  0001 C CNN
 F 3 "~" H 7200 2800 50  0001 C CNN
 	1    7200 2800
@@
 F 0 "C520" H 7600 7350 50  0000 L CNN
 F 1 "47uF" H 7600 7450 50  0000 L CNN
-F 2 "" H 7500 7400 50  0001 C CNN
+F 2 "commons_passives_THT:Passive_THT_capacitor_polarized_W6.35mm_L20.32mm" H 7500 7400 50  0001 C CNN
 F 3 "~" H 7500 7400 50  0001 C CNN
 	1    7500 7400
@@
 F 0 "C518" V 6450 6450 50  0000 L CNN
 F 1 "0.001uF" V 6550 6450 50  0000 L CNN
-F 2 "" H 6638 6250 50  0001 C CNN
+F 2 "commons_passives_THT:Passive_THT_capacitor_W2.54mm_L10.16mm" H 6638 6250 50  0001 C CNN
 F 3 "~" H 6600 6400 50  0001 C CNN
 	1    6600 6400
@@
 F 0 "C522" V 5950 5900 50  0000 L CNN
 F 1 "0.001uF" V 6250 5850 50  0000 L CNN
-F 2 "" H 6138 5850 50  0001 C CNN
+F 2 "commons_passives_THT:Passive_THT_capacitor_W2.54mm_L10.16mm" H 6138 5850 50  0001 C CNN
 F 3 "~" H 6100 6000 50  0001 C CNN
 	1    6100 6000
@@
 F 0 "C517" V 5950 4700 50  0000 L CNN
 F 1 "0.001uF" V 6050 4700 50  0000 L CNN
-F 2 "" H 6138 4500 50  0001 C CNN
+F 2 "commons_passives_THT:Passive_THT_capacitor_W2.54mm_L10.16mm" H 6138 4500 50  0001 C CNN
 F 3 "~" H 6100 4650 50  0001 C CNN
 	1    6100 4650
@@
 F 0 "C521" V 5450 4150 50  0000 L CNN
 F 1 "0.001uF" V 5750 4100 50  0000 L CNN
-F 2 "" H 5638 4100 50  0001 C CNN
+F 2 "commons_passives_THT:Passive_THT_capacitor_W2.54mm_L10.16mm" H 5638 4100 50  0001 C CNN
 F 3 "~" H 5600 4250 50  0001 C CNN
 	1    5600 4250
@@
 F 0 "C508" H 3850 6400 50  0000 L CNN
 F 1 "47uF" H 3850 6500 50  0000 L CNN
-F 2 "" H 4150 6450 50  0001 C CNN
+F 2 "commons_passives_THT:Passive_THT_capacitor_polarized_W6.35mm_L20.32mm" H 4150 6450 50  0001 C CNN
 F 3 "~" H 4150 6450 50  0001 C CNN
 	1    4150 6450
@@
 F 0 "C506" V 3100 5350 50  0000 L CNN
 F 1 "0.001uF" V 3400 5350 50  0000 L CNN
-F 2 "" H 3288 5300 50  0001 C CNN
+F 2 "commons_passives_THT:Passive_THT_capacitor_W2.54mm_L10.16mm" H 3288 5300 50  0001 C CNN
 F 3 "~" H 3250 5450 50  0001 C CNN
 	1    3250 5450
@@
 F 0 "C510" V 2600 4950 50  0000 L CNN
 F 1 "0.001uF" V 2900 4900 50  0000 L CNN
-F 2 "" H 2788 4900 50  0001 C CNN
+F 2 "commons_passives_THT:Passive_THT_capacitor_W2.54mm_L10.16mm" H 2788 4900 50  0001 C CNN
 F 3 "~" H 2750 5050 50  0001 C CNN
 	1    2750 5050
@@
 F 0 "C505" V 2600 3750 50  0000 L CNN
 F 1 "0.001uF" V 2700 3750 50  0000 L CNN
-F 2 "" H 2788 3550 50  0001 C CNN
+F 2 "commons_passives_THT:Passive_THT_capacitor_W2.54mm_L10.16mm" H 2788 3550 50  0001 C CNN
 F 3 "~" H 2750 3700 50  0001 C CNN
 	1    2750 3700
@@
 F 0 "C509" V 2100 3200 50  0000 L CNN
 F 1 "0.001uF" V 2400 3150 50  0000 L CNN
-F 2 "" H 2288 3150 50  0001 C CNN
+F 2 "commons_passives_THT:Passive_THT_capacitor_W2.54mm_L10.16mm" H 2288 3150 50  0001 C CNN
 F 3 "~" H 2250 3300 50  0001 C CNN
 	1    2250 3300
@@
 F 0 "C564" H 6375 1150 50  0000 L CNN
 F 1 "100uF" H 6375 950 50  0000 L CNN
-F 2 "" H 6350 1050 50  0001 C CNN
+F 2 "commons_passives_THT:Passive_THT_capacitor_polarized_W6.35mm_L20.32mm" H 6350 1050 50  0001 C CNN
 F 3 "~" H 6350 1050 50  0001 C CNN
 	1    6350 1050
