File: atari-16-32-bits/motherboards/c300780-001/subsheet_600.sch (KiCad schematic (older format))
At the start: 9 parts, among them U600 SIMM_30_PHY, U601 SIMM_30_PHY, U602 SIMM_30_PHY, U603 SIMM_30_PHY

Commit message: [PCB] continue assigning footprints - done all fixed capacitors
Parts:
- C600: footprint (none) -> commons_passives_THT:Passive_THT_capacitor_polarized_W6.35mm_L20.32mm
- C633, C634, C635, C636: footprint (none) -> commons_passives_THT:Passive_THT_capacitor_mlcc_W2.54mm_L10.16mm
Changed lines of the file:
@@
 F 0 "C633" H 1275 3600 50  0000 L CNN
 F 1 "0.22uF" H 1275 3400 50  0000 L CNN
-F 2 "" H 1288 3350 50  0001 C CNN
+F 2 "commons_passives_THT:Passive_THT_capacitor_mlcc_W2.54mm_L10.16mm" H 1288 3350 50  0001 C CNN
 F 3 "~" H 1250 3500 50  0001 C CNN
 	1    1250 3500
@@
 F 0 "C635" H 7025 3600 50  0000 L CNN
 F 1 "0.22uF" H 7025 3400 50  0000 L CNN
-F 2 "" H 7038 3350 50  0001 C CNN
+F 2 "commons_passives_THT:Passive_THT_capacitor_mlcc_W2.54mm_L10.16mm" H 7038 3350 50  0001 C CNN
 F 3 "~" H 7000 3500 50  0001 C CNN
 	1    7000 3500
@@
 F 0 "C634" H 1275 7600 50  0000 L CNN
 F 1 "0.22uF" H 1275 7400 50  0000 L CNN
-F 2 "" H 1288 7350 50  0001 C CNN
+F 2 "commons_passives_THT:Passive_THT_capacitor_mlcc_W2.54mm_L10.16mm" H 1288 7350 50  0001 C CNN
 F 3 "~" H 1250 7500 50  0001 C CNN
 	1    1250 7500
@@
 F 0 "C636" H 7025 7600 50  0000 L CNN
 F 1 "0.22uF" H 7025 7400 50  0000 L CNN
-F 2 "" H 7038 7350 50  0001 C CNN
+F 2 "commons_passives_THT:Passive_THT_capacitor_mlcc_W2.54mm_L10.16mm" H 7038 7350 50  0001 C CNN
 F 3 "~" H 7000 7500 50  0001 C CNN
 	1    7000 7500
@@
 F 0 "C600" H 4300 1600 50  0000 L CNN
 F 1 "100uF" H 4300 1400 50  0000 L CNN
-F 2 "" H 4250 1500 50  0001 C CNN
+F 2 "commons_passives_THT:Passive_THT_capacitor_polarized_W6.35mm_L20.32mm" H 4250 1500 50  0001 C CNN
 F 3 "~" H 4250 1500 50  0001 C CNN
 	1    4250 1500

Commit message: [PCB] created, assigned SIMM-30 footprint
Parts:
- U600, U601, U602, U603: footprint (none) -> commons-interconnect_THT:socket-simm-30-P2.54mm
Changed lines of the file:
@@
 F 0 "U600" H 2600 5300 50  0000 L TNN
 F 1 "SIMM_30_PHY" H 2600 5200 50  0000 L TNB
-F 2 "" H 3000 3550 50  0001 C CNN
+F 2 "commons-interconnect_THT:socket-simm-30-P2.54mm" H 3000 3550 50  0001 C CNN
 F 3 "" H 2600 5500 50  0001 L TNN
 	1    3000 3550
@@
 F 0 "U601" H 5700 5300 50  0000 L TNN
 F 1 "SIMM_30_PHY" H 5700 5200 50  0000 L TNB
-F 2 "" H 6100 3550 50  0001 C CNN
+F 2 "commons-interconnect_THT:socket-simm-30-P2.54mm" H 6100 3550 50  0001 C CNN
 F 3 "" H 5700 5500 50  0001 L TNN
 	1    6100 3550
@@
 F 0 "U602" H 2600 9300 50  0000 L TNN
 F 1 "SIMM_30_PHY" H 2600 9200 50  0000 L TNB
-F 2 "" H 3000 7550 50  0001 C CNN
+F 2 "commons-interconnect_THT:socket-simm-30-P2.54mm" H 3000 7550 50  0001 C CNN
 F 3 "" H 2600 9500 50  0001 L TNN
 	1    3000 7550
@@
 F 0 "U603" H 5700 9300 50  0000 L TNN
 F 1 "SIMM_30_PHY" H 5700 9200 50  0000 L TNB
-F 2 "" H 6100 7550 50  0001 C CNN
+F 2 "commons-interconnect_THT:socket-simm-30-P2.54mm" H 6100 7550 50  0001 C CNN
 F 3 "" H 5700 9500 50  0001 L TNN
 	1    6100 7550
