File: atari-16-32-bits/motherboards/c300780-001/subsheet_103.sch (KiCad schematic (older format))
At the start: 4 parts, among them J103 Cartridge Port

Commit message: Resolves #41 : [PCB] custom footprint library for passives
Parts:
- L100: footprint (none) -> commons_passives_THT:Passive_THT_ferrite_bead_W3.81mm_L15.24mm
Changed lines of the file:
@@
 F 0 "L100" H 4325 1750 50  0000 L CNN
 F 1 "FB" H 4325 1650 50  0000 L CNN
-F 2 "" V 4180 1700 50  0001 C CNN
+F 2 "commons_passives_THT:Passive_THT_ferrite_bead_W3.81mm_L15.24mm" V 4180 1700 50  0001 C CNN
 F 3 "~" H 4250 1700 50  0001 C CNN
 	1    4250 1700

Commit message: [PCB] continue footprint assignation
Parts:
- C109: footprint (none) -> commons_passives_THT:Passive_THT_capacitor_ceramic_radial_W5.08mm_L6.35mm_X11.43mm
- C110: footprint (none) -> commons_passives_THT:Passive_THT_capacitor_polarized_W6.35mm_L20.32mm
Changed lines of the file:
@@
 F 0 "C109" H 3775 2450 50  0000 L CNN
 F 1 "0.1uF" H 3775 2250 50  0000 L CNN
-F 2 "" H 3788 2200 50  0001 C CNN
+F 2 "commons_passives_THT:Passive_THT_capacitor_ceramic_radial_W5.08mm_L6.35mm_X11.43mm" H 3788 2200 50  0001 C CNN
 F 3 "~" H 3750 2350 50  0001 C CNN
 	1    3750 2350
@@
 F 0 "C110" H 3275 2450 50  0000 L CNN
 F 1 "100uF" H 3275 2250 50  0000 L CNN
-F 2 "" H 3250 2350 50  0001 C CNN
+F 2 "commons_passives_THT:Passive_THT_capacitor_polarized_W6.35mm_L20.32mm" H 3250 2350 50  0001 C CNN
 F 3 "~" H 3250 2350 50  0001 C CNN
 	1    3250 2350

Commit message: [PCB] continue assigning footprints + special libraries of special holes referenced in the measurement schema of the field service manual
Parts:
- J103: footprint (none) -> atari-interconnect:socket-edge-pcb_40p_P2.01mm
Changed lines of the file:
@@
 F 0 "J103" H 5000 5900 50  0000 C CNN
 F 1 "Cartridge Port" H 5000 1800 50  0000 C CNN
-F 2 "" H 5000 3900 50  0001 C CNN
+F 2 "atari-interconnect:socket-edge-pcb_40p_P2.01mm" H 5000 3900 50  0001 C CNN
 F 3 "~" H 5000 3900 50  0001 C CNN
 	1    5000 3900
