File: atari-16-32-bits/motherboards/c300780-001/subsheet_201.sch (KiCad schematic (older format))
At the start: 7 parts, among them J202 BRS — To IKBD, U201 MC6850_PHY

Commit message: [PCB] Assign builtins footprint when possible - resistors, ports
Parts:
- R210: footprint (none) -> Resistor_THT:R_Axial_DIN0204_L3.6mm_D1.6mm_P7.62mm_Horizontal
Changed lines of the file:
@@
 F 0 "R210" H 2150 4450 50  0000 C CNN
 F 1 "10K" H 2150 4550 50  0000 C CNN
-F 2 "" H 2300 4500 50  0001 C CNN
+F 2 "Resistor_THT:R_Axial_DIN0204_L3.6mm_D1.6mm_P7.62mm_Horizontal" H 2300 4500 50  0001 C CNN
 F 3 "~" H 2300 4500 50  0001 C CNN
 	1    2300 4500

Commit message: Resolves #41 : [PCB] custom footprint library for passives
Parts:
- L207, L226, L227: footprint (none) -> commons_passives_THT:Passive_THT_EMI_filter_W5.08mm_L7.62mm
- R210: footprint Resistor_THT:R_Axial_DIN0204_L3.6mm_D1.6mm_P7.62mm_Horizontal -> commons_passives_THT:Passive_THT_resistor_W2.54mm_L12.70mm
Changed lines of the file:
@@
 F 0 "R210" H 2150 4450 50  0000 C CNN
 F 1 "10K" H 2150 4550 50  0000 C CNN
-F 2 "Resistor_THT:R_Axial_DIN0204_L3.6mm_D1.6mm_P7.62mm_Horizontal" H 2300 4500 50  0001 C CNN
+F 2 "commons_passives_THT:Passive_THT_resistor_W2.54mm_L12.70mm" H 2300 4500 50  0001 C CNN
 F 3 "~" H 2300 4500 50  0001 C CNN
 	1    2300 4500
@@
 F 0 "L207" H 3250 4875 50  0000 C CNN
 F 1 "EMI_Filter_LCL" H 3250 4800 50  0000 C CNN
-F 2 "" V 3250 4600 50  0001 C CNN
+F 2 "commons_passives_THT:Passive_THT_EMI_filter_W5.08mm_L7.62mm" V 3250 4600 50  0001 C CNN
 F 3 "http://www.murata.com/~/media/webrenewal/support/library/catalog/products/emc/emifil/c31e.ashx?la=en-gb" V 3250 4600 50  0001 C CNN
 	1    3250 4600
@@
 F 0 "L226" H 4000 5125 50  0000 C CNN
 F 1 "EMI_Filter_LCL" H 4000 5050 50  0000 C CNN
-F 2 "" V 4000 4850 50  0001 C CNN
+F 2 "commons_passives_THT:Passive_THT_EMI_filter_W5.08mm_L7.62mm" V 4000 4850 50  0001 C CNN
 F 3 "http://www.murata.com/~/media/webrenewal/support/library/catalog/products/emc/emifil/c31e.ashx?la=en-gb" V 4000 4850 50  0001 C CNN
 	1    4000 4850
@@
 F 0 "L227" H 3250 5375 50  0000 C CNN
 F 1 "EMI_Filter_LCL" H 3250 5300 50  0000 C CNN
-F 2 "" V 3250 5100 50  0001 C CNN
+F 2 "commons_passives_THT:Passive_THT_EMI_filter_W5.08mm_L7.62mm" V 3250 5100 50  0001 C CNN
 F 3 "http://www.murata.com/~/media/webrenewal/support/library/catalog/products/emc/emifil/c31e.ashx?la=en-gb" V 3250 5100 50  0001 C CNN
 	1    3250 5100

Commit message: [PCB] continue footprint assignation
Parts:
- C210: footprint (none) -> commons_passives_THT:Passive_THT_capacitor_ceramic_radial_W5.08mm_L6.35mm_X11.43mm
Changed lines of the file:
@@
 F 0 "C210" H 2575 3100 50  0000 L CNN
 F 1 "0.1uF" H 2575 2900 50  0000 L CNN
-F 2 "" H 2588 2850 50  0001 C CNN
+F 2 "commons_passives_THT:Passive_THT_capacitor_ceramic_radial_W5.08mm_L6.35mm_X11.43mm" H 2588 2850 50  0001 C CNN
 F 3 "~" H 2550 3000 50  0001 C CNN
 	1    2550 3000

Commit message: [PCB] continue assigning footprints + special libraries of special holes referenced in the measurement schema of the field service manual
Parts:
- J202: footprint (none) -> atari-interconnect:PinHeader_1x08_P2.54mm_Vertical_Ikbd
Changed lines of the file:
@@
 F 0 "J202" H 5950 5050 50  0000 C CNN
 F 1 "BRS — To IKBD" H 5950 4150 50  0000 C CNN
-F 2 "" H 5950 4650 50  0001 C CNN
+F 2 "atari-interconnect:PinHeader_1x08_P2.54mm_Vertical_Ikbd" H 5950 4650 50  0001 C CNN
 F 3 "~" H 5950 4650 50  0001 C CNN
 	1    5950 4650
