File: atari-16-32-bits/motherboards/c300780-001/subsheet_301.sch (KiCad schematic (older format))
At the start: 19 parts, among them J301 DB-19S ACSI Port, U302 74LS245_PHY, U306 74LS74_PHY, U307 74LS244_PHY

Commit message: [PCB] Assign builtins footprint when possible - resistors, ports
Parts:
- R312, R313, R314, R315, R316, R317, R318, R319, R320, R321, R322, R323: footprint (none) -> Resistor_THT:R_Axial_DIN0204_L3.6mm_D1.6mm_P7.62mm_Horizontal
Changed lines of the file:
@@
 F 0 "R323" V 2650 6000 50  0000 C CNN
 F 1 "68" V 2850 6000 50  0000 C CNN
-F 2 "" H 2750 6000 50  0001 C CNN
+F 2 "Resistor_THT:R_Axial_DIN0204_L3.6mm_D1.6mm_P7.62mm_Horizontal" H 2750 6000 50  0001 C CNN
 F 3 "~" H 2750 6000 50  0001 C CNN
 	1    2750 6000
@@
 F 0 "R321" V 2650 6500 50  0000 C CNN
 F 1 "68" V 2850 6500 50  0000 C CNN
-F 2 "" H 2750 6500 50  0001 C CNN
+F 2 "Resistor_THT:R_Axial_DIN0204_L3.6mm_D1.6mm_P7.62mm_Horizontal" H 2750 6500 50  0001 C CNN
 F 3 "~" H 2750 6500 50  0001 C CNN
 	1    2750 6500
@@
 F 0 "R319" V 2650 7000 50  0000 C CNN
 F 1 "68" V 2850 7000 50  0000 C CNN
-F 2 "" H 2750 7000 50  0001 C CNN
+F 2 "Resistor_THT:R_Axial_DIN0204_L3.6mm_D1.6mm_P7.62mm_Horizontal" H 2750 7000 50  0001 C CNN
 F 3 "~" H 2750 7000 50  0001 C CNN
 	1    2750 7000
@@
 F 0 "R317" V 2650 7500 50  0000 C CNN
 F 1 "68" V 2850 7500 50  0000 C CNN
-F 2 "" H 2750 7500 50  0001 C CNN
+F 2 "Resistor_THT:R_Axial_DIN0204_L3.6mm_D1.6mm_P7.62mm_Horizontal" H 2750 7500 50  0001 C CNN
 F 3 "~" H 2750 7500 50  0001 C CNN
 	1    2750 7500
@@
 F 0 "R315" V 2650 8000 50  0000 C CNN
 F 1 "68" V 2850 8000 50  0000 C CNN
-F 2 "" H 2750 8000 50  0001 C CNN
+F 2 "Resistor_THT:R_Axial_DIN0204_L3.6mm_D1.6mm_P7.62mm_Horizontal" H 2750 8000 50  0001 C CNN
 F 3 "~" H 2750 8000 50  0001 C CNN
 	1    2750 8000
@@
 F 0 "R313" V 2650 8500 50  0000 C CNN
 F 1 "68" V 2850 8500 50  0000 C CNN
-F 2 "" H 2750 8500 50  0001 C CNN
+F 2 "Resistor_THT:R_Axial_DIN0204_L3.6mm_D1.6mm_P7.62mm_Horizontal" H 2750 8500 50  0001 C CNN
 F 3 "~" H 2750 8500 50  0001 C CNN
 	1    2750 8500
@@
 F 0 "R322" V 3150 6250 50  0000 C CNN
 F 1 "68" V 3350 6250 50  0000 C CNN
-F 2 "" H 3250 6250 50  0001 C CNN
+F 2 "Resistor_THT:R_Axial_DIN0204_L3.6mm_D1.6mm_P7.62mm_Horizontal" H 3250 6250 50  0001 C CNN
 F 3 "~" H 3250 6250 50  0001 C CNN
 	1    3250 6250
@@
 F 0 "R320" V 3150 6750 50  0000 C CNN
 F 1 "68" V 3350 6750 50  0000 C CNN
-F 2 "" H 3250 6750 50  0001 C CNN
+F 2 "Resistor_THT:R_Axial_DIN0204_L3.6mm_D1.6mm_P7.62mm_Horizontal" H 3250 6750 50  0001 C CNN
 F 3 "~" H 3250 6750 50  0001 C CNN
 	1    3250 6750
@@
 F 0 "R318" V 3150 7250 50  0000 C CNN
 F 1 "68" V 3350 7250 50  0000 C CNN
-F 2 "" H 3250 7250 50  0001 C CNN
+F 2 "Resistor_THT:R_Axial_DIN0204_L3.6mm_D1.6mm_P7.62mm_Horizontal" H 3250 7250 50  0001 C CNN
 F 3 "~" H 3250 7250 50  0001 C CNN
 	1    3250 7250
@@
 F 0 "R316" V 3150 7750 50  0000 C CNN
 F 1 "68" V 3350 7750 50  0000 C CNN
-F 2 "" H 3250 7750 50  0001 C CNN
+F 2 "Resistor_THT:R_Axial_DIN0204_L3.6mm_D1.6mm_P7.62mm_Horizontal" H 3250 7750 50  0001 C CNN
 F 3 "~" H 3250 7750 50  0001 C CNN
 	1    3250 7750
@@
 F 0 "R314" V 3150 8250 50  0000 C CNN
 F 1 "68" V 3350 8250 50  0000 C CNN
-F 2 "" H 3250 8250 50  0001 C CNN
+F 2 "Resistor_THT:R_Axial_DIN0204_L3.6mm_D1.6mm_P7.62mm_Horizontal" H 3250 8250 50  0001 C CNN
 F 3 "~" H 3250 8250 50  0001 C CNN
 	1    3250 8250
@@
 F 0 "R312" V 3150 8750 50  0000 C CNN
 F 1 "68" V 3350 8750 50  0000 C CNN
-F 2 "" H 3250 8750 50  0001 C CNN
+F 2 "Resistor_THT:R_Axial_DIN0204_L3.6mm_D1.6mm_P7.62mm_Horizontal" H 3250 8750 50  0001 C CNN
 F 3 "~" H 3250 8750 50  0001 C CNN
 	1    3250 8750

Commit message: Resolves #41 : [PCB] custom footprint library for passives
Parts:
- R312, R313, R314, R315, R316, R317, R318, R319, R320, R321, R322, R323: footprint Resistor_THT:R_Axial_DIN0204_L3.6mm_D1.6mm_P7.62mm_Horizontal -> commons_passives_THT:Passive_THT_resistor_W2.54mm_L12.70mm
Changed lines of the file:
@@
 F 0 "R323" V 2650 6000 50  0000 C CNN
 F 1 "68" V 2850 6000 50  0000 C CNN
-F 2 "Resistor_THT:R_Axial_DIN0204_L3.6mm_D1.6mm_P7.62mm_Horizontal" H 2750 6000 50  0001 C CNN
+F 2 "commons_passives_THT:Passive_THT_resistor_W2.54mm_L12.70mm" H 2750 6000 50  0001 C CNN
 F 3 "~" H 2750 6000 50  0001 C CNN
 	1    2750 6000
@@
 F 0 "R321" V 2650 6500 50  0000 C CNN
 F 1 "68" V 2850 6500 50  0000 C CNN
-F 2 "Resistor_THT:R_Axial_DIN0204_L3.6mm_D1.6mm_P7.62mm_Horizontal" H 2750 6500 50  0001 C CNN
+F 2 "commons_passives_THT:Passive_THT_resistor_W2.54mm_L12.70mm" H 2750 6500 50  0001 C CNN
 F 3 "~" H 2750 6500 50  0001 C CNN
 	1    2750 6500
@@
 F 0 "R319" V 2650 7000 50  0000 C CNN
 F 1 "68" V 2850 7000 50  0000 C CNN
-F 2 "Resistor_THT:R_Axial_DIN0204_L3.6mm_D1.6mm_P7.62mm_Horizontal" H 2750 7000 50  0001 C CNN
+F 2 "commons_passives_THT:Passive_THT_resistor_W2.54mm_L12.70mm" H 2750 7000 50  0001 C CNN
 F 3 "~" H 2750 7000 50  0001 C CNN
 	1    2750 7000
@@
 F 0 "R317" V 2650 7500 50  0000 C CNN
 F 1 "68" V 2850 7500 50  0000 C CNN
-F 2 "Resistor_THT:R_Axial_DIN0204_L3.6mm_D1.6mm_P7.62mm_Horizontal" H 2750 7500 50  0001 C CNN
+F 2 "commons_passives_THT:Passive_THT_resistor_W2.54mm_L12.70mm" H 2750 7500 50  0001 C CNN
 F 3 "~" H 2750 7500 50  0001 C CNN
 	1    2750 7500
@@
 F 0 "R315" V 2650 8000 50  0000 C CNN
 F 1 "68" V 2850 8000 50  0000 C CNN
-F 2 "Resistor_THT:R_Axial_DIN0204_L3.6mm_D1.6mm_P7.62mm_Horizontal" H 2750 8000 50  0001 C CNN
+F 2 "commons_passives_THT:Passive_THT_resistor_W2.54mm_L12.70mm" H 2750 8000 50  0001 C CNN
 F 3 "~" H 2750 8000 50  0001 C CNN
 	1    2750 8000
@@
 F 0 "R313" V 2650 8500 50  0000 C CNN
 F 1 "68" V 2850 8500 50  0000 C CNN
-F 2 "Resistor_THT:R_Axial_DIN0204_L3.6mm_D1.6mm_P7.62mm_Horizontal" H 2750 8500 50  0001 C CNN
+F 2 "commons_passives_THT:Passive_THT_resistor_W2.54mm_L12.70mm" H 2750 8500 50  0001 C CNN
 F 3 "~" H 2750 8500 50  0001 C CNN
 	1    2750 8500
@@
 F 0 "R322" V 3150 6250 50  0000 C CNN
 F 1 "68" V 3350 6250 50  0000 C CNN
-F 2 "Resistor_THT:R_Axial_DIN0204_L3.6mm_D1.6mm_P7.62mm_Horizontal" H 3250 6250 50  0001 C CNN
+F 2 "commons_passives_THT:Passive_THT_resistor_W2.54mm_L12.70mm" H 3250 6250 50  0001 C CNN
 F 3 "~" H 3250 6250 50  0001 C CNN
 	1    3250 6250
@@
 F 0 "R320" V 3150 6750 50  0000 C CNN
 F 1 "68" V 3350 6750 50  0000 C CNN
-F 2 "Resistor_THT:R_Axial_DIN0204_L3.6mm_D1.6mm_P7.62mm_Horizontal" H 3250 6750 50  0001 C CNN
+F 2 "commons_passives_THT:Passive_THT_resistor_W2.54mm_L12.70mm" H 3250 6750 50  0001 C CNN
 F 3 "~" H 3250 6750 50  0001 C CNN
 	1    3250 6750
@@
 F 0 "R318" V 3150 7250 50  0000 C CNN
 F 1 "68" V 3350 7250 50  0000 C CNN
-F 2 "Resistor_THT:R_Axial_DIN0204_L3.6mm_D1.6mm_P7.62mm_Horizontal" H 3250 7250 50  0001 C CNN
+F 2 "commons_passives_THT:Passive_THT_resistor_W2.54mm_L12.70mm" H 3250 7250 50  0001 C CNN
 F 3 "~" H 3250 7250 50  0001 C CNN
 	1    3250 7250
@@
 F 0 "R316" V 3150 7750 50  0000 C CNN
 F 1 "68" V 3350 7750 50  0000 C CNN
-F 2 "Resistor_THT:R_Axial_DIN0204_L3.6mm_D1.6mm_P7.62mm_Horizontal" H 3250 7750 50  0001 C CNN
+F 2 "commons_passives_THT:Passive_THT_resistor_W2.54mm_L12.70mm" H 3250 7750 50  0001 C CNN
 F 3 "~" H 3250 7750 50  0001 C CNN
 	1    3250 7750
@@
 F 0 "R314" V 3150 8250 50  0000 C CNN
 F 1 "68" V 3350 8250 50  0000 C CNN
-F 2 "Resistor_THT:R_Axial_DIN0204_L3.6mm_D1.6mm_P7.62mm_Horizontal" H 3250 8250 50  0001 C CNN
+F 2 "commons_passives_THT:Passive_THT_resistor_W2.54mm_L12.70mm" H 3250 8250 50  0001 C CNN
 F 3 "~" H 3250 8250 50  0001 C CNN
 	1    3250 8250
@@
 F 0 "R312" V 3150 8750 50  0000 C CNN
 F 1 "68" V 3350 8750 50  0000 C CNN
-F 2 "Resistor_THT:R_Axial_DIN0204_L3.6mm_D1.6mm_P7.62mm_Horizontal" H 3250 8750 50  0001 C CNN
+F 2 "commons_passives_THT:Passive_THT_resistor_W2.54mm_L12.70mm" H 3250 8750 50  0001 C CNN
 F 3 "~" H 3250 8750 50  0001 C CNN
 	1    3250 8750

Commit message: [PCB] continue footprint assignation
Parts:
- C303, C306, C307: footprint (none) -> commons_passives_THT:Passive_THT_capacitor_ceramic_radial_W5.08mm_L6.35mm_X11.43mm
Changed lines of the file:
@@
 F 0 "C303" H 5775 2350 50  0000 L CNN
 F 1 "0.1uF" H 5775 2150 50  0000 L CNN
-F 2 "" H 5788 2100 50  0001 C CNN
+F 2 "commons_passives_THT:Passive_THT_capacitor_ceramic_radial_W5.08mm_L6.35mm_X11.43mm" H 5788 2100 50  0001 C CNN
 F 3 "~" H 5750 2250 50  0001 C CNN
 	1    5750 2250
@@
 F 0 "C306" H 5775 3850 50  0000 L CNN
 F 1 "0.1uF" H 5775 3650 50  0000 L CNN
-F 2 "" H 5788 3600 50  0001 C CNN
+F 2 "commons_passives_THT:Passive_THT_capacitor_ceramic_radial_W5.08mm_L6.35mm_X11.43mm" H 5788 3600 50  0001 C CNN
 F 3 "~" H 5750 3750 50  0001 C CNN
 	1    5750 3750
@@
 F 0 "C307" H 2275 5100 50  0000 L CNN
 F 1 "0.1uF" H 2275 4900 50  0000 L CNN
-F 2 "" H 2288 4850 50  0001 C CNN
+F 2 "commons_passives_THT:Passive_THT_capacitor_ceramic_radial_W5.08mm_L6.35mm_X11.43mm" H 2288 4850 50  0001 C CNN
 F 3 "~" H 2250 5000 50  0001 C CNN
 	1    2250 5000

Commit message: [PCB] continue assigning footprints + special libraries of special holes referenced in the measurement schema of the field service manual
Parts:
- J301: footprint (none) -> atari-interconnect:DSUB-19_Female_Horizontal_P2.77x2.84mm_EdgePinOffset7.70mm_Housed_MountingHolesOffset9.12mm
Changed lines of the file:
@@
 F 0 "J301" H 5650 8300 50  0000 C CNN
 F 1 "DB-19S ACSI Port" H 5650 6300 50  0000 C CNN
-F 2 "" H 5650 7300 50  0001 C CNN
+F 2 "atari-interconnect:DSUB-19_Female_Horizontal_P2.77x2.84mm_EdgePinOffset7.70mm_Housed_MountingHolesOffset9.12mm" H 5650 7300 50  0001 C CNN
 F 3 "~" H 5650 7300 50  0001 C CNN
 	1    5650 7300

Commit message: Resolves #45 : [Atari STE]Use shielded connectors
Parts:
- J301: symbol Connector_Generic:Conn_01x19 -> Connector_Generic_Shielded:Conn_01x19_Shielded
Connections:
- wire segments 101 -> 102
Changed lines of the file:
@@
 $EndComp
 $Comp
-L Connector_Generic:Conn_01x19 J301
+L Connector_Generic_Shielded:Conn_01x19_Shielded J301
 U 1 1 60A88574
 P 5650 7300
 F 0 "J301" H 5650 8300 50  0000 C CNN
-F 1 "DB-19S ACSI Port" H 5650 6300 50  0000 C CNN
+F 1 "DB-19S ACSI Port" H 5650 8400 50  0000 C CNN
 F 2 "atari-interconnect:DSUB-19_Female_Horizontal_P2.77x2.84mm_EdgePinOffset7.70mm_Housed_MountingHolesOffset9.12mm" H 5650 7300 50  0001 C CNN
 F 3 "~" H 5650 7300 50  0001 C CNN
@@
 Wire Wire Line
 	3350 8750 3750 8750
+Text Label 5650 8600 1    50   ~ 0
+GND
+Wire Wire Line
+	5650 8600 5650 8400
 $EndSCHEMATC
