File: atari-16-32-bits/motherboards/c300780-001/subsheet_202.sch (KiCad schematic (older format))
At the start: 15 parts, among them J203 DB-25S Parallel port, U202 YM2149_PHY

Commit message: [PCB] Assign builtins footprint when possible - resistors, ports
Parts:
- R212, R220: footprint (none) -> Resistor_THT:R_Axial_DIN0204_L3.6mm_D1.6mm_P7.62mm_Horizontal
Changed lines of the file:
@@
 F 0 "R220" V 2700 2550 50  0000 C CNN
 F 1 "1K" V 2900 2550 50  0000 C CNN
-F 2 "" H 2800 2550 50  0001 C CNN
+F 2 "Resistor_THT:R_Axial_DIN0204_L3.6mm_D1.6mm_P7.62mm_Horizontal" H 2800 2550 50  0001 C CNN
 F 3 "~" H 2800 2550 50  0001 C CNN
 	1    2800 2550
@@
 F 0 "R212" H 2400 7300 50  0000 C CNN
 F 1 "3K3" H 2400 7200 50  0000 C CNN
-F 2 "" H 2250 7250 50  0001 C CNN
+F 2 "Resistor_THT:R_Axial_DIN0204_L3.6mm_D1.6mm_P7.62mm_Horizontal" H 2250 7250 50  0001 C CNN
 F 3 "~" H 2250 7250 50  0001 C CNN
 	1    2250 7250

Commit message: [PCB] continuing footprint assignement
Parts:
- J203: footprint (none) -> Connector_Dsub:DSUB-25_Female_Horizontal_P2.77x2.84mm_EdgePinOffset7.70mm_Housed_MountingHolesOffset9.12mm
Changed lines of the file:
@@
 F 0 "J203" H 5950 7600 50  0000 C CNN
 F 1 "DB-25S Parallel port" H 5950 5000 50  0000 C CNN
-F 2 "" H 5950 6300 50  0001 C CNN
+F 2 "Connector_Dsub:DSUB-25_Female_Horizontal_P2.77x2.84mm_EdgePinOffset7.70mm_Housed_MountingHolesOffset9.12mm" H 5950 6300 50  0001 C CNN
 F 3 "~" H 5950 6300 50  0001 C CNN
 	1    5950 6300

Commit message: Resolves #41 : [PCB] custom footprint library for passives
Parts:
- L209, L210, L211, L212, L213, L214, L215, L216, L217, L218: footprint (none) -> commons_passives_THT:Passive_THT_EMI_filter_W5.08mm_L7.62mm
- R212, R220: footprint Resistor_THT:R_Axial_DIN0204_L3.6mm_D1.6mm_P7.62mm_Horizontal -> commons_passives_THT:Passive_THT_resistor_W2.54mm_L12.70mm
Changed lines of the file:
@@
 F 0 "L209" H 3250 5625 50  0000 C CNN
 F 1 "EMI_Filter_LCL" H 3250 5550 50  0000 C CNN
-F 2 "" V 3250 5350 50  0001 C CNN
+F 2 "commons_passives_THT:Passive_THT_EMI_filter_W5.08mm_L7.62mm" V 3250 5350 50  0001 C CNN
 F 3 "http://www.murata.com/~/media/webrenewal/support/library/catalog/products/emc/emifil/c31e.ashx?la=en-gb" V 3250 5350 50  0001 C CNN
 	1    3250 5350
@@
 F 0 "L210" H 4000 5875 50  0000 C CNN
 F 1 "EMI_Filter_LCL" H 4000 5800 50  0000 C CNN
-F 2 "" V 4000 5600 50  0001 C CNN
+F 2 "commons_passives_THT:Passive_THT_EMI_filter_W5.08mm_L7.62mm" V 4000 5600 50  0001 C CNN
 F 3 "http://www.murata.com/~/media/webrenewal/support/library/catalog/products/emc/emifil/c31e.ashx?la=en-gb" V 4000 5600 50  0001 C CNN
 	1    4000 5600
@@
 F 0 "L211" H 3250 6125 50  0000 C CNN
 F 1 "EMI_Filter_LCL" H 3250 6050 50  0000 C CNN
-F 2 "" V 3250 5850 50  0001 C CNN
+F 2 "commons_passives_THT:Passive_THT_EMI_filter_W5.08mm_L7.62mm" V 3250 5850 50  0001 C CNN
 F 3 "http://www.murata.com/~/media/webrenewal/support/library/catalog/products/emc/emifil/c31e.ashx?la=en-gb" V 3250 5850 50  0001 C CNN
 	1    3250 5850
@@
 F 0 "L212" H 4000 6375 50  0000 C CNN
 F 1 "EMI_Filter_LCL" H 4000 6300 50  0000 C CNN
-F 2 "" V 4000 6100 50  0001 C CNN
+F 2 "commons_passives_THT:Passive_THT_EMI_filter_W5.08mm_L7.62mm" V 4000 6100 50  0001 C CNN
 F 3 "http://www.murata.com/~/media/webrenewal/support/library/catalog/products/emc/emifil/c31e.ashx?la=en-gb" V 4000 6100 50  0001 C CNN
 	1    4000 6100
@@
 F 0 "L213" H 3250 6625 50  0000 C CNN
 F 1 "EMI_Filter_LCL" H 3250 6550 50  0000 C CNN
-F 2 "" V 3250 6350 50  0001 C CNN
+F 2 "commons_passives_THT:Passive_THT_EMI_filter_W5.08mm_L7.62mm" V 3250 6350 50  0001 C CNN
 F 3 "http://www.murata.com/~/media/webrenewal/support/library/catalog/products/emc/emifil/c31e.ashx?la=en-gb" V 3250 6350 50  0001 C CNN
 	1    3250 6350
@@
 F 0 "L214" H 4000 6875 50  0000 C CNN
 F 1 "EMI_Filter_LCL" H 4000 6800 50  0000 C CNN
-F 2 "" V 4000 6600 50  0001 C CNN
+F 2 "commons_passives_THT:Passive_THT_EMI_filter_W5.08mm_L7.62mm" V 4000 6600 50  0001 C CNN
 F 3 "http://www.murata.com/~/media/webrenewal/support/library/catalog/products/emc/emifil/c31e.ashx?la=en-gb" V 4000 6600 50  0001 C CNN
 	1    4000 6600
@@
 F 0 "L215" H 3250 7125 50  0000 C CNN
 F 1 "EMI_Filter_LCL" H 3250 7050 50  0000 C CNN
-F 2 "" V 3250 6850 50  0001 C CNN
+F 2 "commons_passives_THT:Passive_THT_EMI_filter_W5.08mm_L7.62mm" V 3250 6850 50  0001 C CNN
 F 3 "http://www.murata.com/~/media/webrenewal/support/library/catalog/products/emc/emifil/c31e.ashx?la=en-gb" V 3250 6850 50  0001 C CNN
 	1    3250 6850
@@
 F 0 "L216" H 4000 7375 50  0000 C CNN
 F 1 "EMI_Filter_LCL" H 4000 7300 50  0000 C CNN
-F 2 "" V 4000 7100 50  0001 C CNN
+F 2 "commons_passives_THT:Passive_THT_EMI_filter_W5.08mm_L7.62mm" V 4000 7100 50  0001 C CNN
 F 3 "http://www.murata.com/~/media/webrenewal/support/library/catalog/products/emc/emifil/c31e.ashx?la=en-gb" V 4000 7100 50  0001 C CNN
 	1    4000 7100
@@
 F 0 "L217" H 3250 7625 50  0000 C CNN
 F 1 "EMI_Filter_LCL" H 3250 7550 50  0000 C CNN
-F 2 "" V 3250 7350 50  0001 C CNN
+F 2 "commons_passives_THT:Passive_THT_EMI_filter_W5.08mm_L7.62mm" V 3250 7350 50  0001 C CNN
 F 3 "http://www.murata.com/~/media/webrenewal/support/library/catalog/products/emc/emifil/c31e.ashx?la=en-gb" V 3250 7350 50  0001 C CNN
 	1    3250 7350
@@
 F 0 "L218" H 4000 7875 50  0000 C CNN
 F 1 "EMI_Filter_LCL" H 4000 7800 50  0000 C CNN
-F 2 "" V 4000 7600 50  0001 C CNN
+F 2 "commons_passives_THT:Passive_THT_EMI_filter_W5.08mm_L7.62mm" V 4000 7600 50  0001 C CNN
 F 3 "http://www.murata.com/~/media/webrenewal/support/library/catalog/products/emc/emifil/c31e.ashx?la=en-gb" V 4000 7600 50  0001 C CNN
 	1    4000 7600
@@
 F 0 "R220" V 2700 2550 50  0000 C CNN
 F 1 "1K" V 2900 2550 50  0000 C CNN
-F 2 "Resistor_THT:R_Axial_DIN0204_L3.6mm_D1.6mm_P7.62mm_Horizontal" H 2800 2550 50  0001 C CNN
+F 2 "commons_passives_THT:Passive_THT_resistor_W2.54mm_L12.70mm" H 2800 2550 50  0001 C CNN
 F 3 "~" H 2800 2550 50  0001 C CNN
 	1    2800 2550
@@
 F 0 "R212" H 2400 7300 50  0000 C CNN
 F 1 "3K3" H 2400 7200 50  0000 C CNN
-F 2 "Resistor_THT:R_Axial_DIN0204_L3.6mm_D1.6mm_P7.62mm_Horizontal" H 2250 7250 50  0001 C CNN
+F 2 "commons_passives_THT:Passive_THT_resistor_W2.54mm_L12.70mm" H 2250 7250 50  0001 C CNN
 F 3 "~" H 2250 7250 50  0001 C CNN
 	1    2250 7250

Commit message: [PCB] continue footprint assignation
Parts:
- C214: footprint (none) -> commons_passives_THT:Passive_THT_capacitor_ceramic_radial_W5.08mm_L6.35mm_X11.43mm
Changed lines of the file:
@@
 F 0 "C214" H 5825 2100 50  0000 L CNN
 F 1 "0.1uF" H 5825 1900 50  0000 L CNN
-F 2 "" H 5838 1850 50  0001 C CNN
+F 2 "commons_passives_THT:Passive_THT_capacitor_ceramic_radial_W5.08mm_L6.35mm_X11.43mm" H 5838 1850 50  0001 C CNN
 F 3 "~" H 5800 2000 50  0001 C CNN
 	1    5800 2000

Commit message: Resolves #45 : [Atari STE]Use shielded connectors
Parts:
- J203: symbol Connector_Generic:Conn_01x25 -> Connector_Generic_Shielded:Conn_01x25_Shielded
Connections:
- wire segments 90 -> 91
Changed lines of the file:
@@
 	2700 7250 2950 7250
 $Comp
-L Connector_Generic:Conn_01x25 J203
+L Connector_Generic_Shielded:Conn_01x25_Shielded J203
 U 1 1 60964926
 P 5950 6300
 F 0 "J203" H 5950 7600 50  0000 C CNN
-F 1 "DB-25S Parallel port" H 5950 5000 50  0000 C CNN
+F 1 "DB-25S Parallel port" H 5950 7700 50  0000 C CNN
 F 2 "Connector_Dsub:DSUB-25_Female_Horizontal_P2.77x2.84mm_EdgePinOffset7.70mm_Housed_MountingHolesOffset9.12mm" H 5950 6300 50  0001 C CNN
 F 3 "~" H 5950 6300 50  0001 C CNN
@@
 Text Notes 2200 2250 0    55   ~ 0
 To LMC1992
+Text Label 5950 7900 1    50   ~ 0
+GND
+Wire Wire Line
+	5950 7900 5950 7700
 $EndSCHEMATC

Commit message: Resolves #46 : [PCB] Footprints for shielded ports should have pins named 'SH'
Parts:
- J203: footprint Connector_Dsub:DSUB-25_Female_Horizontal_P2.77x2.84mm_EdgePinOffset7.70mm_Housed_MountingHolesOffset9.12mm -> commons-interconnect_THT:DSUB-25_Female_Horizontal_P2.77x2.84mm_EdgePinOffset7.70mm_Housed_MountingHolesOffset9.12mm
Changed lines of the file:
@@
 F 0 "J203" H 5950 7600 50  0000 C CNN
 F 1 "DB-25S Parallel port" H 5950 7700 50  0000 C CNN
-F 2 "Connector_Dsub:DSUB-25_Female_Horizontal_P2.77x2.84mm_EdgePinOffset7.70mm_Housed_MountingHolesOffset9.12mm" H 5950 6300 50  0001 C CNN
+F 2 "commons-interconnect_THT:DSUB-25_Female_Horizontal_P2.77x2.84mm_EdgePinOffset7.70mm_Housed_MountingHolesOffset9.12mm" H 5950 6300 50  0001 C CNN
 F 3 "~" H 5950 6300 50  0001 C CNN
 	1    5950 6300
