File: atari-16-32-bits/motherboards/c300780-001/subsheet_204.sch (KiCad schematic (older format))
At the start: 17 parts, among them J204 DB-25P Serial Port RS-232, U206 MC1488_QUAD_LINE_EIA-232D_DRI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, U207 MC1489_QUAD_LINE_EIA-232D_REC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

Commit message: [PCB] Assign builtins footprint when possible - resistors, ports
Parts:
- J204: footprint (none) -> Connector_Dsub:DSUB-25_Male_Horizontal_P2.77x2.84mm_EdgePinOffset7.70mm_Housed_MountingHolesOffset9.12mm
Changed lines of the file:
@@
 F 0 "J204" H 6000 7650 50  0000 C CNN
 F 1 "DB-25P Serial Port RS-232" H 6000 5050 50  0000 C CNN
-F 2 "" H 6000 6350 50  0001 C CNN
+F 2 "Connector_Dsub:DSUB-25_Male_Horizontal_P2.77x2.84mm_EdgePinOffset7.70mm_Housed_MountingHolesOffset9.12mm" H 6000 6350 50  0001 C CNN
 F 3 "~" H 6000 6350 50  0001 C CNN
 	1    6000 6350

Commit message: Resolves #41 : [PCB] custom footprint library for passives
Parts:
- L219, L220, L221, L222, L223, L224, L225: footprint (none) -> commons_passives_THT:Passive_THT_EMI_filter_W5.08mm_L7.62mm
Changed lines of the file:
@@
 F 0 "L219" H 4000 5875 50  0000 C CNN
 F 1 "EMI_Filter_LCL" H 4000 5800 50  0000 C CNN
-F 2 "" V 4000 5600 50  0001 C CNN
+F 2 "commons_passives_THT:Passive_THT_EMI_filter_W5.08mm_L7.62mm" V 4000 5600 50  0001 C CNN
 F 3 "http://www.murata.com/~/media/webrenewal/support/library/catalog/products/emc/emifil/c31e.ashx?la=en-gb" V 4000 5600 50  0001 C CNN
 	1    4000 5600
@@
 F 0 "L220" H 3250 6125 50  0000 C CNN
 F 1 "EMI_Filter_LCL" H 3250 6050 50  0000 C CNN
-F 2 "" V 3250 5850 50  0001 C CNN
+F 2 "commons_passives_THT:Passive_THT_EMI_filter_W5.08mm_L7.62mm" V 3250 5850 50  0001 C CNN
 F 3 "http://www.murata.com/~/media/webrenewal/support/library/catalog/products/emc/emifil/c31e.ashx?la=en-gb" V 3250 5850 50  0001 C CNN
 	1    3250 5850
@@
 F 0 "L221" H 4000 6375 50  0000 C CNN
 F 1 "EMI_Filter_LCL" H 4000 6300 50  0000 C CNN
-F 2 "" V 4000 6100 50  0001 C CNN
+F 2 "commons_passives_THT:Passive_THT_EMI_filter_W5.08mm_L7.62mm" V 4000 6100 50  0001 C CNN
 F 3 "http://www.murata.com/~/media/webrenewal/support/library/catalog/products/emc/emifil/c31e.ashx?la=en-gb" V 4000 6100 50  0001 C CNN
 	1    4000 6100
@@
 F 0 "L222" H 3250 6625 50  0000 C CNN
 F 1 "EMI_Filter_LCL" H 3250 6550 50  0000 C CNN
-F 2 "" V 3250 6350 50  0001 C CNN
+F 2 "commons_passives_THT:Passive_THT_EMI_filter_W5.08mm_L7.62mm" V 3250 6350 50  0001 C CNN
 F 3 "http://www.murata.com/~/media/webrenewal/support/library/catalog/products/emc/emifil/c31e.ashx?la=en-gb" V 3250 6350 50  0001 C CNN
 	1    3250 6350
@@
 F 0 "L223" H 4000 6875 50  0000 C CNN
 F 1 "EMI_Filter_LCL" H 4000 6800 50  0000 C CNN
-F 2 "" V 4000 6600 50  0001 C CNN
+F 2 "commons_passives_THT:Passive_THT_EMI_filter_W5.08mm_L7.62mm" V 4000 6600 50  0001 C CNN
 F 3 "http://www.murata.com/~/media/webrenewal/support/library/catalog/products/emc/emifil/c31e.ashx?la=en-gb" V 4000 6600 50  0001 C CNN
 	1    4000 6600
@@
 F 0 "L224" H 3250 7125 50  0000 C CNN
 F 1 "EMI_Filter_LCL" H 3250 7050 50  0000 C CNN
-F 2 "" V 3250 6850 50  0001 C CNN
+F 2 "commons_passives_THT:Passive_THT_EMI_filter_W5.08mm_L7.62mm" V 3250 6850 50  0001 C CNN
 F 3 "http://www.murata.com/~/media/webrenewal/support/library/catalog/products/emc/emifil/c31e.ashx?la=en-gb" V 3250 6850 50  0001 C CNN
 	1    3250 6850
@@
 F 0 "L225" H 4000 7375 50  0000 C CNN
 F 1 "EMI_Filter_LCL" H 4000 7300 50  0000 C CNN
-F 2 "" V 4000 7100 50  0001 C CNN
+F 2 "commons_passives_THT:Passive_THT_EMI_filter_W5.08mm_L7.62mm" V 4000 7100 50  0001 C CNN
 F 3 "http://www.murata.com/~/media/webrenewal/support/library/catalog/products/emc/emifil/c31e.ashx?la=en-gb" V 4000 7100 50  0001 C CNN
 	1    4000 7100

Commit message: [PCB] continue footprint assignation
Parts:
- C203, C206, C228: footprint (none) -> commons_passives_THT:Passive_THT_capacitor_ceramic_radial_W5.08mm_L6.35mm_X11.43mm
- C222, C223, C224, C225: footprint (none) -> commons_passives_THT:Passive_THT_capacitor_W2.54mm_L10.16mm
Changed lines of the file:
@@
 F 0 "C222" H 1125 3950 50  0000 L CNN
 F 1 "100pF" H 1125 3750 50  0000 L CNN
-F 2 "" H 1138 3700 50  0001 C CNN
+F 2 "commons_passives_THT:Passive_THT_capacitor_W2.54mm_L10.16mm" H 1138 3700 50  0001 C CNN
 F 3 "~" H 1100 3850 50  0001 C CNN
 	1    1100 3850
@@
 F 0 "C223" H 1625 3950 50  0000 L CNN
 F 1 "100pF" H 1625 3750 50  0000 L CNN
-F 2 "" H 1638 3700 50  0001 C CNN
+F 2 "commons_passives_THT:Passive_THT_capacitor_W2.54mm_L10.16mm" H 1638 3700 50  0001 C CNN
 F 3 "~" H 1600 3850 50  0001 C CNN
 	1    1600 3850
@@
 F 0 "C224" H 2125 3950 50  0000 L CNN
 F 1 "100pF" H 2125 3750 50  0000 L CNN
-F 2 "" H 2138 3700 50  0001 C CNN
+F 2 "commons_passives_THT:Passive_THT_capacitor_W2.54mm_L10.16mm" H 2138 3700 50  0001 C CNN
 F 3 "~" H 2100 3850 50  0001 C CNN
 	1    2100 3850
@@
 F 0 "C225" H 2625 3950 50  0000 L CNN
 F 1 "100pF" H 2625 3750 50  0000 L CNN
-F 2 "" H 2638 3700 50  0001 C CNN
+F 2 "commons_passives_THT:Passive_THT_capacitor_W2.54mm_L10.16mm" H 2638 3700 50  0001 C CNN
 F 3 "~" H 2600 3850 50  0001 C CNN
 	1    2600 3850
@@
 F 0 "C228" H 6925 3950 50  0000 L CNN
 F 1 "0.1uF" H 6925 3750 50  0000 L CNN
-F 2 "" H 6938 3700 50  0001 C CNN
+F 2 "commons_passives_THT:Passive_THT_capacitor_ceramic_radial_W5.08mm_L6.35mm_X11.43mm" H 6938 3700 50  0001 C CNN
 F 3 "~" H 6900 3850 50  0001 C CNN
 	1    6900 3850
@@
 F 0 "C203" H 6025 2150 50  0000 L CNN
 F 1 "0.1uF" H 6025 1950 50  0000 L CNN
-F 2 "" H 6038 1900 50  0001 C CNN
+F 2 "commons_passives_THT:Passive_THT_capacitor_ceramic_radial_W5.08mm_L6.35mm_X11.43mm" H 6038 1900 50  0001 C CNN
 F 3 "~" H 6000 2050 50  0001 C CNN
 	1    6000 2050
@@
 F 0 "C206" H 6525 2150 50  0000 L CNN
 F 1 "0.1uF" H 6525 1950 50  0000 L CNN
-F 2 "" H 6538 1900 50  0001 C CNN
+F 2 "commons_passives_THT:Passive_THT_capacitor_ceramic_radial_W5.08mm_L6.35mm_X11.43mm" H 6538 1900 50  0001 C CNN
 F 3 "~" H 6500 2050 50  0001 C CNN
 	1    6500 2050

Commit message: Resolves #45 : [Atari STE]Use shielded connectors
Parts:
- J204: symbol Connector_Generic:Conn_01x25 -> Connector_Generic_Shielded:Conn_01x25_Shielded
Connections:
- wire segments 70 -> 71
Changed lines of the file:
@@
 	3550 5750 4550 5750
 $Comp
-L Connector_Generic:Conn_01x25 J204
+L Connector_Generic_Shielded:Conn_01x25_Shielded J204
 U 1 1 609B5CCF
 P 6000 6350
 F 0 "J204" H 6000 7650 50  0000 C CNN
-F 1 "DB-25P Serial Port RS-232" H 6000 5050 50  0000 C CNN
+F 1 "DB-25P Serial Port RS-232" H 6000 7750 50  0000 C CNN
 F 2 "Connector_Dsub:DSUB-25_Male_Horizontal_P2.77x2.84mm_EdgePinOffset7.70mm_Housed_MountingHolesOffset9.12mm" H 6000 6350 50  0001 C CNN
 F 3 "~" H 6000 6350 50  0001 C CNN
@@
 	1    0    0    -1
 $EndComp
+Text Label 6000 7950 1    50   ~ 0
+GND
+Wire Wire Line
+	6000 7950 6000 7750
 $EndSCHEMATC

Commit message: Resolves #46 : [PCB] Footprints for shielded ports should have pins named 'SH'
Parts:
- J204: footprint Connector_Dsub:DSUB-25_Male_Horizontal_P2.77x2.84mm_EdgePinOffset7.70mm_Housed_MountingHolesOffset9.12mm -> commons-interconnect_THT:DSUB-25_Male_Horizontal_P2.77x2.84mm_EdgePinOffset7.70mm_Housed_MountingHolesOffset9.12mm
Changed lines of the file:
@@
 F 0 "J204" H 6000 7650 50  0000 C CNN
 F 1 "DB-25P Serial Port RS-232" H 6000 7750 50  0000 C CNN
-F 2 "Connector_Dsub:DSUB-25_Male_Horizontal_P2.77x2.84mm_EdgePinOffset7.70mm_Housed_MountingHolesOffset9.12mm" H 6000 6350 50  0001 C CNN
+F 2 "commons-interconnect_THT:DSUB-25_Male_Horizontal_P2.77x2.84mm_EdgePinOffset7.70mm_Housed_MountingHolesOffset9.12mm" H 6000 6350 50  0001 C CNN
 F 3 "~" H 6000 6350 50  0001 C CNN
 	1    6000 6350
