File: atari-16-32-bits/motherboards/c300780-001/subsheet_104.sch (KiCad schematic (older format))
At the start: 8 parts, among them U104 LM555_TIMER_PHY

Commit message: [PCB] Assign builtins footprint when possible - resistors, ports
Parts:
- D100: footprint (none) -> Diode_THT:D_DO-35_SOD27_P7.62mm_Horizontal
- R100, R101: footprint (none) -> Resistor_THT:R_Axial_DIN0204_L3.6mm_D1.6mm_P7.62mm_Horizontal
Changed lines of the file:
@@
 F 0 "R100" H 2650 1400 50  0000 C CNN
 F 1 "10K" H 2650 1300 50  0000 C CNN
-F 2 "" V 2540 1340 50  0001 C CNN
+F 2 "Resistor_THT:R_Axial_DIN0204_L3.6mm_D1.6mm_P7.62mm_Horizontal" V 2540 1340 50  0001 C CNN
 F 3 "~" H 2500 1350 50  0001 C CNN
 	1    2500 1350
@@
 F 0 "D100" V 2950 1550 50  0000 C CNN
 F 1 "1N914" V 3050 1550 50  0000 C CNN
-F 2 "" H 3000 1350 50  0001 C CNN
+F 2 "Diode_THT:D_DO-35_SOD27_P7.62mm_Horizontal" H 3000 1350 50  0001 C CNN
 F 3 "~" H 3000 1350 50  0001 C CNN
 	1    3000 1350
@@
 F 0 "R101" H 6650 1400 50  0000 C CNN
 F 1 "12K" H 6650 1300 50  0000 C CNN
-F 2 "" V 6540 1340 50  0001 C CNN
+F 2 "Resistor_THT:R_Axial_DIN0204_L3.6mm_D1.6mm_P7.62mm_Horizontal" V 6540 1340 50  0001 C CNN
 F 3 "~" H 6500 1350 50  0001 C CNN
 	1    6500 1350

Commit message: Resolves #41 : [PCB] custom footprint library for passives
Parts:
- D100: footprint Diode_THT:D_DO-35_SOD27_P7.62mm_Horizontal -> commons_passives_THT:Passive_THT_diode_W2.54mm_L12.70mm
- R100, R101: footprint Resistor_THT:R_Axial_DIN0204_L3.6mm_D1.6mm_P7.62mm_Horizontal -> commons_passives_THT:Passive_THT_resistor_W2.54mm_L12.70mm
Changed lines of the file:
@@
 F 0 "R100" H 2650 1400 50  0000 C CNN
 F 1 "10K" H 2650 1300 50  0000 C CNN
-F 2 "Resistor_THT:R_Axial_DIN0204_L3.6mm_D1.6mm_P7.62mm_Horizontal" V 2540 1340 50  0001 C CNN
+F 2 "commons_passives_THT:Passive_THT_resistor_W2.54mm_L12.70mm" V 2540 1340 50  0001 C CNN
 F 3 "~" H 2500 1350 50  0001 C CNN
 	1    2500 1350
@@
 F 0 "D100" V 2950 1550 50  0000 C CNN
 F 1 "1N914" V 3050 1550 50  0000 C CNN
-F 2 "Diode_THT:D_DO-35_SOD27_P7.62mm_Horizontal" H 3000 1350 50  0001 C CNN
+F 2 "commons_passives_THT:Passive_THT_diode_W2.54mm_L12.70mm" H 3000 1350 50  0001 C CNN
 F 3 "~" H 3000 1350 50  0001 C CNN
 	1    3000 1350
@@
 F 0 "R101" H 6650 1400 50  0000 C CNN
 F 1 "12K" H 6650 1300 50  0000 C CNN
-F 2 "Resistor_THT:R_Axial_DIN0204_L3.6mm_D1.6mm_P7.62mm_Horizontal" V 6540 1340 50  0001 C CNN
+F 2 "commons_passives_THT:Passive_THT_resistor_W2.54mm_L12.70mm" V 6540 1340 50  0001 C CNN
 F 3 "~" H 6500 1350 50  0001 C CNN
 	1    6500 1350

Commit message: [PCB] continue footprint assignation
Parts:
- C100: footprint (none) -> commons_passives_THT:Passive_THT_capacitor_polarized_W5.08mm_L17.78mm
- C101: footprint (none) -> commons_passives_THT:Passive_THT_capacitor_W2.54mm_L10.16mm
- C102: footprint (none) -> commons_passives_THT:Passive_THT_capacitor_polarized_W6.35mm_L20.32mm
Changed lines of the file:
@@
 F 0 "C100" H 2800 2150 50  0000 L CNN
 F 1 "10uF" H 2800 1950 50  0000 L CNN
-F 2 "" H 2750 2050 50  0001 C CNN
+F 2 "commons_passives_THT:Passive_THT_capacitor_polarized_W5.08mm_L17.78mm" H 2750 2050 50  0001 C CNN
 F 3 "~" H 2750 2050 50  0001 C CNN
 	1    2750 2050
@@
 F 0 "C101" H 6050 2350 50  0000 L CNN
 F 1 "0.01uF" H 6050 2150 50  0000 L CNN
-F 2 "" H 6000 2250 50  0001 C CNN
+F 2 "commons_passives_THT:Passive_THT_capacitor_W2.54mm_L10.16mm" H 6000 2250 50  0001 C CNN
 F 3 "~" H 6000 2250 50  0001 C CNN
 	1    6000 2250
@@
 F 0 "C102" H 6550 2150 50  0000 L CNN
 F 1 "22uF" H 6550 1950 50  0000 L CNN
-F 2 "" H 6500 2050 50  0001 C CNN
+F 2 "commons_passives_THT:Passive_THT_capacitor_polarized_W6.35mm_L20.32mm" H 6500 2050 50  0001 C CNN
 F 3 "~" H 6500 2050 50  0001 C CNN
 	1    6500 2050

Commit message: [PCB] assign reset button footprint, adjust ikbd connector and din-14 floppy drive connector
Parts:
- S100: footprint (none) -> atari-interconnect:switch-spdt-momentary-action_Reset_pushbutton
Changed lines of the file:
@@
 F 0 "S100" H 2100 1870 50  0000 C CNN
 F 1 "RESET switch" H 2100 1500 50  0000 C CNN
-F 2 "" H 2100 1700 50  0001 C CNN
+F 2 "atari-interconnect:switch-spdt-momentary-action_Reset_pushbutton" H 2100 1700 50  0001 C CNN
 F 3 "~" H 2100 1700 50  0001 C CNN
 	1    2100 1700

Commit message: Resolves #48 : [Schematic][PCB] Reset button should be shielded
Parts:
- S100: symbol Switch:SW_SPDT -> reset-switch:SW_SPDT_Reset_switch
Connections:
- net GND: now also S100.SH
Changed lines of the file:
@@
 	6500 1700 6500 1900
 $Comp
-L Switch:SW_SPDT S100
+L reset-switch:SW_SPDT_Reset_switch S100
 U 1 1 608C05EE
 P 2100 1700
-F 0 "S100" H 2100 1870 50  0000 C CNN
-F 1 "RESET switch" H 2100 1500 50  0000 C CNN
+F 0 "S100" H 2000 2200 50  0000 L CNN
+F 1 "RESET switch" H 1850 2100 50  0000 L CNN
 F 2 "atari-interconnect:switch-spdt-momentary-action_Reset_pushbutton" H 2100 1700 50  0001 C CNN
 F 3 "~" H 2100 1700 50  0001 C CNN
@@
 Wire Wire Line
 	3850 1800 4100 1800
+Text Label 2100 2200 1    50   ~ 0
+GND
+Wire Wire Line
+	2100 2000 2100 2200
 $EndSCHEMATC
