File: atari-16-32-bits/motherboards/c300780-001/subsheet_101.sch (KiCad schematic (older format))
At the start: 6 parts, among them U101 ST_BLITTER_PHY

Commit message: [PCB] Assign builtins footprint when possible - resistors, ports
Parts:
- R106, R111, R112: footprint (none) -> Resistor_THT:R_Axial_DIN0204_L3.6mm_D1.6mm_P7.62mm_Horizontal
Changed lines of the file:
@@
 F 0 "R111" V 6900 4000 50  0000 C CNN
 F 1 "0" V 6700 4000 50  0000 C CNN
-F 2 "" V 6840 3990 50  0001 C CNN
+F 2 "Resistor_THT:R_Axial_DIN0204_L3.6mm_D1.6mm_P7.62mm_Horizontal" V 6840 3990 50  0001 C CNN
 F 3 "~" H 6800 4000 50  0001 C CNN
 	1    6800 4000
@@
 F 0 "R112" V 6900 4500 50  0000 C CNN
 F 1 "0" V 6700 4500 50  0000 C CNN
-F 2 "" V 6840 4490 50  0001 C CNN
+F 2 "Resistor_THT:R_Axial_DIN0204_L3.6mm_D1.6mm_P7.62mm_Horizontal" V 6840 4490 50  0001 C CNN
 F 3 "~" H 6800 4500 50  0001 C CNN
 	1    6800 4500
@@
 F 0 "R106" V 6900 3000 50  0000 C CNN
 F 1 "4K7" V 6700 3000 50  0000 C CNN
-F 2 "" V 6840 2990 50  0001 C CNN
+F 2 "Resistor_THT:R_Axial_DIN0204_L3.6mm_D1.6mm_P7.62mm_Horizontal" V 6840 2990 50  0001 C CNN
 F 3 "~" H 6800 3000 50  0001 C CNN
 	1    6800 3000

Commit message: Resolves #41 : [PCB] custom footprint library for passives
Parts:
- R106, R111, R112: footprint Resistor_THT:R_Axial_DIN0204_L3.6mm_D1.6mm_P7.62mm_Horizontal -> commons_passives_THT:Passive_THT_resistor_W2.54mm_L12.70mm
Changed lines of the file:
@@
 F 0 "R111" V 6900 4000 50  0000 C CNN
 F 1 "0" V 6700 4000 50  0000 C CNN
-F 2 "Resistor_THT:R_Axial_DIN0204_L3.6mm_D1.6mm_P7.62mm_Horizontal" V 6840 3990 50  0001 C CNN
+F 2 "commons_passives_THT:Passive_THT_resistor_W2.54mm_L12.70mm" V 6840 3990 50  0001 C CNN
 F 3 "~" H 6800 4000 50  0001 C CNN
 	1    6800 4000
@@
 F 0 "R112" V 6900 4500 50  0000 C CNN
 F 1 "0" V 6700 4500 50  0000 C CNN
-F 2 "Resistor_THT:R_Axial_DIN0204_L3.6mm_D1.6mm_P7.62mm_Horizontal" V 6840 4490 50  0001 C CNN
+F 2 "commons_passives_THT:Passive_THT_resistor_W2.54mm_L12.70mm" V 6840 4490 50  0001 C CNN
 F 3 "~" H 6800 4500 50  0001 C CNN
 	1    6800 4500
@@
 F 0 "R106" V 6900 3000 50  0000 C CNN
 F 1 "4K7" V 6700 3000 50  0000 C CNN
-F 2 "Resistor_THT:R_Axial_DIN0204_L3.6mm_D1.6mm_P7.62mm_Horizontal" V 6840 2990 50  0001 C CNN
+F 2 "commons_passives_THT:Passive_THT_resistor_W2.54mm_L12.70mm" V 6840 2990 50  0001 C CNN
 F 3 "~" H 6800 3000 50  0001 C CNN
 	1    6800 3000

Commit message: [PCB] continue footprint assignation
Parts:
- C105, C106: footprint (none) -> commons_passives_THT:Passive_THT_capacitor_ceramic_radial_W5.08mm_L6.35mm_X11.43mm
Changed lines of the file:
@@
 F 0 "C105" H 6525 2100 50  0000 L CNN
 F 1 "0.1uF" H 6525 1900 50  0000 L CNN
-F 2 "" H 6538 1850 50  0001 C CNN
+F 2 "commons_passives_THT:Passive_THT_capacitor_ceramic_radial_W5.08mm_L6.35mm_X11.43mm" H 6538 1850 50  0001 C CNN
 F 3 "~" H 6500 2000 50  0001 C CNN
 	1    6500 2000
@@
 F 0 "C106" H 7025 2100 50  0000 L CNN
 F 1 "0.1uF" H 7025 1900 50  0000 L CNN
-F 2 "" H 7038 1850 50  0001 C CNN
+F 2 "commons_passives_THT:Passive_THT_capacitor_ceramic_radial_W5.08mm_L6.35mm_X11.43mm" H 7038 1850 50  0001 C CNN
 F 3 "~" H 7000 2000 50  0001 C CNN
 	1    7000 2000

Commit message: [PCB][bug] fixed association for U101 and U300_PLCC
Parts:
- U101: footprint Package_LCC:LCC-68_THT-Socket -> Package_LCC:PLCC-68_THT-Socket
Changed lines of the file:
@@
 F 0 "U101" H 4500 5000 50  0000 L TNN
 F 1 "ST_BLITTER_PHY" H 4500 4900 50  0000 L TNB
-F 2 "Package_LCC:LCC-68_THT-Socket" H 4500 5100 50  0001 L TNN
+F 2 "Package_LCC:PLCC-68_THT-Socket" H 4500 5100 50  0001 L TNN
 F 3 "" H 3600 3550 50  0001 C CNN
 	1    3600 3550
