File: atari-16-32-bits/motherboards/c300780-001/subsheet_300.sch (KiCad schematic (older format))
At the start: 4 parts, among them U300_DIP40 ST_DMA_DIP40_PHY, U300_PLCC44 ST_DMA_PLCC44_PHY

Commit message: [PCB] Assign builtins footprint when possible - resistors, ports
Parts:
- R303: footprint (none) -> Resistor_THT:R_Axial_DIN0204_L3.6mm_D1.6mm_P7.62mm_Horizontal
Changed lines of the file:
@@
 F 0 "R303" V 4150 2000 50  0000 C CNN
 F 1 "1K" V 4350 2000 50  0000 C CNN
-F 2 "" H 4250 2000 50  0001 C CNN
+F 2 "Resistor_THT:R_Axial_DIN0204_L3.6mm_D1.6mm_P7.62mm_Horizontal" H 4250 2000 50  0001 C CNN
 F 3 "~" H 4250 2000 50  0001 C CNN
 	1    4250 2000

Commit message: Resolves #41 : [PCB] custom footprint library for passives
Parts:
- R303: footprint Resistor_THT:R_Axial_DIN0204_L3.6mm_D1.6mm_P7.62mm_Horizontal -> commons_passives_THT:Passive_THT_resistor_W2.54mm_L12.70mm
Changed lines of the file:
@@
 F 0 "R303" V 4150 2000 50  0000 C CNN
 F 1 "1K" V 4350 2000 50  0000 C CNN
-F 2 "Resistor_THT:R_Axial_DIN0204_L3.6mm_D1.6mm_P7.62mm_Horizontal" H 4250 2000 50  0001 C CNN
+F 2 "commons_passives_THT:Passive_THT_resistor_W2.54mm_L12.70mm" H 4250 2000 50  0001 C CNN
 F 3 "~" H 4250 2000 50  0001 C CNN
 	1    4250 2000

Commit message: [PCB] continue footprint assignation
Parts:
- C302: footprint (none) -> commons_passives_THT:Passive_THT_capacitor_ceramic_radial_W5.08mm_L6.35mm_X11.43mm
Changed lines of the file:
@@
 F 0 "C302" H 3025 4600 50  0000 L CNN
 F 1 "0.1uF" H 3025 4400 50  0000 L CNN
-F 2 "" H 3038 4350 50  0001 C CNN
+F 2 "commons_passives_THT:Passive_THT_capacitor_ceramic_radial_W5.08mm_L6.35mm_X11.43mm" H 3038 4350 50  0001 C CNN
 F 3 "~" H 3000 4500 50  0001 C CNN
 	1    3000 4500

Commit message: [PCB][bug] fixed association for U101 and U300_PLCC
Parts:
- U300_PLCC44: footprint Package_LCC:LCC-44_THT-Socket -> Package_LCC:PLCC-44_THT-Socket
Changed lines of the file:
@@
 F 0 "U300_PLCC44" H 6300 4550 50  0000 L TNN
 F 1 "ST_DMA_PLCC44_PHY" H 6300 4450 50  0000 L TNB
-F 2 "Package_LCC:LCC-44_THT-Socket" H 6300 4650 50  0001 L TNN
+F 2 "Package_LCC:PLCC-44_THT-Socket" H 6300 4650 50  0001 L TNN
 F 3 "https://docs.dev-docs.org/htm/search.php?find=Atari+STBook+Schematic+" H 6300 4750 50  0001 L TNN
 	1    5700 3450
