File: atari-16-32-bits/motherboards/c300780-001/subsheet_105.sch (KiCad schematic (older format))
At the start: 5 parts, among them J100 Power

Commit message: [PCB] continuing footprint assignement
Parts:
- J100: footprint (none) -> Connector_Molex:Molex_KK-254_AE-6410-05A_1x05_P2.54mm_Vertical
Changed lines of the file:
@@
 F 0 "J100" H 1300 2200 50  0000 C CNN
 F 1 "Power" H 1300 1500 50  0000 C CNN
-F 2 "" H 1300 1900 50  0001 C CNN
+F 2 "Connector_Molex:Molex_KK-254_AE-6410-05A_1x05_P2.54mm_Vertical" H 1300 1900 50  0001 C CNN
 F 3 "~" H 1300 1900 50  0001 C CNN
 	1    1300 1900

Commit message: [PCB] continue footprint assignation
Parts:
- C104, C108: footprint (none) -> commons_passives_THT:Passive_THT_capacitor_ceramic_radial_W5.08mm_L6.35mm_X11.43mm
- C107: footprint (none) -> commons_passives_THT:Passive_THT_capacitor_polarized_W6.35mm_L20.32mm
Changed lines of the file:
@@
 F 0 "C107" H 3775 2100 50  0000 L CNN
 F 1 "100uF" H 3775 1900 50  0000 L CNN
-F 2 "" H 3750 2000 50  0001 C CNN
+F 2 "commons_passives_THT:Passive_THT_capacitor_polarized_W6.35mm_L20.32mm" H 3750 2000 50  0001 C CNN
 F 3 "~" H 3750 2000 50  0001 C CNN
 	1    3750 2000
@@
 F 0 "C104" H 3025 2100 50  0000 L CNN
 F 1 "0.1uF" H 3025 1900 50  0000 L CNN
-F 2 "" H 3038 1850 50  0001 C CNN
+F 2 "commons_passives_THT:Passive_THT_capacitor_ceramic_radial_W5.08mm_L6.35mm_X11.43mm" H 3038 1850 50  0001 C CNN
 F 3 "~" H 3000 2000 50  0001 C CNN
 	1    3000 2000
@@
 F 0 "C108" H 4275 2100 50  0000 L CNN
 F 1 "0.1uF" H 4275 1900 50  0000 L CNN
-F 2 "" H 4288 1850 50  0001 C CNN
+F 2 "commons_passives_THT:Passive_THT_capacitor_ceramic_radial_W5.08mm_L6.35mm_X11.43mm" H 4288 1850 50  0001 C CNN
 F 3 "~" H 4250 2000 50  0001 C CNN
 	1    4250 2000

Commit message: [PCB] continue footprints assignements
Parts:
- C103: footprint (none) -> commons_passives_THT:Passive_THT_capacitor_polarized_W16.51mm_L45.72mm
Changed lines of the file:
@@
 F 0 "C103" H 2525 2100 50  0000 L CNN
 F 1 "4700uF" H 2525 1900 50  0000 L CNN
-F 2 "" H 2500 2000 50  0001 C CNN
+F 2 "commons_passives_THT:Passive_THT_capacitor_polarized_W16.51mm_L45.72mm" H 2500 2000 50  0001 C CNN
 F 3 "~" H 2500 2000 50  0001 C CNN
 	1    2500 2000

Commit message: [PCB] done E0..7 and RAM connectors
Parts:
- J100: footprint Connector_Molex:Molex_KK-254_AE-6410-05A_1x05_P2.54mm_Vertical -> Connector_Molex:Molex_KK-254_AE-6410-06A_1x06_P2.54mm_Vertical
Changed lines of the file:
@@
 F 0 "J100" H 1300 2200 50  0000 C CNN
 F 1 "Power" H 1300 1500 50  0000 C CNN
-F 2 "Connector_Molex:Molex_KK-254_AE-6410-05A_1x05_P2.54mm_Vertical" H 1300 1900 50  0001 C CNN
+F 2 "Connector_Molex:Molex_KK-254_AE-6410-06A_1x06_P2.54mm_Vertical" H 1300 1900 50  0001 C CNN
 F 3 "~" H 1300 1900 50  0001 C CNN
 	1    1300 1900
