File: atari-16-32-bits/motherboards/c300780-001/subsheet_203.sch (KiCad schematic (older format))
At the start: 14 parts, among them U203 MC68901_DIP_48_PHY, U209 74LS86_PHY, U211 74LS04_PHY, U900 74LS164_PHY, Y200 2.4576 MHz

Commit message: [PCB] Assign builtins footprint when possible - resistors, ports
Parts:
- R215, R216, R217: footprint (none) -> Resistor_THT:R_Axial_DIN0204_L3.6mm_D1.6mm_P7.62mm_Horizontal
Changed lines of the file:
@@
 F 0 "R217" V 6150 3250 50  0000 C CNN
 F 1 "4K7" V 6350 3250 50  0000 C CNN
-F 2 "" H 6250 3250 50  0001 C CNN
+F 2 "Resistor_THT:R_Axial_DIN0204_L3.6mm_D1.6mm_P7.62mm_Horizontal" H 6250 3250 50  0001 C CNN
 F 3 "~" H 6250 3250 50  0001 C CNN
 	1    6250 3250
@@
 F 0 "R215" V 6150 2750 50  0000 C CNN
 F 1 "4K7" V 6350 2750 50  0000 C CNN
-F 2 "" H 6250 2750 50  0001 C CNN
+F 2 "Resistor_THT:R_Axial_DIN0204_L3.6mm_D1.6mm_P7.62mm_Horizontal" H 6250 2750 50  0001 C CNN
 F 3 "~" H 6250 2750 50  0001 C CNN
 	1    6250 2750
@@
 F 0 "R216" V 6150 3750 50  0000 C CNN
 F 1 "4K7" V 6350 3750 50  0000 C CNN
-F 2 "" H 6250 3750 50  0001 C CNN
+F 2 "Resistor_THT:R_Axial_DIN0204_L3.6mm_D1.6mm_P7.62mm_Horizontal" H 6250 3750 50  0001 C CNN
 F 3 "~" H 6250 3750 50  0001 C CNN
 	1    6250 3750

Commit message: [PCB] continuing footprint assignement
Parts:
- Y200: footprint (none) -> Crystal:Crystal_HC18-U_Horizontal
Changed lines of the file:
@@
 F 0 "Y200" H 6250 1900 50  0000 C CNN
 F 1 "2.4576 MHz" H 6250 1600 50  0000 C CNN
-F 2 "" H 6250 1750 50  0001 C CNN
+F 2 "Crystal:Crystal_HC18-U_Horizontal" H 6250 1750 50  0001 C CNN
 F 3 "~" H 6250 1750 50  0001 C CNN
 	1    6250 1750

Commit message: Resolves #41 : [PCB] custom footprint library for passives
Parts:
- R215, R216, R217: footprint Resistor_THT:R_Axial_DIN0204_L3.6mm_D1.6mm_P7.62mm_Horizontal -> commons_passives_THT:Passive_THT_resistor_W2.54mm_L12.70mm
Changed lines of the file:
@@
 F 0 "R217" V 6150 3250 50  0000 C CNN
 F 1 "4K7" V 6350 3250 50  0000 C CNN
-F 2 "Resistor_THT:R_Axial_DIN0204_L3.6mm_D1.6mm_P7.62mm_Horizontal" H 6250 3250 50  0001 C CNN
+F 2 "commons_passives_THT:Passive_THT_resistor_W2.54mm_L12.70mm" H 6250 3250 50  0001 C CNN
 F 3 "~" H 6250 3250 50  0001 C CNN
 	1    6250 3250
@@
 F 0 "R215" V 6150 2750 50  0000 C CNN
 F 1 "4K7" V 6350 2750 50  0000 C CNN
-F 2 "Resistor_THT:R_Axial_DIN0204_L3.6mm_D1.6mm_P7.62mm_Horizontal" H 6250 2750 50  0001 C CNN
+F 2 "commons_passives_THT:Passive_THT_resistor_W2.54mm_L12.70mm" H 6250 2750 50  0001 C CNN
 F 3 "~" H 6250 2750 50  0001 C CNN
 	1    6250 2750
@@
 F 0 "R216" V 6150 3750 50  0000 C CNN
 F 1 "4K7" V 6350 3750 50  0000 C CNN
-F 2 "Resistor_THT:R_Axial_DIN0204_L3.6mm_D1.6mm_P7.62mm_Horizontal" H 6250 3750 50  0001 C CNN
+F 2 "commons_passives_THT:Passive_THT_resistor_W2.54mm_L12.70mm" H 6250 3750 50  0001 C CNN
 F 3 "~" H 6250 3750 50  0001 C CNN
 	1    6250 3750

Commit message: [PCB] continue footprint assignation
Parts:
- C219, C220: footprint (none) -> commons_passives_THT:Passive_THT_capacitor_W2.54mm_L10.16mm
- C221, C229, C230, C900: footprint (none) -> commons_passives_THT:Passive_THT_capacitor_ceramic_radial_W5.08mm_L6.35mm_X11.43mm
Changed lines of the file:
@@
 F 0 "C900" H 4575 8650 50  0000 L CNN
 F 1 "0.1uF" H 4575 8450 50  0000 L CNN
-F 2 "" H 4588 8400 50  0001 C CNN
+F 2 "commons_passives_THT:Passive_THT_capacitor_ceramic_radial_W5.08mm_L6.35mm_X11.43mm" H 4588 8400 50  0001 C CNN
 F 3 "~" H 4550 8550 50  0001 C CNN
 	1    4550 8550
@@
 F 0 "C230" H 4275 7200 50  0000 L CNN
 F 1 "0.1uF" H 4275 7000 50  0000 L CNN
-F 2 "" H 4288 6950 50  0001 C CNN
+F 2 "commons_passives_THT:Passive_THT_capacitor_ceramic_radial_W5.08mm_L6.35mm_X11.43mm" H 4288 6950 50  0001 C CNN
 F 3 "~" H 4250 7100 50  0001 C CNN
 	1    4250 7100
@@
 F 0 "C229" H 5275 5400 50  0000 L CNN
 F 1 "0.1uF" H 5275 5200 50  0000 L CNN
-F 2 "" H 5288 5150 50  0001 C CNN
+F 2 "commons_passives_THT:Passive_THT_capacitor_ceramic_radial_W5.08mm_L6.35mm_X11.43mm" H 5288 5150 50  0001 C CNN
 F 3 "~" H 5250 5300 50  0001 C CNN
 	1    5250 5300
@@
 F 0 "C221" H 1025 3200 50  0000 L CNN
 F 1 "0.1uF" H 1025 3000 50  0000 L CNN
-F 2 "" H 1038 2950 50  0001 C CNN
+F 2 "commons_passives_THT:Passive_THT_capacitor_ceramic_radial_W5.08mm_L6.35mm_X11.43mm" H 1038 2950 50  0001 C CNN
 F 3 "~" H 1000 3100 50  0001 C CNN
 	1    1000 3100
@@
 F 0 "C219" H 5775 2100 50  0000 L CNN
 F 1 "30pF" H 5775 1900 50  0000 L CNN
-F 2 "" H 5788 1850 50  0001 C CNN
+F 2 "commons_passives_THT:Passive_THT_capacitor_W2.54mm_L10.16mm" H 5788 1850 50  0001 C CNN
 F 3 "~" H 5750 2000 50  0001 C CNN
 	1    5750 2000
@@
 F 0 "C220" H 6775 2100 50  0000 L CNN
 F 1 "30pF" H 6775 1900 50  0000 L CNN
-F 2 "" H 6788 1850 50  0001 C CNN
+F 2 "commons_passives_THT:Passive_THT_capacitor_W2.54mm_L10.16mm" H 6788 1850 50  0001 C CNN
 F 3 "~" H 6750 2000 50  0001 C CNN
 	1    6750 2000

Commit message: [PCB] done E0..7 and RAM connectors
Parts:
- U203: footprint Package_DIP:DIP-40_W15.24mm_LongPads -> Package_DIP:DIP-48_W15.24mm_Socket_LongPads
Changed lines of the file:
@@
 F 0 "U203" H 2400 4350 50  0000 L TNN
 F 1 "MC68901_DIP_48_PHY" H 2400 4250 50  0000 L TNB
-F 2 "Package_DIP:DIP-40_W15.24mm_LongPads" H 2400 4450 50  0001 L TNN
+F 2 "Package_DIP:DIP-48_W15.24mm_Socket_LongPads" H 2400 4450 50  0001 L TNN
 F 3 "" H 2400 4550 50  0001 L TNN
 	1    2850 2900
