File: atari-16-32-bits/motherboards/c300780-001/subsheet_601.sch (KiCad schematic (older format))
At the start: 11 parts, among them P600 10K ×8, U632 74LS244_PHY

Commit message: [PCB] continuing footprint assignement
Parts:
- E0, E1, E2, E3, E4, E5, E6, E7: footprint (none) -> Jumper:SolderJumper-2_P1.3mm_Open_Pad1.0x1.5mm
Changed lines of the file:
@@
 F 0 "E0" H 2000 2080 50  0000 C CNN
 F 1 "SolderJumper_2_Open" H 2000 1900 50  0000 C CNN
-F 2 "" H 2000 2000 50  0001 C CNN
+F 2 "Jumper:SolderJumper-2_P1.3mm_Open_Pad1.0x1.5mm" H 2000 2000 50  0001 C CNN
 F 3 "~" H 2000 2000 50  0001 C CNN
 	1    2000 2000
@@
 F 0 "E1" H 2000 2580 50  0000 C CNN
 F 1 "SolderJumper_2_Open" H 2000 2400 50  0000 C CNN
-F 2 "" H 2000 2500 50  0001 C CNN
+F 2 "Jumper:SolderJumper-2_P1.3mm_Open_Pad1.0x1.5mm" H 2000 2500 50  0001 C CNN
 F 3 "~" H 2000 2500 50  0001 C CNN
 	1    2000 2500
@@
 F 0 "E2" H 2000 3080 50  0000 C CNN
 F 1 "SolderJumper_2_Open" H 2000 2900 50  0000 C CNN
-F 2 "" H 2000 3000 50  0001 C CNN
+F 2 "Jumper:SolderJumper-2_P1.3mm_Open_Pad1.0x1.5mm" H 2000 3000 50  0001 C CNN
 F 3 "~" H 2000 3000 50  0001 C CNN
 	1    2000 3000
@@
 F 0 "E3" H 2000 3580 50  0000 C CNN
 F 1 "SolderJumper_2_Open" H 2000 3400 50  0000 C CNN
-F 2 "" H 2000 3500 50  0001 C CNN
+F 2 "Jumper:SolderJumper-2_P1.3mm_Open_Pad1.0x1.5mm" H 2000 3500 50  0001 C CNN
 F 3 "~" H 2000 3500 50  0001 C CNN
 	1    2000 3500
@@
 F 0 "E4" H 2000 4080 50  0000 C CNN
 F 1 "SolderJumper_2_Open" H 2000 3900 50  0000 C CNN
-F 2 "" H 2000 4000 50  0001 C CNN
+F 2 "Jumper:SolderJumper-2_P1.3mm_Open_Pad1.0x1.5mm" H 2000 4000 50  0001 C CNN
 F 3 "~" H 2000 4000 50  0001 C CNN
 	1    2000 4000
@@
 F 0 "E5" H 2000 4580 50  0000 C CNN
 F 1 "SolderJumper_2_Open" H 2000 4400 50  0000 C CNN
-F 2 "" H 2000 4500 50  0001 C CNN
+F 2 "Jumper:SolderJumper-2_P1.3mm_Open_Pad1.0x1.5mm" H 2000 4500 50  0001 C CNN
 F 3 "~" H 2000 4500 50  0001 C CNN
 	1    2000 4500
@@
 F 0 "E6" H 2000 5080 50  0000 C CNN
 F 1 "SolderJumper_2_Open" H 2000 4900 50  0000 C CNN
-F 2 "" H 2000 5000 50  0001 C CNN
+F 2 "Jumper:SolderJumper-2_P1.3mm_Open_Pad1.0x1.5mm" H 2000 5000 50  0001 C CNN
 F 3 "~" H 2000 5000 50  0001 C CNN
 	1    2000 5000
@@
 F 0 "E7" H 2000 5580 50  0000 C CNN
 F 1 "SolderJumper_2_Open" H 2000 5400 50  0000 C CNN
-F 2 "" H 2000 5500 50  0001 C CNN
+F 2 "Jumper:SolderJumper-2_P1.3mm_Open_Pad1.0x1.5mm" H 2000 5500 50  0001 C CNN
 F 3 "~" H 2000 5500 50  0001 C CNN
 	1    2000 5500

Commit message: [PCB] continue footprint assignation
Parts:
- C632: footprint (none) -> commons_passives_THT:Passive_THT_capacitor_ceramic_radial_W5.08mm_L6.35mm_X11.43mm
Changed lines of the file:
@@
 F 0 "C632" H 7025 2600 50  0000 L CNN
 F 1 "0.1uF" H 7025 2400 50  0000 L CNN
-F 2 "" H 7038 2350 50  0001 C CNN
+F 2 "commons_passives_THT:Passive_THT_capacitor_ceramic_radial_W5.08mm_L6.35mm_X11.43mm" H 7038 2350 50  0001 C CNN
 F 3 "~" H 7000 2500 50  0001 C CNN
 	1    7000 2500

Commit message: [PCB] done E0..7 and RAM connectors
Parts:
- C632: footprint commons_passives_THT:Passive_THT_capacitor_ceramic_radial_W5.08mm_L6.35mm_X11.43mm -> commons_passives_THT:Passive_THT_capacitor_mlcc_W2.54mm_L7.62mm
Changed lines of the file:
@@
 F 0 "C632" H 7025 2600 50  0000 L CNN
 F 1 "0.1uF" H 7025 2400 50  0000 L CNN
-F 2 "commons_passives_THT:Passive_THT_capacitor_ceramic_radial_W5.08mm_L6.35mm_X11.43mm" H 7038 2350 50  0001 C CNN
+F 2 "commons_passives_THT:Passive_THT_capacitor_mlcc_W2.54mm_L7.62mm" H 7038 2350 50  0001 C CNN
 F 3 "~" H 7000 2500 50  0001 C CNN
 	1    7000 2500
