File: atari-16-32-bits/motherboards/c300780-001/subsheet_106.sch (KiCad schematic (older format))
At the start: 47 parts, among them Q100 2N3904, Q101 2N3904, Q102 2N3904, Q103 2N3904, Q104 2N3904, U402 32.215905 MHz (NTSC) — 32.084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, Y100 4.433618MHz, Y101 32.084988MHz

Commit message: [PCB] Assign builtins footprint when possible - resistors, ports
Parts:
- R113, R114, R115, R116, R117, R118, R119, R120, R121, R122, R123, R124, R125, R126, R127, R128, R129, R130: footprint (none) -> Resistor_THT:R_Axial_DIN0204_L3.6mm_D1.6mm_P7.62mm_Horizontal
Changed lines of the file:
@@
 F 0 "R113" H 3550 4850 50  0000 L CNN
 F 1 "22K" H 3550 4750 50  0000 L CNN
-F 2 "" H 3500 4800 50  0001 C CNN
+F 2 "Resistor_THT:R_Axial_DIN0204_L3.6mm_D1.6mm_P7.62mm_Horizontal" H 3500 4800 50  0001 C CNN
 F 3 "~" H 3500 4800 50  0001 C CNN
 	1    3500 4800
@@
 F 0 "R114" H 3550 5350 50  0000 L CNN
 F 1 "10K" H 3550 5250 50  0000 L CNN
-F 2 "" H 3500 5300 50  0001 C CNN
+F 2 "Resistor_THT:R_Axial_DIN0204_L3.6mm_D1.6mm_P7.62mm_Horizontal" H 3500 5300 50  0001 C CNN
 F 3 "~" H 3500 5300 50  0001 C CNN
 	1    3500 5300
@@
 F 0 "R116" H 5700 4800 50  0000 L CNN
 F 1 "18K" H 5700 4700 50  0000 L CNN
-F 2 "" H 5650 4750 50  0001 C CNN
+F 2 "Resistor_THT:R_Axial_DIN0204_L3.6mm_D1.6mm_P7.62mm_Horizontal" H 5650 4750 50  0001 C CNN
 F 3 "~" H 5650 4750 50  0001 C CNN
 	1    5650 4750
@@
 F 0 "R117" H 5700 5300 50  0000 L CNN
 F 1 "2K4" H 5700 5200 50  0000 L CNN
-F 2 "" H 5650 5250 50  0001 C CNN
+F 2 "Resistor_THT:R_Axial_DIN0204_L3.6mm_D1.6mm_P7.62mm_Horizontal" H 5650 5250 50  0001 C CNN
 F 3 "~" H 5650 5250 50  0001 C CNN
 	1    5650 5250
@@
 F 0 "R115" H 4550 5850 50  0000 L CNN
 F 1 "1K" H 4550 5750 50  0000 L CNN
-F 2 "" H 4500 5800 50  0001 C CNN
+F 2 "Resistor_THT:R_Axial_DIN0204_L3.6mm_D1.6mm_P7.62mm_Horizontal" H 4500 5800 50  0001 C CNN
 F 3 "~" H 4500 5800 50  0001 C CNN
 	1    4500 5800
@@
 F 0 "R118" H 6350 4600 50  0000 L CNN
 F 1 "1K" H 6350 4500 50  0000 L CNN
-F 2 "" H 6300 4550 50  0001 C CNN
+F 2 "Resistor_THT:R_Axial_DIN0204_L3.6mm_D1.6mm_P7.62mm_Horizontal" H 6300 4550 50  0001 C CNN
 F 3 "~" H 6300 4550 50  0001 C CNN
 	1    6300 4550
@@
 F 0 "R119" V 1700 7000 50  0000 C CNN
 F 1 "2K2" V 1500 7000 50  0000 C CNN
-F 2 "" V 1640 6990 50  0001 C CNN
+F 2 "Resistor_THT:R_Axial_DIN0204_L3.6mm_D1.6mm_P7.62mm_Horizontal" V 1640 6990 50  0001 C CNN
 F 3 "~" H 1600 7000 50  0001 C CNN
 	1    1600 7000
@@
 F 0 "R120" H 2300 6550 50  0000 L CNN
 F 1 "2K2" H 2300 6450 50  0000 L CNN
-F 2 "" H 2250 6500 50  0001 C CNN
+F 2 "Resistor_THT:R_Axial_DIN0204_L3.6mm_D1.6mm_P7.62mm_Horizontal" H 2250 6500 50  0001 C CNN
 F 3 "~" H 2250 6500 50  0001 C CNN
 	1    2250 6500
@@
 F 0 "R121" H 2800 6950 50  0000 L CNN
 F 1 "100K" H 2800 6850 50  0000 L CNN
-F 2 "" H 2750 6900 50  0001 C CNN
+F 2 "Resistor_THT:R_Axial_DIN0204_L3.6mm_D1.6mm_P7.62mm_Horizontal" H 2750 6900 50  0001 C CNN
 F 3 "~" H 2750 6900 50  0001 C CNN
 	1    2750 6900
@@
 F 0 "R122" H 3300 7350 50  0000 L CNN
 F 1 "100K" H 3300 7250 50  0000 L CNN
-F 2 "" H 3250 7300 50  0001 C CNN
+F 2 "Resistor_THT:R_Axial_DIN0204_L3.6mm_D1.6mm_P7.62mm_Horizontal" H 3250 7300 50  0001 C CNN
 F 3 "~" H 3250 7300 50  0001 C CNN
 	1    3250 7300
@@
 F 0 "R123" V 3850 7800 50  0000 C CNN
 F 1 "4K7" V 3650 7800 50  0000 C CNN
-F 2 "" V 3790 7790 50  0001 C CNN
+F 2 "Resistor_THT:R_Axial_DIN0204_L3.6mm_D1.6mm_P7.62mm_Horizontal" V 3790 7790 50  0001 C CNN
 F 3 "~" H 3750 7800 50  0001 C CNN
 	1    3750 7800
@@
 F 0 "R124" H 4800 7350 50  0000 L CNN
 F 1 "6K8" H 4800 7250 50  0000 L CNN
-F 2 "" H 4750 7300 50  0001 C CNN
+F 2 "Resistor_THT:R_Axial_DIN0204_L3.6mm_D1.6mm_P7.62mm_Horizontal" H 4750 7300 50  0001 C CNN
 F 3 "~" H 4750 7300 50  0001 C CNN
 	1    4750 7300
@@
 F 0 "R125" H 4800 7850 50  0000 L CNN
 F 1 "5K6" H 4800 7750 50  0000 L CNN
-F 2 "" H 4750 7800 50  0001 C CNN
+F 2 "Resistor_THT:R_Axial_DIN0204_L3.6mm_D1.6mm_P7.62mm_Horizontal" H 4750 7800 50  0001 C CNN
 F 3 "~" H 4750 7800 50  0001 C CNN
 	1    4750 7800
@@
 F 0 "R126" H 5300 8750 50  0000 L CNN
 F 1 "560" H 5300 8650 50  0000 L CNN
-F 2 "" H 5250 8700 50  0001 C CNN
+F 2 "Resistor_THT:R_Axial_DIN0204_L3.6mm_D1.6mm_P7.62mm_Horizontal" H 5250 8700 50  0001 C CNN
 F 3 "~" H 5250 8700 50  0001 C CNN
 	1    5250 8700
@@
 F 0 "R127" H 5780 8020 50  0000 L CNN
 F 1 "430" H 5780 7960 50  0000 L CNN
-F 2 "" H 5750 8000 50  0001 C CNN
+F 2 "Resistor_THT:R_Axial_DIN0204_L3.6mm_D1.6mm_P7.62mm_Horizontal" H 5750 8000 50  0001 C CNN
 F 3 "~" H 5750 8000 50  0001 C CNN
 	1    5750 8000
@@
 F 0 "R128" H 6300 7650 50  0000 L CNN
 F 1 "2K7" H 6300 7550 50  0000 L CNN
-F 2 "" H 6250 7600 50  0001 C CNN
+F 2 "Resistor_THT:R_Axial_DIN0204_L3.6mm_D1.6mm_P7.62mm_Horizontal" H 6250 7600 50  0001 C CNN
 F 3 "~" H 6250 7600 50  0001 C CNN
 	1    6250 7600
@@
 F 0 "R129" H 6300 8550 50  0000 L CNN
 F 1 "3K6" H 6300 8450 50  0000 L CNN
-F 2 "" H 6250 8500 50  0001 C CNN
+F 2 "Resistor_THT:R_Axial_DIN0204_L3.6mm_D1.6mm_P7.62mm_Horizontal" H 6250 8500 50  0001 C CNN
 F 3 "~" H 6250 8500 50  0001 C CNN
 	1    6250 8500
@@
 F 0 "R130" H 6800 8550 50  0000 L CNN
 F 1 "150" H 6800 8450 50  0000 L CNN
-F 2 "" H 6750 8500 50  0001 C CNN
+F 2 "Resistor_THT:R_Axial_DIN0204_L3.6mm_D1.6mm_P7.62mm_Horizontal" H 6750 8500 50  0001 C CNN
 F 3 "~" H 6750 8500 50  0001 C CNN
 	1    6750 8500

Commit message: [PCB] continuing footprint assignement
Parts:
- Q100, Q101, Q102, Q103, Q104: footprint (none) -> Package_TO_SOT_THT:TO-92_Inline_Wide
- Y100, Y101: footprint (none) -> Crystal:Crystal_HC18-U_Horizontal
Changed lines of the file:
@@
 F 0 "Y100" H 3000 5150 50  0000 C CNN
 F 1 "4.433618MHz" H 3000 4850 50  0000 C CNN
-F 2 "" H 3000 5000 50  0001 C CNN
+F 2 "Crystal:Crystal_HC18-U_Horizontal" H 3000 5000 50  0001 C CNN
 F 3 "~" H 3000 5000 50  0001 C CNN
 	1    3000 5000
@@
 F 0 "Q100" H 4600 5150 50  0000 L CNN
 F 1 "2N3904" H 4600 5050 50  0000 L CNN
-F 2 "" H 4600 5200 50  0001 C CNN
+F 2 "Package_TO_SOT_THT:TO-92_Inline_Wide" H 4600 5200 50  0001 C CNN
 F 3 "~" H 4400 5100 50  0001 C CNN
 	1    4400 5100
@@
 F 0 "Q101" H 6400 5100 50  0000 L CNN
 F 1 "2N3904" H 6400 5000 50  0000 L CNN
-F 2 "" H 6400 5150 50  0001 C CNN
+F 2 "Package_TO_SOT_THT:TO-92_Inline_Wide" H 6400 5150 50  0001 C CNN
 F 3 "~" H 6200 5050 50  0001 C CNN
 	1    6200 5050
@@
 F 0 "Q102" H 2350 7050 50  0000 L CNN
 F 1 "2N3904" H 2350 6950 50  0000 L CNN
-F 2 "" H 2350 7100 50  0001 C CNN
+F 2 "Package_TO_SOT_THT:TO-92_Inline_Wide" H 2350 7100 50  0001 C CNN
 F 3 "~" H 2150 7000 50  0001 C CNN
 	1    2150 7000
@@
 F 0 "Y101" H 4250 7650 50  0000 C CNN
 F 1 "32.084988MHz" H 4250 7350 50  0000 C CNN
-F 2 "" H 4250 7500 50  0001 C CNN
+F 2 "Crystal:Crystal_HC18-U_Horizontal" H 4250 7500 50  0001 C CNN
 F 3 "~" H 4250 7500 50  0001 C CNN
 	1    4250 7500
@@
 F 0 "Q103" H 5350 7650 50  0000 L CNN
 F 1 "2N3904" H 5350 7550 50  0000 L CNN
-F 2 "" H 5350 7700 50  0001 C CNN
+F 2 "Package_TO_SOT_THT:TO-92_Inline_Wide" H 5350 7700 50  0001 C CNN
 F 3 "~" H 5150 7600 50  0001 C CNN
 	1    5150 7600
@@
 F 0 "Q104" H 6850 8050 50  0000 L CNN
 F 1 "2N3904" H 6850 7950 50  0000 L CNN
-F 2 "" H 6850 8100 50  0001 C CNN
+F 2 "Package_TO_SOT_THT:TO-92_Inline_Wide" H 6850 8100 50  0001 C CNN
 F 3 "~" H 6650 8000 50  0001 C CNN
 	1    6650 8000

Commit message: Resolves #41 : [PCB] custom footprint library for passives
Parts:
- D101, D102: footprint (none) -> commons_passives_THT:Passive_THT_diode_W2.54mm_L12.70mm
- L101, L102, L103: footprint (none) -> commons_passives_THT:Passive_THT_inductor_W5.08mm_L15.24mm
- R113, R114, R115, R116, R117, R118, R119, R120, R121, R122, R123, R124, R125, R126, R127, R128, R129, R130: footprint Resistor_THT:R_Axial_DIN0204_L3.6mm_D1.6mm_P7.62mm_Horizontal -> commons_passives_THT:Passive_THT_resistor_W2.54mm_L12.70mm
Changed lines of the file:
@@
 F 0 "R113" H 3550 4850 50  0000 L CNN
 F 1 "22K" H 3550 4750 50  0000 L CNN
-F 2 "Resistor_THT:R_Axial_DIN0204_L3.6mm_D1.6mm_P7.62mm_Horizontal" H 3500 4800 50  0001 C CNN
+F 2 "commons_passives_THT:Passive_THT_resistor_W2.54mm_L12.70mm" H 3500 4800 50  0001 C CNN
 F 3 "~" H 3500 4800 50  0001 C CNN
 	1    3500 4800
@@
 F 0 "R114" H 3550 5350 50  0000 L CNN
 F 1 "10K" H 3550 5250 50  0000 L CNN
-F 2 "Resistor_THT:R_Axial_DIN0204_L3.6mm_D1.6mm_P7.62mm_Horizontal" H 3500 5300 50  0001 C CNN
+F 2 "commons_passives_THT:Passive_THT_resistor_W2.54mm_L12.70mm" H 3500 5300 50  0001 C CNN
 F 3 "~" H 3500 5300 50  0001 C CNN
 	1    3500 5300
@@
 F 0 "R116" H 5700 4800 50  0000 L CNN
 F 1 "18K" H 5700 4700 50  0000 L CNN
-F 2 "Resistor_THT:R_Axial_DIN0204_L3.6mm_D1.6mm_P7.62mm_Horizontal" H 5650 4750 50  0001 C CNN
+F 2 "commons_passives_THT:Passive_THT_resistor_W2.54mm_L12.70mm" H 5650 4750 50  0001 C CNN
 F 3 "~" H 5650 4750 50  0001 C CNN
 	1    5650 4750
@@
 F 0 "R117" H 5700 5300 50  0000 L CNN
 F 1 "2K4" H 5700 5200 50  0000 L CNN
-F 2 "Resistor_THT:R_Axial_DIN0204_L3.6mm_D1.6mm_P7.62mm_Horizontal" H 5650 5250 50  0001 C CNN
+F 2 "commons_passives_THT:Passive_THT_resistor_W2.54mm_L12.70mm" H 5650 5250 50  0001 C CNN
 F 3 "~" H 5650 5250 50  0001 C CNN
 	1    5650 5250
@@
 F 0 "R115" H 4550 5850 50  0000 L CNN
 F 1 "1K" H 4550 5750 50  0000 L CNN
-F 2 "Resistor_THT:R_Axial_DIN0204_L3.6mm_D1.6mm_P7.62mm_Horizontal" H 4500 5800 50  0001 C CNN
+F 2 "commons_passives_THT:Passive_THT_resistor_W2.54mm_L12.70mm" H 4500 5800 50  0001 C CNN
 F 3 "~" H 4500 5800 50  0001 C CNN
 	1    4500 5800
@@
 F 0 "R118" H 6350 4600 50  0000 L CNN
 F 1 "1K" H 6350 4500 50  0000 L CNN
-F 2 "Resistor_THT:R_Axial_DIN0204_L3.6mm_D1.6mm_P7.62mm_Horizontal" H 6300 4550 50  0001 C CNN
+F 2 "commons_passives_THT:Passive_THT_resistor_W2.54mm_L12.70mm" H 6300 4550 50  0001 C CNN
 F 3 "~" H 6300 4550 50  0001 C CNN
 	1    6300 4550
@@
 F 0 "L101" H 1280 8040 50  0000 L CNN
 F 1 "0.27uH" H 1280 7960 50  0000 L CNN
-F 2 "" H 1250 8000 50  0001 C CNN
+F 2 "commons_passives_THT:Passive_THT_inductor_W5.08mm_L15.24mm" H 1250 8000 50  0001 C CNN
 F 3 "~" H 1250 8000 50  0001 C CNN
 	1    1250 8000
@@
 F 0 "R119" V 1700 7000 50  0000 C CNN
 F 1 "2K2" V 1500 7000 50  0000 C CNN
-F 2 "Resistor_THT:R_Axial_DIN0204_L3.6mm_D1.6mm_P7.62mm_Horizontal" V 1640 6990 50  0001 C CNN
+F 2 "commons_passives_THT:Passive_THT_resistor_W2.54mm_L12.70mm" V 1640 6990 50  0001 C CNN
 F 3 "~" H 1600 7000 50  0001 C CNN
 	1    1600 7000
@@
 F 0 "R120" H 2300 6550 50  0000 L CNN
 F 1 "2K2" H 2300 6450 50  0000 L CNN
-F 2 "Resistor_THT:R_Axial_DIN0204_L3.6mm_D1.6mm_P7.62mm_Horizontal" H 2250 6500 50  0001 C CNN
+F 2 "commons_passives_THT:Passive_THT_resistor_W2.54mm_L12.70mm" H 2250 6500 50  0001 C CNN
 F 3 "~" H 2250 6500 50  0001 C CNN
 	1    2250 6500
@@
 F 0 "R121" H 2800 6950 50  0000 L CNN
 F 1 "100K" H 2800 6850 50  0000 L CNN
-F 2 "Resistor_THT:R_Axial_DIN0204_L3.6mm_D1.6mm_P7.62mm_Horizontal" H 2750 6900 50  0001 C CNN
+F 2 "commons_passives_THT:Passive_THT_resistor_W2.54mm_L12.70mm" H 2750 6900 50  0001 C CNN
 F 3 "~" H 2750 6900 50  0001 C CNN
 	1    2750 6900
@@
 F 0 "R122" H 3300 7350 50  0000 L CNN
 F 1 "100K" H 3300 7250 50  0000 L CNN
-F 2 "Resistor_THT:R_Axial_DIN0204_L3.6mm_D1.6mm_P7.62mm_Horizontal" H 3250 7300 50  0001 C CNN
+F 2 "commons_passives_THT:Passive_THT_resistor_W2.54mm_L12.70mm" H 3250 7300 50  0001 C CNN
 F 3 "~" H 3250 7300 50  0001 C CNN
 	1    3250 7300
@@
 F 0 "L102" V 3700 7500 50  0000 C CNN
 F 1 "1.5uH" V 3825 7500 50  0000 C CNN
-F 2 "" H 3750 7500 50  0001 C CNN
+F 2 "commons_passives_THT:Passive_THT_inductor_W5.08mm_L15.24mm" H 3750 7500 50  0001 C CNN
 F 3 "~" H 3750 7500 50  0001 C CNN
 	1    3750 7500
@@
 F 0 "R123" V 3850 7800 50  0000 C CNN
 F 1 "4K7" V 3650 7800 50  0000 C CNN
-F 2 "Resistor_THT:R_Axial_DIN0204_L3.6mm_D1.6mm_P7.62mm_Horizontal" V 3790 7790 50  0001 C CNN
+F 2 "commons_passives_THT:Passive_THT_resistor_W2.54mm_L12.70mm" V 3790 7790 50  0001 C CNN
 F 3 "~" H 3750 7800 50  0001 C CNN
 	1    3750 7800
@@
 F 0 "D102" V 2650 8300 50  0000 L CNN
 F 1 "1SV69" V 2850 8300 50  0000 L CNN
-F 2 "" H 2750 8250 50  0001 C CNN
+F 2 "commons_passives_THT:Passive_THT_diode_W2.54mm_L12.70mm" H 2750 8250 50  0001 C CNN
 F 3 "~" H 2750 8250 50  0001 C CNN
 	1    2750 8250
@@
 F 0 "D101" V 2150 8300 50  0000 L CNN
 F 1 "1SV69" V 2350 8300 50  0000 L CNN
-F 2 "" H 2250 8250 50  0001 C CNN
+F 2 "commons_passives_THT:Passive_THT_diode_W2.54mm_L12.70mm" H 2250 8250 50  0001 C CNN
 F 3 "~" H 2250 8250 50  0001 C CNN
 	1    2250 8250
@@
 F 0 "R124" H 4800 7350 50  0000 L CNN
 F 1 "6K8" H 4800 7250 50  0000 L CNN
-F 2 "Resistor_THT:R_Axial_DIN0204_L3.6mm_D1.6mm_P7.62mm_Horizontal" H 4750 7300 50  0001 C CNN
+F 2 "commons_passives_THT:Passive_THT_resistor_W2.54mm_L12.70mm" H 4750 7300 50  0001 C CNN
 F 3 "~" H 4750 7300 50  0001 C CNN
 	1    4750 7300
@@
 F 0 "R125" H 4800 7850 50  0000 L CNN
 F 1 "5K6" H 4800 7750 50  0000 L CNN
-F 2 "Resistor_THT:R_Axial_DIN0204_L3.6mm_D1.6mm_P7.62mm_Horizontal" H 4750 7800 50  0001 C CNN
+F 2 "commons_passives_THT:Passive_THT_resistor_W2.54mm_L12.70mm" H 4750 7800 50  0001 C CNN
 F 3 "~" H 4750 7800 50  0001 C CNN
 	1    4750 7800
@@
 F 0 "L103" H 5280 7140 50  0000 L CNN
 F 1 "1uH" H 5280 7060 50  0000 L CNN
-F 2 "" H 5250 7100 50  0001 C CNN
+F 2 "commons_passives_THT:Passive_THT_inductor_W5.08mm_L15.24mm" H 5250 7100 50  0001 C CNN
 F 3 "~" H 5250 7100 50  0001 C CNN
 	1    5250 7100
@@
 F 0 "R126" H 5300 8750 50  0000 L CNN
 F 1 "560" H 5300 8650 50  0000 L CNN
-F 2 "Resistor_THT:R_Axial_DIN0204_L3.6mm_D1.6mm_P7.62mm_Horizontal" H 5250 8700 50  0001 C CNN
+F 2 "commons_passives_THT:Passive_THT_resistor_W2.54mm_L12.70mm" H 5250 8700 50  0001 C CNN
 F 3 "~" H 5250 8700 50  0001 C CNN
 	1    5250 8700
@@
 F 0 "R127" H 5780 8020 50  0000 L CNN
 F 1 "430" H 5780 7960 50  0000 L CNN
-F 2 "Resistor_THT:R_Axial_DIN0204_L3.6mm_D1.6mm_P7.62mm_Horizontal" H 5750 8000 50  0001 C CNN
+F 2 "commons_passives_THT:Passive_THT_resistor_W2.54mm_L12.70mm" H 5750 8000 50  0001 C CNN
 F 3 "~" H 5750 8000 50  0001 C CNN
 	1    5750 8000
@@
 F 0 "R128" H 6300 7650 50  0000 L CNN
 F 1 "2K7" H 6300 7550 50  0000 L CNN
-F 2 "Resistor_THT:R_Axial_DIN0204_L3.6mm_D1.6mm_P7.62mm_Horizontal" H 6250 7600 50  0001 C CNN
+F 2 "commons_passives_THT:Passive_THT_resistor_W2.54mm_L12.70mm" H 6250 7600 50  0001 C CNN
 F 3 "~" H 6250 7600 50  0001 C CNN
 	1    6250 7600
@@
 F 0 "R129" H 6300 8550 50  0000 L CNN
 F 1 "3K6" H 6300 8450 50  0000 L CNN
-F 2 "Resistor_THT:R_Axial_DIN0204_L3.6mm_D1.6mm_P7.62mm_Horizontal" H 6250 8500 50  0001 C CNN
+F 2 "commons_passives_THT:Passive_THT_resistor_W2.54mm_L12.70mm" H 6250 8500 50  0001 C CNN
 F 3 "~" H 6250 8500 50  0001 C CNN
 	1    6250 8500
@@
 F 0 "R130" H 6800 8550 50  0000 L CNN
 F 1 "150" H 6800 8450 50  0000 L CNN
-F 2 "Resistor_THT:R_Axial_DIN0204_L3.6mm_D1.6mm_P7.62mm_Horizontal" H 6750 8500 50  0001 C CNN
+F 2 "commons_passives_THT:Passive_THT_resistor_W2.54mm_L12.70mm" H 6750 8500 50  0001 C CNN
 F 3 "~" H 6750 8500 50  0001 C CNN
 	1    6750 8500

Commit message: [PCB] continue footprint assignation
Parts:
- C115, C121, C123, C124, C125, C126, C127, C128, C129: footprint (none) -> commons_passives_THT:Passive_THT_capacitor_W2.54mm_L10.16mm
- C116: footprint (none) -> commons_passives_THT:Passive_THT_capacitor_mlcc_W2.54mm_L10.16mm
- C118, C119, C120, C122: footprint (none) -> commons_passives_THT:Passive_THT_capacitor_W2.54mm_L12.70mm
Changed lines of the file:
@@
 F 0 "C115" H 1025 5350 50  0000 L CNN
 F 1 "4700pF" H 1025 5150 50  0000 L CNN
-F 2 "" H 1038 5100 50  0001 C CNN
+F 2 "commons_passives_THT:Passive_THT_capacitor_W2.54mm_L10.16mm" H 1038 5100 50  0001 C CNN
 F 3 "~" H 1000 5250 50  0001 C CNN
 	1    1000 5250
@@
 F 0 "C120" H 1525 5350 50  0000 L CNN
 F 1 "1000pF" H 1525 5150 50  0000 L CNN
-F 2 "" H 1538 5100 50  0001 C CNN
+F 2 "commons_passives_THT:Passive_THT_capacitor_W2.54mm_L12.70mm" H 1538 5100 50  0001 C CNN
 F 3 "~" H 1500 5250 50  0001 C CNN
 	1    1500 5250
@@
 F 0 "C118" H 2525 5350 50  0000 L CNN
 F 1 "8.2pF" H 2525 5150 50  0000 L CNN
-F 2 "" H 2538 5100 50  0001 C CNN
+F 2 "commons_passives_THT:Passive_THT_capacitor_W2.54mm_L12.70mm" H 2538 5100 50  0001 C CNN
 F 3 "~" H 2500 5250 50  0001 C CNN
 	1    2500 5250
@@
 F 0 "C119" H 4025 5450 50  0000 L CNN
 F 1 "470pF" H 4025 5250 50  0000 L CNN
-F 2 "" H 4038 5200 50  0001 C CNN
+F 2 "commons_passives_THT:Passive_THT_capacitor_W2.54mm_L12.70mm" H 4038 5200 50  0001 C CNN
 F 3 "~" H 4000 5350 50  0001 C CNN
 	1    4000 5350
@@
 F 0 "C121" H 5175 5300 50  0000 L CNN
 F 1 "100pF" H 5175 5100 50  0000 L CNN
-F 2 "" H 5188 5050 50  0001 C CNN
+F 2 "commons_passives_THT:Passive_THT_capacitor_W2.54mm_L10.16mm" H 5188 5050 50  0001 C CNN
 F 3 "~" H 5150 5200 50  0001 C CNN
 	1    5150 5200
@@
 F 0 "C122" H 5175 5800 50  0000 L CNN
 F 1 "220pF" H 5175 5600 50  0000 L CNN
-F 2 "" H 5188 5550 50  0001 C CNN
+F 2 "commons_passives_THT:Passive_THT_capacitor_W2.54mm_L12.70mm" H 5188 5550 50  0001 C CNN
 F 3 "~" H 5150 5700 50  0001 C CNN
 	1    5150 5700
@@
 F 0 "C116" H 1275 8600 50  0000 L CNN
 F 1 "0.47uF" H 1275 8400 50  0000 L CNN
-F 2 "" H 1288 8350 50  0001 C CNN
+F 2 "commons_passives_THT:Passive_THT_capacitor_mlcc_W2.54mm_L10.16mm" H 1288 8350 50  0001 C CNN
 F 3 "~" H 1250 8500 50  0001 C CNN
 	1    1250 8500
@@
 F 0 "C124" H 2775 7450 50  0000 L CNN
 F 1 "22nF" H 2775 7250 50  0000 L CNN
-F 2 "" H 2788 7200 50  0001 C CNN
+F 2 "commons_passives_THT:Passive_THT_capacitor_W2.54mm_L10.16mm" H 2788 7200 50  0001 C CNN
 F 3 "~" H 2750 7350 50  0001 C CNN
 	1    2750 7350
@@
 F 0 "C129" H 3275 8350 50  0000 L CNN
 F 1 "27pF" H 3275 8150 50  0000 L CNN
-F 2 "" H 3288 8100 50  0001 C CNN
+F 2 "commons_passives_THT:Passive_THT_capacitor_W2.54mm_L10.16mm" H 3288 8100 50  0001 C CNN
 F 3 "~" H 3250 8250 50  0001 C CNN
 	1    3250 8250
@@
 F 0 "C127" H 5775 8850 50  0000 L CNN
 F 1 "68pF" H 5775 8650 50  0000 L CNN
-F 2 "" H 5788 8600 50  0001 C CNN
+F 2 "commons_passives_THT:Passive_THT_capacitor_W2.54mm_L10.16mm" H 5788 8600 50  0001 C CNN
 F 3 "~" H 5750 8750 50  0001 C CNN
 	1    5750 8750
@@
 F 0 "C125" H 5775 7150 50  0000 L CNN
 F 1 "8.2pF" H 5775 6950 50  0000 L CNN
-F 2 "" H 5788 6900 50  0001 C CNN
+F 2 "commons_passives_THT:Passive_THT_capacitor_W2.54mm_L10.16mm" H 5788 6900 50  0001 C CNN
 F 3 "~" H 5750 7050 50  0001 C CNN
 	1    5750 7050
@@
 F 0 "C126" H 5775 7650 50  0000 L CNN
 F 1 "33pF" H 5775 7450 50  0000 L CNN
-F 2 "" H 5788 7400 50  0001 C CNN
+F 2 "commons_passives_THT:Passive_THT_capacitor_W2.54mm_L10.16mm" H 5788 7400 50  0001 C CNN
 F 3 "~" H 5750 7550 50  0001 C CNN
 	1    5750 7550
@@
 F 0 "C123" H 7025 5600 50  0000 L CNN
 F 1 "1000pF" H 7025 5400 50  0000 L CNN
-F 2 "" H 7038 5350 50  0001 C CNN
+F 2 "commons_passives_THT:Passive_THT_capacitor_W2.54mm_L10.16mm" H 7038 5350 50  0001 C CNN
 F 3 "~" H 7000 5500 50  0001 C CNN
 	1    7000 5500
@@
 F 0 "C128" H 7025 7100 50  0000 L CNN
 F 1 "1000pF" H 7025 6900 50  0000 L CNN
-F 2 "" H 7038 6850 50  0001 C CNN
+F 2 "commons_passives_THT:Passive_THT_capacitor_W2.54mm_L10.16mm" H 7038 6850 50  0001 C CNN
 F 3 "~" H 7000 7000 50  0001 C CNN
 	1    7000 7000

Commit message: [PCB] continue footprints assignements
Parts:
- C409: footprint (none) -> commons_passives_THT:Passive_THT_capacitor_mlcc_W2.54mm_L7.62mm
Changed lines of the file:
@@
 F 0 "C409" H 3275 2350 50  0000 L CNN
 F 1 "100pF" H 3275 2150 50  0000 L CNN
-F 2 "" H 3288 2100 50  0001 C CNN
+F 2 "commons_passives_THT:Passive_THT_capacitor_mlcc_W2.54mm_L7.62mm" H 3288 2100 50  0001 C CNN
 F 3 "~" H 3250 2250 50  0001 C CNN
 	1    3250 2250

Commit message: [PCB] done assigning all the passives and builtin footprints
Parts:
- C117: footprint (none) -> commons_passives_THT:Passive_THT_variable_capacitor_rad_D7.62mm_P5.08mm
Changed lines of the file:
@@
 F 0 "C117" H 2025 5175 50  0000 L CNN
 F 1 "2.7–10pF" H 2025 5100 50  0000 L CNN
-F 2 "" H 2000 5250 50  0001 C CNN
+F 2 "commons_passives_THT:Passive_THT_variable_capacitor_rad_D7.62mm_P5.08mm" H 2000 5250 50  0001 C CNN
 F 3 "~" H 2000 5250 50  0001 C CNN
 	1    2000 5250

Commit message: Fixed : wrong pin numbers for transistors, should be ebc, not bce
Parts:
- Q100, Q101, Q102, Q103, Q104: symbol Device:Q_NPN_BCE -> Device:Q_NPN_EBC
Connections:
- net 32MHZ: now also Q104.1 (E); no longer Q104.3 (E)
- net CCLK: now also Q101.3 (C); no longer Q101.2 (C)
- net GND: now also Q101.1 (E), Q102.1 (E); no longer Q101.3 (E), Q102.3 (E)
- net VCC: now also Q100.3 (C); no longer Q100.2 (C)
- net VLL: now also Q104.3 (C); no longer Q104.2 (C)
- net at C119.1, R113.2, R114.1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: now also Q100.2 (B); no longer Q100.1 (B)
- net at C121.1, R116.2, R117.1: now also Q101.2 (B); no longer Q101.1 (B)
- net at C119.2, C121.2, C122.1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: now also Q100.1 (E); no longer Q100.3 (E)
- net at R119.1: now also Q102.2 (B); no longer Q102.1 (B)
- net at R120.2, R121.1: now also Q102.3 (C); no longer Q102.2 (C)
- net at R124.2, R125.1, Y101.1: now also Q103.2 (B); no longer Q103.1 (B)
- net at C125.2, C126.1, L103.2: now also Q103.3 (C); no longer Q103.2 (C)
- net at C127.1, R126.1: now also Q103.1 (E); no longer Q103.3 (E)
- net at C126.2, R127.1, R127.2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: now also Q104.2 (B); no longer Q104.1 (B)
Changed lines of the file:
@@
 	2000 5000 2500 5000
 $Comp
-L Device:Q_NPN_BCE Q100
+L Device:Q_NPN_EBC Q100
 U 1 1 60873EA1
 P 4400 5100
@@
 	4500 5450 4500 5600
 $Comp
-L Device:Q_NPN_BCE Q101
+L Device:Q_NPN_EBC Q101
 U 1 1 60882AEC
 P 6200 5050
@@
 $EndComp
 $Comp
-L Device:Q_NPN_BCE Q102
+L Device:Q_NPN_EBC Q102
 U 1 1 608A007A
 P 2150 7000
@@
 	4750 7500 4750 7600
 $Comp
-L Device:Q_NPN_BCE Q103
+L Device:Q_NPN_EBC Q103
 U 1 1 608DF2CF
 P 5150 7600
@@
 $EndComp
 $Comp
-L Device:Q_NPN_BCE Q104
+L Device:Q_NPN_EBC Q104
 U 1 1 6093547F
 P 6650 8000
