File: atari-16-32-bits/motherboards/c300780-001/subsheet_501.sch (KiCad schematic (older format))
At the start: 11 parts, among them P500 4K7 ×8, P501 4K7 ×8, P502 4K7 ×8, U509 74LS244_PHY, U510 74LS244_PHY, U511 74LS373_PHY, U512 74LS244_PHY

Commit message: Fixes #51 : [bug][schematics] fix the association of mlcc capacitors and their footprint in schematics to match the association done in the pcb
Parts:
- C550, C551, C552, C553: footprint commons_passives_THT:Passive_THT_capacitor_ceramic_radial_W5.08mm_L6.35mm_X11.43mm -> commons_passives_THT:Passive_THT_capacitor_mlcc_W2.54mm_L7.62mm
Changed lines of the file:
@@
 F 0 "C553" H 1775 2350 50  0000 L CNN
 F 1 "0.1uF" H 1775 2150 50  0000 L CNN
-F 2 "commons_passives_THT:Passive_THT_capacitor_ceramic_radial_W5.08mm_L6.35mm_X11.43mm" H 1788 2100 50  0001 C CNN
+F 2 "commons_passives_THT:Passive_THT_capacitor_mlcc_W2.54mm_L7.62mm" H 1788 2100 50  0001 C CNN
 F 3 "~" H 1750 2250 50  0001 C CNN
 	1    1750 2250
@@
 F 0 "C551" H 1775 3850 50  0000 L CNN
 F 1 "0.1uF" H 1775 3650 50  0000 L CNN
-F 2 "commons_passives_THT:Passive_THT_capacitor_ceramic_radial_W5.08mm_L6.35mm_X11.43mm" H 1788 3600 50  0001 C CNN
+F 2 "commons_passives_THT:Passive_THT_capacitor_mlcc_W2.54mm_L7.62mm" H 1788 3600 50  0001 C CNN
 F 3 "~" H 1750 3750 50  0001 C CNN
 	1    1750 3750
@@
 F 0 "C552" H 1775 5350 50  0000 L CNN
 F 1 "0.1uF" H 1775 5150 50  0000 L CNN
-F 2 "commons_passives_THT:Passive_THT_capacitor_ceramic_radial_W5.08mm_L6.35mm_X11.43mm" H 1788 5100 50  0001 C CNN
+F 2 "commons_passives_THT:Passive_THT_capacitor_mlcc_W2.54mm_L7.62mm" H 1788 5100 50  0001 C CNN
 F 3 "~" H 1750 5250 50  0001 C CNN
 	1    1750 5250
@@
 F 0 "C550" H 1775 6850 50  0000 L CNN
 F 1 "0.1uF" H 1775 6650 50  0000 L CNN
-F 2 "commons_passives_THT:Passive_THT_capacitor_ceramic_radial_W5.08mm_L6.35mm_X11.43mm" H 1788 6600 50  0001 C CNN
+F 2 "commons_passives_THT:Passive_THT_capacitor_mlcc_W2.54mm_L7.62mm" H 1788 6600 50  0001 C CNN
 F 3 "~" H 1750 6750 50  0001 C CNN
 	1    1750 6750
